File: 490_0/490_0.kicad_sch (KiCad schematic)
At the start: 33 parts, among them J1 DF40C-100DS-0.4V_51_, J2 DF40C-100DS-0.4V_51_, J3 Micro_SD_Card, Q1 NMOS, SW1 SW_DPST_x2, U1 RT9742GGJ5

Commit message: USB and POWER
Parts:
- added D2: USBLC6-2P6, PCM_Package_TO_SOT_SMD_AKL:SOT-666, symbol PCM_Diode_TVS_AKL:USBLC6-2P6
- added J4: USB_A, symbol Connector:USB_A
- added J5: USB_C_Receptacle, PCM_SparkFun-Connector:USB-C_16, symbol PCM_SparkFun-Connector:USB_C_Receptacle
Connections:
- net GND: now also D2.2 (VN), J4.4 (GND), J4.5 (Shield)
- net USB_N: now also D2.4 (L2)
- net USB_P: now also D2.6 (L1)
- new net: D2.3 (L2), J4.2 (D-)
- new net: D2.1 (L1), J4.3 (D+)
- new net: J5.A6 (D+), J5.B6 (D+)
- new net: J5.A7 (D-), J5.B7 (D-)
- new net + 5V: D2.5 (VP), J4.1 (VBUS)

Commit message: Update 490_0.kicad_sch
Parts:
- added U2: MCP73832-2-OT, Package_TO_SOT_SMD:SOT-23-5, symbol Battery_Management:MCP73832-2-OT
Changed lines of the file:
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@@
+	)
+	(symbol
+		(lib_id "Battery_Management:MCP73832-2-OT")
+		(at 119.38 91.44 0)
+		(unit 1)
+		(exclude_from_sim no)
+		(in_bom yes)
+		(on_board yes)
+		(dnp no)
+		(fields_autoplaced yes)
+		(property "Reference" "U2"
+			(at 121.5233 81.28 0)
+			(effects
+				(font
+					(size 1.27 1.27)
+				)
+				(justify left)
+			)
+		)
+		(property "Value" "MCP73832-2-OT"
+			(at 121.5233 83.82 0)
+			(effects
+				(font
+					(size 1.27 1.27)
+				)
+				(justify left)
+			)
+		)
+		(property "Footprint" "Package_TO_SOT_SMD:SOT-23-5"
+			(at 120.65 97.79 0)
+			(effects
+				(font
+					(size 1.27 1.27)
+					(italic yes)
+				)
+				(justify left)
+				(hide yes)
+			)
+		)
+		(property "Datasheet" "http://ww1.microchip.com/downloads/en/DeviceDoc/20001984g.pdf"
+			(at 119.38 110.236 0)
+			(effects
+				(font
+					(size 1.27 1.27)
+				)
+				(hide yes)
+			)
+		)
+		(property "Description" "Single cell, Li-Ion/Li-Po charge management controller, 4.20V, Open-Drain Status Output, in SOT23-5 package"
+			(at 119.38 91.44 0)
+			(effects
+				(font
+					(size 1.27 1.27)
+				)
+				(hide yes)
+			)
+		)
+		(pin "3"
+		)
+		(pin "5"
+		)
+		(pin "4"
+		)
+		(pin "2"
+		)
+		(pin "1"
+		)
+		(instances
+			(project ""
+				(path "/365a82ed-827d-43e1-aa2f-b98221c4179c"
+					(reference "U2")
+					(unit 1)
+				)
+			)
+		)
 	)
 	(symbol

Commit message: Startted power
Parts:
- removed J5: USB_C_Receptacle, PCM_SparkFun-Connector:USB-C_16, symbol PCM_SparkFun-Connector:USB_C_Receptacle
- removed U2: MCP73832-2-OT, Package_TO_SOT_SMD:SOT-23-5, symbol Battery_Management:MCP73832-2-OT
- added C2: 10uF, PCM_SparkFun-Capacitor:C_0603_1608Metric, symbol PCM_SparkFun-Capacitor:10uF_0603_10V_20%
- added J6: USB_B_Micro, symbol Connector:USB_B_Micro
- added LED3: LED_1.8mm_Red, PCM_LED_THT_AKL:LED_D1.8mm_W3.3mm_H2.4mm, symbol PCM_LED_AKL:LED_1.8mm_Red
- added LED4: LED_1.8mm_SMD_Green, PCM_LED_SMD_AKL:LED_1.8mm_GullWing, symbol PCM_LED_AKL:LED_1.8mm_SMD_Green
- added R21, R22: 1k, Resistor_THT:R_Axial_DIN0207_L6.3mm_D2.5mm_P10.16mm_Horizontal, symbol PCM_SL_Resistors:1k
- added R23: 2k_0603, 4ms_Resistor:R_0603, symbol PCM_4ms_Resistor:2k_0603
- added U2: TP4057, Package_TO_SOT_SMD:TSOT-23-6, symbol Battery_Management:TP4057
- added U3: DW01, DW01:SOT23-6, symbol capstone_parts:DW01
Connections:
- net GND: now also C2.2, J6.5 (GND), R23.2, U2.2 (GND)
- new net: R21.2, U2.1 (~{CHRG})
- new net: C2.1, J6.1 (VBUS), LED3.2 (A), LED4.2 (A), U2.4 (V_{CC})
- new net: R22.2, U2.5 (STDBY)
- new net: R23.1, U2.6 (PROG)
- new net: LED3.1 (K), R21.1
- new net: LED4.1 (K), R22.1
- new net +BATT: U2.3 (BAT)

Commit message: Added USB hub
Parts:
- removed J4: USB_A, symbol Connector:USB_A
- added C10, C11, C12, C13, C15, C16, C17, C18, C19, C20, C21, C23, C24, C27, C29, C31, C33, C35, C37, C38, C39, C40, C43, C44, C45, C46, C48, C50, C51, C52: 100n, symbol PCM_Elektuur:C
- added C14, C25: 22u, symbol PCM_Elektuur:C
- added C22, C26, C28, C30, C32, C34, C36, C47, C49, C7, C8, C9: 10n, symbol PCM_Elektuur:C
- added C3: 0.1uF, PCM_SparkFun-Capacitor:C_0402_1005Metric, symbol PCM_SparkFun-Capacitor:0.1uF_0402_16V_10%
- added C41, C42: 18p, symbol PCM_Elektuur:C
- added C5, C6: 150u, Capacitor_THT:CP_Radial_D5.0mm_P2.50mm, symbol PCM_SL_Devices:Capacitor_PO
- added D3, D6: USBULC6-2M6, PCM_Package_TO_SOT_SMD_AKL:SOT-666, symbol PCM_Diode_TVS_AKL:USBLC6-2P6
- added D4, D5: LED, PCM_SparkFun-LED:LED_0603_1608Metric, symbol PCM_SparkFun-LED:LED
- added FB1: 220 @ 100 MHz, symbol Device:FerriteBead
- added J4: USB3_A_Stacked, symbol Connector:USB3_A_Stacked
- added J7: USB_B_Micro, symbol Connector:USB_B_Micro
- added Q2: FS8205A, FS8205A:SOP65P640X120-8N, symbol FS8205A:FS8205A
- added R18: 2k_0603, 4ms_Resistor:R_0603, symbol PCM_4ms_Resistor:2k_0603
- added R19: 4.7k, symbol PCM_Elektuur:R
- added R20: 100ohm, Resistor_THT:R_Axial_DIN0207_L6.3mm_D2.5mm_P10.16mm_Horizontal, symbol PCM_SL_Resistors:100ohm
- added R24: 1M, symbol PCM_Elektuur:R
- added R25: 9.09k 1%, symbol PCM_Elektuur:R
- added R26, R27, R32, R33: R, symbol PCM_Elektuur:R
- added R28, R30, R31, R34, R35: 10k, symbol PCM_Elektuur:R
- added U4: TUSB7320RKMR, RKM100_5P5X5P5, symbol capstone_parts:TUSB7320RKMR
- added U5, U6: ECMF04-4HSWM10, Package_DFN_QFN:UDFN-10_1.35x2.6mm_P0.5mm, symbol Power_Protection:ECMF04-4HSWM10
- added U7: TPS2560DRCR, TPS2560DRCR:VREG_V62_16624-01YE, symbol capstone_parts:TPS2560DRCR
- added X1: ECS-480-18-33-JGN-TR, symbol PCM_Elektuur_1:X-crystal
- D2: value USBLC6-2P6 -> USBULC6-2M6
Connections:
- net + 5V: now also C43.1 (+), C44.1 (+), C46.1 (+), C50.1 (+), D3.5 (VP), D6.5 (VP), J7.1 (VBUS), U7.2 (IN), U7.3 (IN__1)
- net +3.3V: now also C23.1 (+), C24.1 (+), C38.1 (+), C39.1 (+), C40.1 (+), FB1.1, U4.A3 (VDD33), U4.A34 (VDD33), U4.A39 (VDD33), U4.A47 (VDD33), U4.A51 (VDD33)
- net +BATT: now also R20.1
- net GND: now also C10.2 (-), C11.2 (-), C12.2 (-), C13.2 (-), C14.2 (-), C15.2 (-), C16.2 (-), C17.2 (-), C18.2 (-), C19.2 (-), C20.2 (-), C21.2 (-), C22.2 (-), C23.2 (-), C24.2 (-), C25.2 (-), C26.2 (-), C27.2 (-), C28.2 (-), C29.2 (-), C30.2 (-), C31.2 (-), C32.2 (-), C33.2 (-), C34.2 (-), C35.2 (-), C36.2 (-), C37.2 (-), C38.2 (-), C39.2 (-), C40.2 (-), C41.2 (-), C42.2 (-), C43.2 (-), C44.2 (-), C45.2 (-), C46.2 (-), C47.2 (-), C48.2 (-), C49.2 (-), C5.2, C50.2 (-), C51.2 (-), C52.2 (-), C6.2, C7.2 (-), C8.2 (-), C9.2 (-), D3.2 (VN), D4.1 (K), D5.1 (K), D6.2 (VN), J4.13 (GND2), J4.4 (GND1), J7.5 (GND), Q2.6, Q2.7, R18.2, R19.2 (-), R26.2 (-), R27.2 (-), R31.2 (-), R34.2 (-), U4.A53 (VSS_NC), U4.B20 (VSS_NC), U4.B21 (VSS_OSC), U4.C1 (VSS_NC), U4.C2 (VSS_NC), U4.C3 (VSS_NC), U4.C4 (VSS_NC), U5.3 (GND), U5.8 (GND), U6.3 (GND), U6.8 (GND), U7.1 (GND), U7.11 (PAD)
- net PCIe_CLK_P: now also U4.A45 (PCIE_REFCLKP)
- net PCIe_CLK_nREQ: now also U4.B36 (*CLKREQ); no longer J2.12
- net PCIe_RX_N: now also U4.A42 (PCIE_RXN)
- net PCIe_RX_P: now also U4.B39 (PCIE_RXP)
- net PCIe_TX_N: now also U4.A41 (PCIE_TXN)
- net PCIe_TX_P: now also U4.B38 (PCIE_TXP)
- net PCIe_nRST: now also U4.A40 (*PERST)
- net USB_N: now also D3.4 (L2); no longer D2.4 (L2)
- net USB_P: now also D3.6 (L1); no longer D2.6 (L1)
- net at D2.3 (L2): now also U4.B12 (USB_DP_DN2)
- net at D2.1 (L1): now also U4.A13 (USB_DM_DN2)
- net at U3.1: now also Q2.4
- net at U3.2: now also R18.1
- net at U3.3: now also Q2.5
- net at U3.5: now also C3.2, R20.2
- net -BATT: now reaches U3.6
- net -BATT: now also C3.1, Q2.2, Q2.3
- new net: R28.2 (-), U4.A36 (*OVERCUR1), U7.10 (~{FAULT1})
- new net: U4.B33 (*PWRON1), U7.4 (EN1)
- new net: U4.B34 (*PWRON2), U7.5 (EN2)
- new net: R30.2 (-), U4.A37 (*OVERCUR2), U7.6 (~{FAULT2})
- new net: R31.1 (+), U7.7 (ILIM)
- new net: C48.1 (+), C49.1 (+), J4.19 (SHIELD), R27.1 (+)
- new net: C41.1 (+), R24.1 (+), U4.A22 (XO), X1.1 (+)
- new net: C42.1 (+), R24.2 (-), U4.A23 (XI), X1.2 (-)
- new net: D2.6 (L1), J4.11 (D2-)
- new net: D2.4 (L2), J4.12 (D2+)
- new net: J4.14 (SSRX2-), U6.10 (Out_1+)
- new net: J4.15 (SSRX2+), U6.9 (Out_1+)
- new net: J4.17 (SSTX2-), U6.7 (Out_1+)
- new net: J4.18 (SSTX2+), U6.6 (Out_1+)
- new net: R25.1 (+), U4.A24 (R1EXT)
- new net: R25.2 (-), U4.B23 (R1EXTRTN)
- new net: D6.1 (L1), U4.B18 (USB_DM_DN1)
- new net: D6.3 (L2), U4.A20 (USB_DP_DN1)
- new net: D6.4 (L2), J4.3 (D1+)
- new net: D6.6 (L1), J4.2 (D1-)
- new net: C45.1 (+), C47.1 (+), J4.19 (SHIELD), R26.1 (+)
- new net: U4.A18 (USB_SSRXN_DN1), U5.1 (In_1+)
- new net: J4.5 (SSRX1-), U5.10 (Out_1+)
- new net: U4.B16 (USB_SSRXP_DN1), U5.2 (In_1-)
- new net: U4.B15 (USB_SSTXN_DN1), U5.4 (In_1+)
- new net: U4.A17 (USB_SSTXP_DN1), U5.5 (In_1-)
- new net: J4.9 (SSTX1+), U5.6 (Out_1+)
- new net: J4.8 (SSTX1-), U5.7 (Out_1+)
- new net: J4.6 (SSRX1+), U5.9 (Out_1+)
- new net: U4.A10 (USB_SSRXN_DN2), U6.1 (In_1+)
- new net: U4.A11 (USB_SSTXP_DN2), U6.5 (In_1-)
- new net: R34.1 (+), R35.2 (-), U4.A52 (AUX_DET)
- new net: U4.B10 (USB_SSTXN_DN2), U6.4 (In_1+)
- new net: R19.1 (+), U4.B14 (FREQSEL)
- new net: U4.B9 (USB_SSRXP_DN2), U6.2 (In_1-)
- new net: D5.2 (A), R33.2 (-)
- new net: D3.3 (L2), J7.2 (D-)
- new net: D3.1 (L1), J7.3 (D+)
- new net: D4.2 (A), R32.2 (-)
- new net: Q2.1, Q2.8
- new net +1V1: C15.1 (+), C16.1 (+), C17.1 (+), C18.1 (+), C19.1 (+), C20.1 (+), C21.1 (+), C22.1 (+), C25.1 (+), C26.1 (+), C27.1 (+), C28.1 (+), C29.1 (+), C30.1 (+), C31.1 (+), C32.1 (+), C33.1 (+), C34.1 (+), C35.1 (+), C36.1 (+), C37.1 (+), U4.A1 (VDD11), U4.A12 (VDD11), U4.A16 (VDD11), U4.A28 (VDD11), U4.A31 (VDD11), U4.A33 (VDD11), U4.A38 (VDD11), U4.A4 (VDD11), U4.A50 (VDD11), U4.A6 (VDD11), U4.A9 (VDD11), U4.B1 (VDD11), U4.B17 (VDD11), U4.B19 (VDD11), U4.B24 (VDD11), U4.B37 (VDD11), U4.B40 (VDD11), U4.B42 (VDD11), U4.B44 (VDD11)
- new net +3.3VA: C10.1 (+), C11.1 (+), C12.1 (+), C13.1 (+), C14.1 (+), C7.1 (+), C8.1 (+), C9.1 (+), FB1.2, U4.A19 (VDDA_3P3), U4.A21 (VDDA_3P3), U4.A25 (VDDA_3P3), U4.A44 (VDDA_3P3), U4.B11 (VDDA_3P3), U4.B22 (VDDA_3P3)
- new net 3.3V: R28.1 (+), R30.1 (+), R35.1 (+)
- new net PCIe_CLK_N: J2.12, U4.B41 (PCIE_REFCLKN)
- new net To_GPIO: U4.A15 (*GRST), U4.A49 (GPIO[0]), U4.B3 (SMI), U4.B35 (*WAKE), U4.B46 (GPIO[1]), U4.B47 (GPIO[2]), U4.B48 (GPIO[3])
- new net To_GPIO_I2C: U4.A2 (SDA), U4.B2 (SCL)
- new net VBUS1: C5.1, C51.1 (+), J4.1 (VBUS1), R32.1 (+), U7.9 (OUT1)
- new net VBUS2: C52.1 (+), C6.1, J4.10 (VBUS2), R33.1 (+), U7.8 (OUT2)
- no-connect marks 34 -> 64
Other:
- note added: "PCIe to USB 3.0 bridge"
- moved on the sheet: U3

Commit message: Added speakers, motors and started HDMI
Parts:
- added C0(ceramic), C0(ceramic)1, C0(ceramic)2, C0(ceramic)3, C0(ceramic)4, C5(ceramic), C6(ceramic), Cx(ceramic): 100nF, Capacitor_SMD:C_0603_1608Metric, symbol Device:C
- added C0(radial), C0(radial)1, C0(radial)2, C0(radial)3, C0(radial)4, C5(radial), C6(radial), Cx(radial): 10uF, Capacitor_THT:CP_Radial_D5.0mm_P2.50mm, symbol Device:C
- added D10, D11, D12, D8, D9: D, symbol Device:D
- added D7: USBULC6-2M6, PCM_Package_TO_SOT_SMD_AKL:SOT-666, symbol PCM_Diode_TVS_AKL:USBLC6-2P6
- added FB2 (x2): FerriteBead, Capacitor_SMD:C_0603_1608Metric, symbol Device:FerriteBead_Small
- added J10, J8 (x2), J9 (x2): Conn_01x02_Pin, symbol Connector:Conn_01x02_Pin
- added J5: HDMI_D_1.4, symbol Connector:HDMI_D_1.4
- added JP10: SJ_A3, Jumper:SolderJumper-2_P1.3mm_Open_RoundedPad1.0x1.5mm, symbol Jumper:SolderJumper_2_Open
- added JP11: SJ_A4, Jumper:SolderJumper-2_P1.3mm_Open_RoundedPad1.0x1.5mm, symbol Jumper:SolderJumper_2_Open
- added JP12: SJ_A5, Jumper:SolderJumper-2_P1.3mm_Open_RoundedPad1.0x1.5mm, symbol Jumper:SolderJumper_2_Open
- added JP3: SJ_A0, Jumper:SolderJumper-2_P1.3mm_Open_RoundedPad1.0x1.5mm, symbol Jumper:SolderJumper_2_Open
- added JP8: SJ_A1, Jumper:SolderJumper-2_P1.3mm_Open_RoundedPad1.0x1.5mm, symbol Jumper:SolderJumper_2_Open
- added JP9: SJ_A2, Jumper:SolderJumper-2_P1.3mm_Open_RoundedPad1.0x1.5mm, symbol Jumper:SolderJumper_2_Open
- added PD1, PU1, R (x2), Rgd0, Rgd1, Rgd2, Rgd3, Rgd4: 100K, symbol Device:R
- added Q0, Q3 (x2), Q4, Q5: NMOS, symbol Simulation_SPICE:NMOS
- added R1G$1, R1G$2, R1G$3, R1G$4, R1G$5, R1G$6, R36: 10K, symbol Device:R
- added Rg0, Rg1, Rg2, Rg3, Rg4: 220, symbol Device:R
- added S1: Speaker_Left, Connector_JST:JST_PH_S2B-PH-K_1x02_P2.00mm_Horizontal, symbol Connector_Generic:Conn_01x02
- added S2: Speaker_Right, Connector_JST:JST_PH_S2B-PH-K_1x02_P2.00mm_Horizontal, symbol Connector_Generic:Conn_01x02
- added SW2: SW_Push0, symbol Switch:SW_Push
- added SW3: SW_Push1, symbol Switch:SW_Push
- added SW4: SW_Push2, symbol Switch:SW_Push
- added SW5: SW_Push3, symbol Switch:SW_Push
- added SW6: SW_Push4, symbol Switch:SW_Push
- added U10: PCA9685, PCA9685:TSSOP28, symbol capstone_parts:PCA9685
- added U11, U12: MAX98357A, Package_DFN_QFN:TQFN-16-1EP_3x3mm_P0.5mm_EP1.23x1.23mm_ThermalVias, symbol Audio:MAX98357A
- added U13: 74HC4051, symbol 74xx:74HC4051
- added U8, U9: ECMF04-4HSWM10, Package_DFN_QFN:UDFN-10_1.35x2.6mm_P0.5mm, symbol Power_Protection:ECMF04-4HSWM10
Connections:
- net +3.3V: now also Cx(ceramic).1, Cx(radial).1, JP10.2 (B), JP11.2 (B), JP12.2 (B), JP3.2 (B), JP8.2 (B), JP9.2 (B), PU1.1, R.1, U10.28 (VDD)
- net +5V: now also C5(ceramic).1, C5(radial).1, C6(ceramic).1, C6(radial).1, FB2.1, FB2.1
- net GND: now also C0(ceramic).2, C0(ceramic)1.2, C0(ceramic)2.2, C0(ceramic)3.2, C0(ceramic)4.2, C0(radial).2, C0(radial)1.2, C0(radial)2.2, C0(radial)3.2, C0(radial)4.2, C5(ceramic).2, C5(radial).2, C6(ceramic).2, C6(radial).2, Cx(ceramic).2, Cx(radial).2, PD1.2, Q0.3 (S), Q3.3 (S), Q3.3 (S), Q4.3 (S), Q5.3 (S), R.2, R1G$1.1, R1G$2.1, R1G$3.1, R1G$4.1, R1G$5.1, R1G$6.1, R36.1, Rgd0.1, Rgd1.1, Rgd2.1, Rgd3.1, Rgd4.1, SW2.2, SW3.2, SW4.2, SW5.2, SW6.2, U10.14 (GND), U10.25 (EXTCLK), U11.11 (GND), U11.15 (GND), U11.17 (PAD), U11.3 (GND), U12.11 (GND), U12.15 (GND), U12.17 (PAD), U12.3 (GND)
- net GPIO16: now also SW2.1
- net GPIO17: now also SW3.1
- net GPIO18: now also U11.16 (BCLK), U12.16 (BCLK)
- net GPIO19: now also U11.14 (LRCLK), U12.14 (LRCLK)
- net GPIO2: now also U10.27 (SDA)
- net GPIO20: now also U11.1 (DIN), U12.1 (DIN)
- net GPIO22: now also SW4.1
- net GPIO23: now also SW5.1
- net GPIO26: now also SW6.1
- net GPIO3: now also U10.26 (SCL)
- net HDMI0_CLK_N: now also U9.5 (In_1-)
- net HDMI0_CLK_P: now also U9.4 (In_1+)
- net HDMI0_TX0_N: now also U9.2 (In_1-)
- net HDMI0_TX0_P: now also U9.1 (In_1+)
- net HDMI0_TX1_N: now also U8.5 (In_1-)
- net HDMI0_TX1_P: now also U8.4 (In_1+)
- net HDMI0_TX2_N: now also U8.2 (In_1-)
- net HDMI0_TX2_P: now also U8.1 (In_1+)
- new net: Q4.2 (G), Rg3.2
- new net: D9.2 (A), J9.2 (Pin_2), Q0.1 (D)
- new net: Q0.2 (G), Rg0.2
- new net: D8.2 (A), J8.2 (Pin_2), Q3.1 (D)
- new net: Q3.2 (G), Rg2.2
- new net: PU1.2, U12.4 (~{SD_MODE})
- new net: J5.3 (D2+), U8.10 (Out_1+)
- new net: U8.3 (GND), U8.8 (GND)
- new net: J5.8 (D1-), U8.6 (Out_1+)
- new net: J5.6 (D1+), U8.7 (Out_1+)
- new net: J5.5 (D2-), U8.9 (Out_1+)
- new net: FB2.2, U11.7 (VDD), U11.8 (VDD)
- new net: S1.1 (Pin_1), U11.9 (OUTP)
- new net: S1.2 (Pin_2), U11.10 (OUTN)
- new net: FB2.2, U12.7 (VDD), U12.8 (VDD)
- new net: R36.2, U10.23 (#OE)
- new net: S2.1 (Pin_1), U12.9 (OUTP)
- new net: S2.2 (Pin_2), U12.10 (OUTN)
- new net: D10.2 (A), J9.2 (Pin_2), Q5.1 (D)
- new net: Q3.2 (G), Rg1.2
- new net: D11.2 (A), J10.2 (Pin_2), Q3.1 (D)
- new net: Q5.2 (G), Rg4.2
- new net: J5.9 (D0+), U9.10 (Out_1+)
- new net: U9.3 (GND), U9.8 (GND)
- new net: J5.14 (CK-), U9.6 (Out_1+)
- new net: J5.12 (CK+), U9.7 (Out_1+)
- new net: J5.11 (D0-), U9.9 (Out_1+)
- new net: D12.2 (A), J8.2 (Pin_2), Q4.1 (D)
- new net: R.1, U11.2 (GAIN_SLOT)
- new net: PD1.1, U12.2 (GAIN_SLOT)
- new net: R.2, U11.4 (~{SD_MODE})
- new net 5V: C0(ceramic).1, C0(ceramic)1.1, C0(ceramic)2.1, C0(ceramic)3.1, C0(ceramic)4.1, C0(radial).1, C0(radial)1.1, C0(radial)2.1, C0(radial)3.1, C0(radial)4.1, D10.1 (K), D11.1 (K), D12.1 (K), D8.1 (K), D9.1 (K), J10.1 (Pin_1), J8.1 (Pin_1), J8.1 (Pin_1), J9.1 (Pin_1), J9.1 (Pin_1)
- new net A0: JP12.1 (A), R1G$1.2, U10.1 (A0)
- new net A1: JP11.1 (A), R1G$2.2, U10.2 (A1)
- new net A2: JP10.1 (A), R1G$3.2, U10.3 (A2)
- new net A3: JP9.1 (A), R1G$4.2, U10.4 (A3)
- new net A4: JP8.1 (A), R1G$5.2, U10.5 (A4)
- new net A5: JP3.1 (A), R1G$6.2, U10.24 (A5)
- new net PWM0: Rg0.1, Rgd0.2, U10.6 (PWM0)
- new net PWM1: Rg2.1, Rgd2.2, U10.7 (PWM1)
- new net PWM2: Rg1.1, Rgd1.2, U10.8 (PWM2)
- new net PWM3: Rg3.1, Rgd3.2, U10.9 (PWM3)
- new net PWM4: Rg4.1, Rgd4.2, U10.10 (PWM4)
- no-connect marks 64 -> 75
Other:
- note added: "I2C Address = 1 + A5 + A4 + A3 + A2 + A1 + RW Open = 0 / Closed = 1"
- note added: "PCM_CLK"
- note added: "PCM_DIN"
- note added: "PCM_FS"
- note added: "Push-buttons"
- note added: "REMOVE, RASPBERRY CAN ALREADY DO THIS"
- note added: "Sample MUX for the PWM substitution"
- note added: "Speaker (Left)"
- note added: "Speaker (Right)"
- note added: "Vibration Motor #1"
- note added: "Vibration Motor #2"
- note added: "Vibration Motor #3"
- note added: "Vibration Motor #4"
- note added: "Vibration Motor #5"

Commit message: Power Supply
Parts:
- added C4, C53: ?, symbol PCM_Elektuur:C
- added L1: 1u, WE-MAPI_4030:WE-MAPI_4030, symbol capstone_parts:74438357010
- added R37, R38: ?, Resistor_THT:R_Axial_DIN0207_L6.3mm_D2.5mm_P10.16mm_Horizontal, symbol PCM_SL_Resistors:100ohm
- added U15: TPS61023DRLR, DRL0006A, symbol capstone_parts:TPS61023DRLR
Connections:
- net +5V: no longer J1.77, J1.79, J1.81, J1.83, J1.85, J1.87
- net +BATT: now also C4.1 (+), L1.1, U15.2 (EN), U15.3 (VIN)
- net GND: now also C4.2 (-), C53.1 (+), R38.1, U15.4 (GND)
- new net: R37.1, R38.2, U15.1 (FB)
- new net: L1.2, U15.5 (SW)
- new net: C53.2 (-), J1.77, J1.79, J1.81, J1.83, J1.85, J1.87, R37.2, U15.6 (VOUT)
Other:
- note added: "Battery Charging and Power Supply Unit"
- note added: "Micro HDMI"
- note added: "PWM and Motors"
- moved on the sheet: C0(ceramic), C0(ceramic)1, C0(ceramic)2, C0(ceramic)3, C0(ceramic)4, C0(radial), C0(radial)1, C0(radial)2, C0(radial)3, C0(radial)4, C1, C2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

Commit message: Phase 2
Parts:
- removed C43: 100n, symbol PCM_Elektuur:C
- removed D3: USBULC6-2M6, PCM_Package_TO_SOT_SMD_AKL:SOT-666, symbol PCM_Diode_TVS_AKL:USBLC6-2P6
- removed J7: USB_B_Micro, symbol Connector:USB_B_Micro
- added C54: 100n, symbol PCM_Elektuur:C
- added D13: USBULC6-2M6, PCM_Package_TO_SOT_SMD_AKL:SOT-666, symbol PCM_Diode_TVS_AKL:USBLC6-2P6
- added J11: Conn_01x02_Pin, symbol Connector:Conn_01x02_Pin
Connections:
- net GND: now also C54.2 (-), D13.2 (VN)
- net USB_N: now also D13.4 (L2)
- net USB_P: now also D13.6 (L1)
- net VBUS_5V: now reaches C53.2 (-), J1.77, J1.79, J1.81, J1.83, J1.85, J1.87, R37.2, U15.6 (VOUT)
- net VBUS_5V: now also C54.1 (+), D13.5 (VP)
- net at J6.2 (D-): now also D13.3 (L2)
- net at J6.3 (D+): now also D13.1 (L1)
- net +BATT: no longer names the net of C4.1 (+), L1.1, R20.1, U15.2 (EN), U15.3 (VIN), U2.3 (BAT)
- net +BATT: now also J11.1 (Pin_1)
- net -BATT: no longer names the net of C3.1, Q2.2, Q2.3, U3.6
- net -BATT: now also J11.2 (Pin_2)
- no-connect marks 75 -> 76
Other:
- moved on the sheet: C0(ceramic), C0(ceramic)1, C0(ceramic)2, C0(ceramic)3, C0(ceramic)4, C0(radial), C0(radial)1, C0(radial)2, C0(radial)3, C0(radial)4, C1, C2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
