File: 490_0/490_0.kicad_sch (KiCad schematic)
At the start: 200 parts, among them J1 DF40C-100DS-0.4V_51_, J10 Conn_01x02_Pin, J11 Conn_01x02_Pin, J2 DF40C-100DS-0.4V_51_, J3 Micro_SD_Card, J4 USB3_A_Stacked, J5 HDMI_D_1.4, J6 USB_B_Micro, J8 Conn_01x02_Pin, J9 Conn_01x02_Pin, Q0 NMOS, Q1 NMOS, Q2 FS8205A, Q3 NMOS, Q4 NMOS, Q5 NMOS, SW1 SW_DPST_x2, SW2 SW_Push0, SW3 SW_Push1, SW4 SW_Push2, SW5 SW_Push3, SW6 SW_Push4, U1 RT9742GGJ5, U10 PCA9685, U11 MAX98357A, U12 MAX98357A, U13 74HC4051, U15 TPS61023DRLR, U2 TP4057, U3 DW01, U4 TUSB7320RKMR, U5 ECMF04-4HSWM10, U6 ECMF04-4HSWM10, U7 TPS2560DRCR, U8 ECMF04-4HSWM10, U9 ECMF04-4HSWM10, X1 ECS-480-18-33-JGN-TR

Commit message: Small update
Parts:
- added C52, C53: 100n, symbol PCM_Elektuur:C
- added C55: 4.7u, symbol PCM_Elektuur:C
- added D12: USBULC6-2M6, PCM_Package_TO_SOT_SMD_AKL:SOT-666, symbol PCM_Diode_TVS_AKL:USBLC6-2P6
- added J1, J2: ArduCAM ToF Connector, symbol Connector_Generic:Conn_02x15_Counter_Clockwise
- renumbered C0(ceramic) to C0(ceramic)2, C0(ceramic)4 to C0(ceramic)3, C0(ceramic)2 to C0(ceramic)4, C0(ceramic)3 to C0(ceramic)5, C0(radial) to C0(radial)2, C0(radial)4 to C0(radial)3, C0(radial)2 to C0(radial)4, C0(radial)3 to C0(radial)5, C14 to C1, C29 to C10, C17 to C11, C28 to C12, C23 to C13, C11 to C14, C31 to C15, C18 to C16, C30 to C17, C24 to C18, C10 to C19, C25 to C2, C33 to C20, C19 to C21, C32 to C22, C38 to C23, C9 to C24, C35 to C25, C20 to C26, C34 to C27, C39 to C28, C8 to C29, C15 to C3, C37 to C30, C21 to C31, C36 to C32, C40 to C33, C7 to C34, C41 to C35, C42 to C36, C50 to C37, C52 to C38, C51 to C39, C22 to C4, C46 to C40, C44 to C41, C48 to C42, C45 to C43, C49 to C44, C47 to C45, C54 to C46, C2 to C47, C6 to C48, C5 to C49, C13 to C5, C5(ceramic) to C5(ceramic)1, C5(radial) to C5(radial)1, C4 to C50, C3 to C51, C53 to C54, C1 to C56, C27 to C6, C6(ceramic) to C6(ceramic)1, C6(radial) to C6(radial)1, C16 to C7, C26 to C8, C12 to C9, Cin to Cin1, Cx(ceramic) to Cx(ceramic)1, Cx(radial) to Cx(radial)1, D6 to D1, D12 to D10, D7 to D11, D1 to D13, D13 to D3, D8 to D4, D9 to D5, D10 to D6, D5 to D7, D4 to D8, D11 to D9, FB2 to FB3, J8 to J10, J5 to J12, J1 to J13, J3 to J14, J2 to J3, J6 to J4, J8 to J5, J9 to J6, J9 to J7, J4 to J8, J10 to J9, JP3 to JP1, JP6 to JP10, JP5 to JP11, JP4 to JP12, JP8 to JP2, JP9 to JP3, JP10 to JP4, JP11 to JP5, JP12 to JP6, JP2 to JP8, JP1 to JP9, LED3 to LED1, LED4 to LED2, Q3 to Q1, Q0 to Q2, Q5 to Q3, Q3 to Q4, Q4 to Q5, Q2 to Q6, Q1 to Q7, R19 to R1, R27 to R10, R26 to R11, R21 to R12, R22 to R13, R33 to R14, R32 to R15, R23 to R16, R18 to R17, R20 to R18, R37 to R19, R35 to R2, R38 to R20, R15 to R21, R16 to R22, R6 to R23, R17 to R24, R1 to R25, R2 to R26, R3 to R27, R4 to R28, R5 to R29, R34 to R3, R14 to R30, R29 to R31, R12 to R32, R13 to R33, R7 to R34, R8 to R35, R to R36, R9 to R37, R10 to R38, R11 to R39, R24 to R4, R to R40, R25 to R5, R31 to R6, R36 to R7, R28 to R8, R30 to R9, Rg0 to Rg2, Rg4 to Rg3, Rg2 to Rg4, Rg3 to Rg5, Rgd0 to Rgd2, Rgd4 to Rgd3, Rgd2 to Rgd4, Rgd3 to Rgd5, U4 to U1, U9 to U10, U13 to U11, U1 to U12, U11 to U13, U12 to U14, U7 to U2, U10 to U3, U5 to U4, U6 to U5, U2 to U6, U3 to U7, U15 to U8, U8 to U9
Connections:
- net + 5V: now also D11.5 (VP), C52.1 (+), C53.1 (+), D12.5 (VP)
- net CAM0_C_N: now also J1.8 (Pin_8), J2.8 (Pin_8)
- net CAM0_C_P: now also J1.9 (Pin_9), J2.9 (Pin_9)
- net CAM0_D0_N: now also J1.2 (Pin_2), J2.2 (Pin_2)
- net CAM0_D0_P: now also J1.3 (Pin_3), J2.3 (Pin_3)
- net CAM0_D1_N: now also J1.5 (Pin_5), J2.5 (Pin_5)
- net CAM0_D1_P: now also J1.6 (Pin_6), J2.6 (Pin_6)
- net Camera_GPIO: now also J1.11 (Pin_11), J2.11 (Pin_11)
- net GND: now also D11.2 (VN), J12.10 (D0S), J12.13 (CKS), J12.16 (GND), J12.4 (D2S), J12.7 (D1S), J12.SH, J8.16 (DRAIN2), J8.7 (DRAIN1), U10.3 (GND), U10.8 (GND), U9.3 (GND), U9.8 (GND), C52.2 (-), C53.2 (-), C55.2 (-), D12.2 (VN), J1.1 (Pin_1), J1.10 (Pin_10), J1.4 (Pin_4), J1.7 (Pin_7), J2.1 (Pin_1), J2.10 (Pin_10), J2.4 (Pin_4), J2.7 (Pin_7)
- net HDMI0_CEC: now also D12.1 (L1)
- net HDMI0_HOTPLUG: now also D12.3 (L2)
- net HDMI0_SCL: now also D11.3 (L2)
- net HDMI0_SDA: now also D11.1 (L1)
- net SCL0: now also J1.13 (Pin_13), J2.13 (Pin_13)
- net SDA0: now also J1.14 (Pin_14), J2.14 (Pin_14)
- net VBUS_5V: now also J12.19 (+5V), C55.1 (+)
- net D-: now reaches J8.14 (SSRX2-), U5.10 (Out_1+)
- net D+: now reaches J8.15 (SSRX2+), U5.9 (Out_1+)
- net at D11.4 (L2): now also J12.17 (SCL)
- net at D11.6 (L1): now also J12.18 (SDA)
- net at J12.1 (HPD/HEAC-): now also D12.4 (L2)
- net at J12.15 (CEC): now also D12.6 (L1)
- no-connect marks 76 -> 109
Other:
- note added: "The chip is designed if we dont have PWM"
- moved on the sheet: C5(ceramic)1, C5(radial)1, C6(ceramic)1, C6(radial)1, D11, FB2, FB3, J12, PD1, PU1, R36, R40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

Commit message: Changed charging circuit
Parts:
- removed C47: 10uF, PCM_SparkFun-Capacitor:C_0603_1608Metric, symbol PCM_SparkFun-Capacitor:10uF_0603_10V_20%
- removed C50, C54: ?, symbol PCM_Elektuur:C
- removed C51: 0.1uF, PCM_SparkFun-Capacitor:C_0402_1005Metric, symbol PCM_SparkFun-Capacitor:0.1uF_0402_16V_10%
- removed J11: Conn_01x02_Pin, symbol Connector:Conn_01x02_Pin
- removed J4: USB_B_Micro, symbol Connector:USB_B_Micro
- removed L1: 1u, WE-MAPI_4030:WE-MAPI_4030, symbol capstone_parts:74438357010
- removed LED1: LED_1.8mm_Red, PCM_LED_THT_AKL:LED_D1.8mm_W3.3mm_H2.4mm, symbol PCM_LED_AKL:LED_1.8mm_Red
- removed LED2: LED_1.8mm_SMD_Green, PCM_LED_SMD_AKL:LED_1.8mm_GullWing, symbol PCM_LED_AKL:LED_1.8mm_SMD_Green
- removed Q6: FS8205A, FS8205A:SOP65P640X120-8N, symbol FS8205A:FS8205A
- removed R12, R13: 1k, Resistor_THT:R_Axial_DIN0207_L6.3mm_D2.5mm_P10.16mm_Horizontal, symbol PCM_SL_Resistors:1k
- removed R16, R17: 2k_0603, 4ms_Resistor:R_0603, symbol PCM_4ms_Resistor:2k_0603
- removed R18: 100ohm, Resistor_THT:R_Axial_DIN0207_L6.3mm_D2.5mm_P10.16mm_Horizontal, symbol PCM_SL_Resistors:100ohm
- removed R19, R20: ?, Resistor_THT:R_Axial_DIN0207_L6.3mm_D2.5mm_P10.16mm_Horizontal, symbol PCM_SL_Resistors:100ohm
- removed U6: TP4057, Package_TO_SOT_SMD:TSOT-23-6, symbol Battery_Management:TP4057
- removed U7: DW01, DW01:SOT23-6, symbol capstone_parts:DW01
- removed U8: TPS61023DRLR, DRL0006A, symbol capstone_parts:TPS61023DRLR
- added C57: 100n, symbol PCM_Elektuur:C
- added C58: 10uF, PCM_SparkFun-Capacitor:C_0603_1608Metric, symbol PCM_SparkFun-Capacitor:10uF_0603_10V_20%
- added C59, C61: ?, symbol PCM_Elektuur:C
- added C60: 0.1uF, PCM_SparkFun-Capacitor:C_0402_1005Metric, symbol PCM_SparkFun-Capacitor:0.1uF_0402_16V_10%
- added C62: 22u, symbol PCM_Elektuur:C
- added C63, C67: 0.1u, symbol PCM_Elektuur:C
- added C64, C65, C66, C68: TBD, symbol PCM_Elektuur:C
- added D14: USBULC6-2M6, PCM_Package_TO_SOT_SMD_AKL:SOT-666, symbol PCM_Diode_TVS_AKL:USBLC6-2P6
- added D15, D16, D17, D18, D19: LED, symbol Device:LED
- added J15: USB_B_Micro, symbol Connector:USB_B_Micro
- added J16: Conn_01x02_Pin, symbol Connector:Conn_01x02_Pin
- added J17: Conn_01x03_Pin, symbol Connector:Conn_01x03_Pin
- added JP13: SolderJumper_3_Open, symbol Jumper:SolderJumper_3_Open
- added L2: 1u, WE-MAPI_4030:WE-MAPI_4030, symbol capstone_parts:74438357010
- added L3: 2.2uH, PCM_SparkFun-Coil:0806, symbol PCM_SparkFun-Coil:2.2uH_0806_1.2A
- added LED3: LED_1.8mm_Red, PCM_LED_THT_AKL:LED_D1.8mm_W3.3mm_H2.4mm, symbol PCM_LED_AKL:LED_1.8mm_Red
- added LED4: LED_1.8mm_SMD_Green, PCM_LED_SMD_AKL:LED_1.8mm_GullWing, symbol PCM_LED_AKL:LED_1.8mm_SMD_Green
- added P1: USB_C_Plug_USB2.0, symbol Connector:USB_C_Plug_USB2.0
- added Q8: FS8205A, FS8205A:SOP65P640X120-8N, symbol FS8205A:FS8205A
- added R41, R42: 1k, Resistor_THT:R_Axial_DIN0207_L6.3mm_D2.5mm_P10.16mm_Horizontal, symbol PCM_SL_Resistors:1k
- added R43, R44: 2k_0603, 4ms_Resistor:R_0603, symbol PCM_4ms_Resistor:2k_0603
- added R45: 100ohm, Resistor_THT:R_Axial_DIN0207_L6.3mm_D2.5mm_P10.16mm_Horizontal, symbol PCM_SL_Resistors:100ohm
- added R46, R47: ?, Resistor_THT:R_Axial_DIN0207_L6.3mm_D2.5mm_P10.16mm_Horizontal, symbol PCM_SL_Resistors:100ohm
- added R48: 5.1k, symbol Device:R
- added R49, R50, R53, R54, R55, R56, R57, R58, R59: TBD, symbol Device:R
- added R51: 49.9k, symbol Device:R
- added R52: 10m, symbol Device:R
- added SW7: SW_Push, symbol Switch:SW_Push
- added U15: MP2632BGR-Z, IC26_MP2632BGR-Z_MNP, symbol capstone_parts:MP2632BGR-Z
- added U16: TP4057, Package_TO_SOT_SMD:TSOT-23-6, symbol Battery_Management:TP4057
- added U17: DW01, DW01:SOT23-6, symbol capstone_parts:DW01
- added U18: TPS61023DRLR, DRL0006A, symbol capstone_parts:TPS61023DRLR
Connections:
- net GND: now also C57.2 (-), C58.2, C59.2 (-), C61.1 (+), C62.2 (-), C63.2 (-), C64.2 (-), C65.2 (-), C66.2 (-), C67.2 (-), C68.2 (-), D14.2 (VN), J15.5 (GND), J17.2 (Pin_2), JP13.3 (B), P1.A1 (GND), P1.A12 (GND), P1.B1 (GND), P1.B12 (GND), Q8.6, Q8.7, R43.2, R44.2, R47.1, R48.1, R49.1, R50.1, R51.1, R53.1, SW7.2, U15.1 (PGND), U15.17 (AGND), U16.2 (GND), U18.4 (GND)
- net USB_N: now also D14.4 (L2), U15.10 (DM2); no longer D3.4 (L2)
- net USB_P: now also D14.6 (L1), U15.11 (DP2); no longer D3.6 (L1)
- net VBUS_5V: now also C57.1 (+), C65.1 (+), C66.1 (+), D14.5 (VP), R56.1, R57.1, R58.1, R59.1, U15.3 (SYS), U15.4 (SYS); no longer C46.1 (+), D3.5 (VP)
- net at D3.3 (L2): now also P1.A6 (D+)
- net at D3.1 (L1): now also P1.A7 (D-)
- new net: C60.1, J16.2 (Pin_2), Q8.2, Q8.3, U17.6
- new net: C60.2, R45.2, U17.5
- new net: C58.1, J15.1 (VBUS), LED3.2 (A), LED4.2 (A), U16.4 (V_{CC})
- new net: D16.2 (A), R56.2
- new net: C46.1 (+), C62.1 (+), D3.5 (VP), P1.A4 (VBUS), P1.A9 (VBUS), P1.B4 (VBUS), P1.B9 (VBUS), U15.5 (VIN)
- new net: LED4.1 (K), R42.1
- new net: LED3.1 (K), R41.1
- new net: R41.2, U16.1 (~{CHRG})
- new net: C59.1 (+), J16.1 (Pin_1), L2.1, R45.1, U16.3 (BAT), U18.2 (EN), U18.3 (VIN)
- new net: L2.2, U18.5 (SW)
- new net: R46.1, R47.2, U18.1 (FB)
- new net: D17.1 (K), U15.25 (LED2)
- new net: D17.2 (A), R57.2
- new net: D19.1 (K), U15.23 (LED4)
- new net: D19.2 (A), R59.2
- new net: C61.2 (-), R46.2, U18.6 (VOUT)
- new net: J17.1 (Pin_1), R53.2, R54.1, U15.19 (NTC)
- new net: R42.2, U16.5 (STDBY)
- new net: R43.1, U16.6 (PROG)
- new net: C67.1 (+), SW7.1, U15.12 (PB)
- new net: D18.1 (K), U15.24 (LED3)
- new net: D18.2 (A), R58.2
- new net: D15.1 (K), U15.8 (TC)
- new net: D15.2 (A), R55.2
- new net: C63.1 (+), U15.13 (TMR)
- new net: L3.1, U15.2 (SW)
- new net: L3.2, R52.2, U15.22 (CSP)
- new net: R50.2, U15.14 (ISET)
- new net: R51.2, U15.15 (OLIM)
- new net: C68.1 (+), JP13.1 (A), U15.16 (VCC)
- new net: R54.2, U15.18 (VNTC)
- new net: JP13.2 (C), U15.20 (VB)
- new net: D16.1 (K), U15.26 (LED1)
- new net: R49.2, U15.9 (ILIM)
- new net: D14.1 (L1), J15.3 (D+)
- new net: D14.3 (L2), J15.2 (D-)
- new net: P1.A5 (CC), R48.2
- new net: Q8.1, Q8.8
- new net: Q8.4, U17.1
- new net: Q8.5, U17.3
- new net: R44.1, U17.2
- new net USB1_N: D3.6 (L1), U15.6 (DM1)
- new net USB1_P: D3.4 (L2), U15.7 (DP1)
- new net VBATT: C64.1 (+), J17.3 (Pin_3), R52.1, R55.1, U15.21 (BATT)
- no-connect marks 109 -> 112
Other:
- note added: "^For Charge current"
- moved on the sheet: C46, D3
