File: 490_0/_autosave-490_0.kicad_sch (KiCad schematic)
At the start: 250 parts, among them J1 ArduCAM ToF Connector, J10 Conn_01x02_Pin, J12 HDMI_D_1.4, J13 DF40C-100DS-0.4V_51_, J14 Micro_SD_Card, J15 USB_B_Micro, J16 Conn_01x02_Pin, J17 Conn_01x03_Pin, J2 ArduCAM ToF Connector, J3 DF40C-100DS-0.4V_51_, J5 Conn_01x02_Pin, J6 Conn_01x02_Pin, J7 Conn_01x02_Pin, J8 USB3_A_Stacked, J9 Conn_01x02_Pin, P1 USB_C_Plug_USB2.0, Q1 NMOS, Q2 NMOS, Q3 NMOS, Q4 NMOS, Q5 NMOS, Q7 NMOS, Q8 FS8205A, SW1 SW_DPST_x2, SW2 SW_Push0, SW3 SW_Push1, SW4 SW_Push2, SW5 SW_Push3, SW6 SW_Push4, SW7 SW_Push, U1 TUSB7320RKMR, U10 ECMF04-4HSWM10, U11 74HC4051, U12 RT9742GGJ5, U13 MAX98357A, U14 MAX98357A, U15 MP2632BGR-Z, U16 TP4057, U17 DW01, U18 TPS61023DRLR, U2 TPS2560DRCR, U3 PCA9685, U4 ECMF04-4HSWM10, U5 ECMF04-4HSWM10, U6 BD9G401EFJ, U9 ECMF04-4HSWM10, X1 ECS-480-18-33-JGN-TR

Commit message: Finished USB C charger (3.3 and 5V)
Added buck converter after the charging IC for 3.3 and 5V outputs.
Parts:
- C57, C58, C59, C60, C61, D14, J15, J16, L2, LED3, LED4, Q8, R41, R42, R43, R44, R45, R46, R47, U16, U17, U18: now not fitted; now left out of the parts list
- R12: value TBD -> 110k
- R13: value TBD -> 43k
- R16: value TBD -> 510k
- R17: value TBD -> 270k
Other:
- moved on the sheet: C46, C47, C5(ceramic)1, C5(radial)1, C50, C51, C54, C56, C6(ceramic)1, C6(radial)1, C62, C63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
