File: 490_0/pci_bridge.kicad_sch (KiCad schematic)
At the start: 36 parts, among them U8 TUSB7320RKMR

Commit message: US letter format
Changed lines of the file:
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@@
 	(generator "eeschema")
 	(generator_version "9.0")
-	(paper "A4")
+	(paper "USLetter")
 	(junction
 		(at 130.81 90.17)
@@
 	)
 	(sheet
-		(at 16.51 165.1)
-		(size 157.48 27.94)
+		(at 20.32 170.18)
+		(size 124.46 27.94)
 		(exclude_from_sim no)
 		(in_bom yes)
@@
 		)
 		(property "Sheetname" "IC of the Power Module"
-			(at 16.51 164.3884 0)
+			(at 20.32 169.4684 0)
 			(effects
 				(font
@@
 		)
 		(property "Sheetfile" "power_ic.kicad_sch"
-			(at 16.51 193.6246 0)
+			(at 20.32 198.7046 0)
 			(effects
 				(font

Commit message: Minor updates
Parts:
- renumbered C81 to C17, C86 to C18, C91 to C19, C96 to C20, C101 to C21, C69 to C22, C73 to C23, C77 to C24, C82 to C25, C87 to C26, C92 to C27, C97 to C28, C102 to C29, C70 to C30, C74 to C31, C78 to C32, C83 to C33, C88 to C34, C93 to C35, C98 to C36, C71 to C37, C75 to C38, C79 to C39, C84 to C40, C89 to C41, C94 to C42, C99 to C43, C72 to C44, C76 to C45, C80 to C46, C85 to C47, C90 to C48, C95 to C49, C100 to C50, FB4 to FB1, U8 to U7
