File: 490_0/power_ic.kicad_sch (KiCad schematic)
At the start: 35 parts, among them J11 USB3_A_Stacked, U11 TPS2560DRCR, U19 ECMF04-4HSWM10, U20 ECMF04-4HSWM10, U3 TUSB7320RKMR, X2 ECS-480-18-33-JGN-TR

Commit message: Minor updates
Parts:
- renumbered C108 to C57, C115 to C58, C106 to C59, C107 to C60, C105 to C61, C111 to C62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
