File: 490_0/micro_sd.kicad_sch (KiCad schematic)
At the start: 5 parts, among them J26 Micro_SD_Card, U27 RT9742GGJ5

Commit message: Minor fixes
Parts:
- R107: value 12K 1% -> 5.1K 1%
Connections:
- net +3.3V: no longer R107.2
- net GND: now also R107.1
- net at U27.4 (EN): now also R107.2; no longer R107.1
Other:
- moved on the sheet: R107
Changed lines of the file:
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@@
+	(wire
+		(pts
+			(xy 74.93 99.06) (xy 74.93 102.87)
+		)
+		(stroke
+			(width 0)
+			(type default)
+		)
+	)
 	(wire
 		(pts
@@
 	(wire
 		(pts
-			(xy 74.93 93.98) (xy 74.93 99.06)
-		)
-		(stroke
-			(width 0)
-			(type default)
-		)
-	)
-	(wire
-		(pts
 			(xy 177.8 86.36) (xy 180.34 86.36)
 		)
@@
 	(wire
 		(pts
+			(xy 74.93 111.76) (xy 74.93 110.49)
+		)
+		(stroke
+			(width 0)
+			(type default)
+		)
+	)
+	(wire
+		(pts
 			(xy 121.92 91.44) (xy 121.92 95.25)
 		)
@@
 	(wire
 		(pts
-			(xy 74.93 85.09) (xy 74.93 86.36)
-		)
-		(stroke
-			(width 0)
-			(type default)
-		)
-	)
-	(wire
-		(pts
 			(xy 74.93 99.06) (xy 90.17 99.06)
 		)
@@
 		(pts
 			(xy 180.34 96.52) (xy 157.48 96.52)
-		)
-		(stroke
-			(width 0)
-			(type default)
-		)
-	)
-	(wire
-		(pts
-			(xy 74.93 85.09) (xy 83.82 85.09)
 		)
 		(stroke
@@
 	(symbol
 		(lib_id "Device:R")
-		(at 74.93 90.17 0)
+		(at 74.93 106.68 0)
 		(mirror x)
 		(unit 1)
@@
 		(fields_autoplaced yes)
 		(property "Reference" "R107"
-			(at 72.39 88.8999 0)
+			(at 72.39 105.4099 0)
 			(effects
 				(font
@@
 			)
 		)
-		(property "Value" "12K 1%"
-			(at 72.39 91.4399 0)
+		(property "Value" "5.1K 1%"
+			(at 72.39 107.9499 0)
 			(effects
 				(font
@@
 		)
 		(property "Footprint" ""
-			(at 73.152 90.17 90)
+			(at 73.152 106.68 90)
 			(effects
 				(font
@@
 		)
 		(property "Datasheet" "~"
-			(at 74.93 90.17 0)
+			(at 74.93 106.68 0)
 			(effects
 				(font
@@
 		)
 		(property "Description" "Resistor"
-			(at 74.93 90.17 0)
+			(at 74.93 106.68 0)
 			(effects
 				(font
@@
 					(unit 1)
 				)
+			)
+		)
+	)
+	(symbol
+		(lib_id "power:GND")
+		(at 74.93 111.76 0)
+		(mirror y)
+		(unit 1)
+		(exclude_from_sim no)
+		(in_bom yes)
+		(on_board yes)
+		(dnp no)
+		(fields_autoplaced yes)
+		(property "Reference" "#PWR027"
+			(at 74.93 118.11 0)
+			(effects
+				(font
+					(size 1.27 1.27)
+				)
+				(hide yes)
+			)
+		)
+		(property "Value" "GND"
+			(at 74.93 116.84 0)
+			(effects
+				(font
+					(size 1.27 1.27)
+				)
+			)
+		)
+		(property "Footprint" ""
+			(at 74.93 111.76 0)
+			(effects
+				(font
+					(size 1.27 1.27)
+				)
+				(hide yes)
+			)
+		)
+		(property "Datasheet" ""
+			(at 74.93 111.76 0)
+			(effects
+				(font
+					(size 1.27 1.27)
+				)
+				(hide yes)
+			)
+		)
+		(property "Description" "Power symbol creates a global label with name \"GND\" , ground"
+			(at 74.93 111.76 0)
+			(effects
+				(font
+					(size 1.27 1.27)
+				)
+				(hide yes)
+			)
+		)
+		(pin "1"
+		)
+		(instances
+			(project "490_0"
+				(path "/365a82ed-827d-43e1-aa2f-b98221c4179c/758ed409-e21d-4faf-b2fa-7f148daf6972"
+					(reference "#PWR027")
+					(unit 1)
+				)

Commit message: Minor updates
Parts:
- renumbered C131 to C56, Cin2 to Cin1, J26 to J16, R107 to R50, U27 to U11

Commit message: BOM + ESD replacement for HDMI
Started BOM and changed ESD chips that were obsolete. Also added 2 pin connectors
Parts:
- U11: Current - Load (none) -> 1A; Digikey Link (none) -> https://www.digikey.ca/en/products/detail/richtek-usa-inc/R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; Manufacturer (none) -> Richtek USA Inc.; Manufacturer Part (none) -> RT9742GGJ5; Package (none) -> TSOT-23-5; Price (none) -> 0.46; Supplier (none) -> DigiKey; Supplier P/N (none) -> 1028-1436-1-ND; Type (none) -> SMD; Unit (none) -> pcs; Voltage - Load (none) -> 2.7V ~ 6V
