File: 490_0/PCB1.kicad_sch (KiCad schematic)
At the start: 4 parts, among them J14 Conn_01x08, J15 Conn_01x11, J16 5051102291, J17 S2B-XH-A

Commit message: Updated the schematic
Parts:
- removed J14: Conn_01x08, symbol PCM_4ms_Connector:Conn_01x08
- removed J15: Conn_01x11, symbol Connector_Generic:Conn_01x11
- added J1: Conn_01x08, symbol PCM_4ms_Connector:Conn_01x08
Connections:
- net +3.3V: now also J1.2 (Pin_2)
- net +5V: now also J1.1 (Pin_1)
- net GND: now also J1.8 (Pin_8)
- net PCB1-Board Connector A/GPIO13: now also J1.5 (Pin_5)
- net PCB1-Charging and Power Port + USB switch/USBhub_N: now also J1.3 (Pin_3)
- net PCB1-Charging and Power Port + USB switch/USBhub_P: now also J1.4 (Pin_4)
- net SCL1: now also J1.7 (Pin_7)
- net SDA1: now also J1.6 (Pin_6)
Other:
- added sheet PCB1-Buttons (pushbuttons.kicad_sch)
- added sheet PCB1-Speakers and Connectors (speakers.kicad_sch)
- note removed: "Button Connector"
- note removed: "I2S_BCLK"
- note removed: "I2S_DIN"
- note removed: "I2S_LRCLK"

Commit message: Implemented Dmitry comments
Parts:
- removed J17: S2B-XH-A, 4ms_Connector:Pins_1x08_2.54mm_TH, symbol capstone_parts:S2B-XH-A
- added J10: S2B-XH-A, S2B-XH-A:JST_S2B-XH-A, symbol PCM_4ms_Connector:Conn_01x02
- renumbered J1 to J11, J16 to J12
Connections:
- net +5V: now also J10.2 (Pin_2)
- net GND: now also J10.1 (Pin_1)
Other:
- removed sheet PCB1-Buttons
- sheet PCB1-Board Connector A ports: added none; removed GPIO10, GPIO17, GPIO22, GPIO23, GPIO24, GPIO25

Commit message: Final Fixes
Parts:
- removed J12: 5051102291, CON_5051102291_MOL, symbol capstone_parts:5051102291
- added J12: 0522711579, symbol Connector_Generic:Conn_01x15
- renumbered J10 to J13
Connections:
- net +3.3V: now also J12.15 (Pin_15)
- net GND: now also J12.1 (Pin_1), J12.10 (Pin_10), J12.4 (Pin_4), J12.7 (Pin_7)
- net PCB1-Board Connector A/CAM1_C_N: now also J12.8 (Pin_8)
- net PCB1-Board Connector A/CAM1_C_P: now also J12.9 (Pin_9)
- net PCB1-Board Connector A/CAM1_D0_N: now also J12.2 (Pin_2)
- net PCB1-Board Connector A/CAM1_D0_P: now also J12.3 (Pin_3)
- net PCB1-Board Connector A/CAM1_D1_N: now also J12.5 (Pin_5)
- net PCB1-Board Connector A/CAM1_D1_P: now also J12.6 (Pin_6)
- net PCB1-Board Connector A/Camera_GPIO: now also J12.11 (Pin_11)
- net SCL1: now also J12.13 (Pin_13)
- net SDA1: now also J12.14 (Pin_14)
Other:
- sheet PCB1-Board Connector A ports: added none; removed CAM1_D2_N, CAM1_D2_P, CAM1_D3_N, CAM1_D3_P
- note added: "Camera CSI Connector 0.5mm pitch, 15-pin FFC"
- note removed: "Camera CSI Connector 0.5mm pitch, 22-pin FFC"

Commit message: update
Parts:
- J13: value S2B-XH-A -> S2B-ZR; Digikey Link https://www.digikey.ca/en/products/detail/jst-sales-america-inc/S2B-XH-A/1651055 -> https://www.digikey.ca/en/products/detail/jst-sales-america-inc/s2b-zr/926576; Manufacturer Part S2B-XH-A -> S2B-ZR; Price 0.12 -> 0.11; Supplier P/N 455-S2B-XH-A-ND -> 455-1669-ND
Other:
- note added: "in config.txt: dtoverlay=arducam-pivariety,i2c_bus=1 - i2c_bus=1: Don't look at the camera port (I2C0), look at the user header pins (I2C1)."
Changed lines of the file:
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@@
+		)
+	)
+	(text "in config.txt:\ndtoverlay=arducam-pivariety,i2c_bus=1\n- i2c_bus=1: Don't look at the camera port (I2C0), look at the user header pins (I2C1)."
+		(exclude_from_sim no)
+		(at 66.802 118.872 0)
+		(effects
+			(font
+				(size 0.635 0.635)
+			)
+			(justify left)
 		)
 	)
@@
 			)
 		)
-		(property "Value" "S2B-XH-A"
+		(property "Value" "S2B-ZR"
 			(at 65.278 144.272 0)
 			(effects
@@
 			)
 		)
-		(property "Datasheet" "kicad-embed://B2B-XH-A 2 pin connector.pdf"
+		(property "Datasheet" "kicad-embed://eZH.pdf"
 			(at 68.58 139.7 0)
 			(effects
@@
 			)
 		)
-		(property "Description" "CONN HEADER R/A 2POS 2.5MM"
+		(property "Description" "CONN HEADER R/A 2POS 1.5MM"
 			(at 68.58 139.7 0)
 			(effects
@@
 			)
 		)
-		(property "Digikey Link" "https://www.digikey.ca/en/products/detail/jst-sales-america-inc/S2B-XH-A/1651055"
+		(property "Digikey Link" "https://www.digikey.ca/en/products/detail/jst-sales-america-inc/s2b-zr/926576"
 			(at 68.58 139.7 0)
 			(effects
@@
 			)
 		)
-		(property "Manufacturer Part" "S2B-XH-A"
+		(property "Manufacturer Part" "S2B-ZR"
 			(at 68.58 139.7 0)
 			(effects
@@
 			)
 		)
-		(property "Price" "0.12"
+		(property "Price" "0.11"
 			(at 68.58 139.7 0)
 			(effects
@@
 			)
 		)
-		(property "Supplier P/N" "455-S2B-XH-A-ND"
+		(property "Supplier P/N" "455-1669-ND"
 			(at 68.58 139.7 0)
 			(effects
