File: 490_0/charging_power.kicad_sch (KiCad schematic)
At the start: 46 parts, among them J1 S2B-XH-A, SW7 TL2230EEF140, U7 TPS566247DRLR, U8 MP2639AGR-Z

Commit message: Final Fixes
Parts:
- added C33: 10u, symbol PCM_Elektuur:C
- R24: renamed from R36; value 34.8k -> 30.1k; Digikey Link https://www.digikey.ca/en/products/detail/yageo/RC1206FR-0734K8L/728829 -> https://www.digikey.ca/en/products/detail/yageo/RC1206FR-0730K1L/728801; Manufacturer Part RC1206FR-0734K8L -> RC1206FR-0730K1L; Supplier P/N 311-34.8KFRCT-ND -> 311-30.1KFRCT-ND
- R35: renamed from R49; value 118k -> 120k; Digikey Link https://www.digikey.ca/en/products/detail/yageo/RC1206FR-07118KL/728514 -> https://www.digikey.ca/en/products/detail/yageo/RC1206FR-07120KL/728524; Manufacturer Part RC1206FR-07118KL -> RC1206FR-07120KL; Supplier P/N 311-118KFRCT-ND -> 311-120KFRCT-ND
- renumbered C38 to C32, C39 to C34, C40 to C35, C41 to C36, C42 to C37, C43 to C38, C44 to C39, C45 to C40, C46 to C41, C47 to C42, C48 to C43, C49 to C44, C50 to C45, C51 to C46, C52 to C47, C53 to C48, C54 to C49, J1 to J15, R34 to R22, R35 to R23, R37 to R25, R40 to R26, R42 to R27, R43 to R28, R9 to R29, R44 to R30, R45 to R31, R46 to R32, R47 to R33, R48 to R34, R50 to R36, SW7 to SW1
Connections:
- net +VBATT_7V4: now also C33.2 (-)
- net GND: now also C33.1 (+)
Other:
- note added: "Charge Current - ISET - 215 kΩ = 1A Input Limit - ILIM - 120 kΩ = 1.77A (slightly below 1.8A Limit from micro USB) Discharge Limit - OLIM - NA (only charging)"
- note removed: "Charge Current - ISET - 215 kΩ = 1A Input Limit - ILIM - 118 kΩ = 1.8A Limit from micro USB Discharge Limit - OLIM - NA (only charging)"
- moved on the sheet: C32, C34

Commit message: Implemented Dmitry recommendations
Parts:
- added C55: 0.1u, symbol PCM_Elektuur:C
- added J20: YO0201500000G, 4ms_Connector:Pins_1x02_2.54mm_TH, symbol PCM_4ms_Connector:Conn_01x02
- added R10: 10k, symbol Device:R
- added R8: 76.8k, Resistor_THT:R_Axial_DIN0207_L6.3mm_D2.5mm_P10.16mm_Horizontal, symbol PCM_SL_Resistors:0ohm
- added R9: 24.3k, Resistor_THT:R_Axial_DIN0207_L6.3mm_D2.5mm_P10.16mm_Horizontal, symbol PCM_SL_Resistors:0ohm
- added SW8: TL1105LF160Q, symbol Switch:SW_Push
- C35: Digikey Link https://www.digikey.ca/en/products/detail/yageo/CC0603KRX7R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 -> https://www.digikey.ca/en/products/detail/yageo/CC0805KRX7R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; Manufacturer Part CC0603KRX7R9BB104 -> CC0805KRX7R9BB104; Package 0603 (1608 Metric) -> 0805 (2012 Metric); Supplier P/N 311-1344-1-ND -> 311-1140-1-ND
- C36: Digikey Link https://www.digikey.ca/en/products/detail/kemet/c0603c330j5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 -> https://www.digikey.ca/en/products/detail/kemet/C0805C330J5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; Manufacturer Part 399-C0603C330J5GACTUCT-ND -> C0805C330J5GACTU; Package 0603 -> 0805; Price 0.12 -> 0.1; Supplier P/N 399-C0603C330J5GACTUCT-ND -> 399-C0805C330J5GACTUCT-ND
- J15: value S2B-XH-A -> S3B-XH-A; footprint S2B-XH-A:JST_S2B-XH-A -> 4ms_Connector:Pins_1x03_2.54mm_TH_AudioInsRGndL; symbol PCM_4ms_Connector:Conn_01x02 -> PCM_4ms_Connector:Conn_01x03; Digikey Link https://www.digikey.ca/en/products/detail/jst-sales-america-inc/S2B-XH-A/1651055 -> https://www.digikey.ca/en/products/detail/jst-sales-america-inc/S3B-XH-A/1651048; Manufacturer Part S2B-XH-A -> S3B-XH-A; Part Number 1-0201FBV0T -> 1-0301FBV0T; Price 0.12 -> 0.15; Specifications Pins_01x02, Header, Male Pins, 1*2, spacing 2.54mm, straigh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 -> HEADER 1x3 MALE PINS 0.100” 180deg; Supplier P/N 455-S2B-XH-A-ND -> 455-S3B-XH-A-ND
- NT1, TP1: now in the parts list
Connections:
- net +VBATT_7V4: now also J20.1 (Pin_1); no longer C43.1 (+), C44.2 (-), J15.2 (Pin_2), U8.3 (VH)
- net AGND: now also C55.1 (+); no longer R28.1, R30.1, R31.1, R33.1, R34.1, U8.17 (FB)
- net GND: now also J20.2 (Pin_2), R9.1, SW8.1; no longer U8.12 (MID)
- net VBUS_5V: now also R8.2
- net at TP1.1: now also C55.2 (-), R10.2; no longer U8.21 (IB)
- net at R26.2, U8.19 (VNTC): now also R28.1, R30.1, R31.1, R33.1, R34.1
- net at U8.7 (PB): now also SW8.2
- new net: J15.2 (Pin_2), U8.12 (MID)
- new net: C43.1 (+), C44.2 (-), J15.3 (Pin_3), U8.3 (VH)
- new net: R10.1, U8.21 (IB)
- new net: R8.1, R9.2, U8.17 (FB)
- no-connect marks 3 -> 2
Other:
- note removed: "BATTERY HAS BUILT IN BMS"
- moved on the sheet: TP1

Commit message: Implemented suggestions
notes on schematics:
Overall: Schematics needs to be improved, more compact and cleaner
=========================
I) on root page (page 1):
overall: needs a bit of clean up of the diagram

1. the diagram shows pcb3 and pcb1, but no pcb2, it is probably outdated and therefore might have errors in it, fix it to the latest version and rename things to reflect what it actually is. Also try to clean it up a bit
2. The PCB-3 seem to have the cameras directly connected to the usb hub, how will this be connected? with connectors? if so add them to the diagram, if it's with wires soldered directly to the pcb, try to make note of it for clarity
4. for some reason your TOF is above PCB-3 but is only connected to PCB1, will the TOF be on the glasses, or will you be moving this to the main board? maybe have TOF on the chest for depth, and 2 cameras on glasses for vision, it will also reduce length of cable, which is ideal, i don't think it will work if you run it from the glasses to pcb1 though.
I know, this is a problem, we discussed the chest thing, the problem is the length of the cable but also the haptic feedback is weird if they turn their head.
5. Rename PCB1/PCB3 to PCB1 (chest) PCB3 (glasses) for clarity. Also i don't think (mayeb i'm wrong) that the 5 conected buttons should be on a bus, a bus implies that multiple devices communicate on the same single line. You're using individual lines for each to individual gpio, no?

=========================
II) on PCB-3 usb 2.0 bridge page (page 10)
overall: check datasheet and make sure you've done the connection right and values are selected properly, with the chip data lines properly pulled up/down whether externally or internally. This is important

1. C3/C11 are the input capacitors to U2/u3 TPS553DBVR, datasheet says 100nF, you used 10uF, why? stick to 100nF
2. you seem to have implemented one of /Uthe typical application circuit, look at the others. You have on page 21 of datasheet an auto-retry wi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
Parts:
- added C5: 0.1u, symbol PCM_Elektuur:C
- added R2: 215k, symbol Device:R
Connections:
- net GND: now also C5.1 (+), R2.1; no longer U8.22 (OLIM)
- net at SW8.2, U8.7 (PB): now also C5.2 (-)
- net AGND renamed GNDA
- new net: R2.2, U8.22 (OLIM)
Other:
- moved on the sheet: SW8

Commit message: FFC to HDMI change
Parts:
- NT1, TP1: now left out of the parts list
Changed lines of the file:
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@@
 		(unit 1)
 		(exclude_from_sim no)
-		(in_bom yes)
+		(in_bom no)
 		(on_board yes)
 		(dnp no)
@@
 		(unit 1)
 		(exclude_from_sim no)
-		(in_bom yes)
+		(in_bom no)
 		(on_board yes)
 		(dnp no)

Commit message: Footprint Update
1st half of footprints updated
Parts:
- D11, D12, D13, D14, D15: footprint (none) -> LED_SMD:LED_0805_2012Metric
- J15: footprint 4ms_Connector:Pins_1x03_2.54mm_TH_AudioInsRGndL -> Connector_JST:JST_XH_S3B-XH-A_1x03_P2.50mm_Horizontal
- J20: footprint 4ms_Connector:Pins_1x02_2.54mm_TH -> Connector_PinHeader_2.54mm:PinHeader_1x02_P2.54mm_Vertical
- L1, L2: footprint (none) -> *CapStone*:IND_SRP6540-2R2M_BRN
- U7: footprint SOT-5X3-6_DRL_TEX -> (none)
Changed lines of the file:
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@@
 			)
 		)
-		(property "Footprint" ""
+		(property "Footprint" "LED_SMD:LED_0805_2012Metric"
 			(at 135.89 132.08 0)
 			(effects
@@
 			)
 		)
-		(property "Footprint" ""
+		(property "Footprint" "LED_SMD:LED_0805_2012Metric"
 			(at 130.81 127 0)
 			(effects
@@
 			)
 		)
-		(property "Footprint" ""
+		(property "Footprint" "*CapStone*:IND_SRP6540-2R2M_BRN"
 			(at 142.24 90.17 0)
 			(effects
@@
 			)
 		)
-		(property "Footprint" "4ms_Connector:Pins_1x03_2.54mm_TH_AudioInsRGndL"
+		(property "Footprint" "Connector_JST:JST_XH_S3B-XH-A_1x03_P2.50mm_Horizontal"
 			(at 228.6 106.045 0)
 			(effects
@@
 			)
 		)
-		(property "Footprint" ""
+		(property "Footprint" "LED_SMD:LED_0805_2012Metric"
 			(at 123.19 121.92 0)
 			(effects
@@
 			)
 		)
-		(property "Footprint" "4ms_Connector:Pins_1x02_2.54mm_TH"
+		(property "Footprint" "Connector_PinHeader_2.54mm:PinHeader_1x02_P2.54mm_Vertical"
 			(at 227.965 71.755 0)
 			(effects
@@
 			)
 		)
-		(property "Footprint" "SOT-5X3-6_DRL_TEX"
+		(property "Footprint" ""
 			(at 83.82 25.4 0)
 			(effects
@@
 			)
 		)
-		(property "Footprint" ""
+		(property "Footprint" "LED_SMD:LED_0805_2012Metric"
 			(at 152.4 142.24 0)
 			(effects
@@
 			)
 		)
-		(property "Footprint" ""
+		(property "Footprint" "LED_SMD:LED_0805_2012Metric"
 			(at 143.51 137.16 0)
 			(effects
@@
 			)
 		)
-		(property "Footprint" ""
+		(property "Footprint" "*CapStone*:IND_SRP6540-2R2M_BRN"
 			(at 137.16 31.75 0)
 			(effects
