File: 490_0/charging_power.kicad_sch (KiCad schematic)
At the start: 55 parts, among them J15 S3B-XH-A, J20 YO0201500000G, SW1 TL2230EEF140, SW8 TL1105LF160Q, U7 TPS566247DRLR, U8 MP2639AGR-Z

Commit message: Footprint Update #2
All footprints except for the capacitors have been attributed
Parts:
- NT1: footprint (none) -> NetTie:NetTie-2_SMD_Pad2.0mm
- R10, R2, R22, R23, R24, R25, R26, R27, R28, R29, R30, R31, R32, R33, R34, R35, R36: footprint (none) -> Resistor_SMD:R_0603_1608Metric
- SW1: footprint (none) -> *CapStone*:SW_TL2230EEF140
- SW8: footprint (none) -> *CapStone*:SW_TL1105LF160Q
- TP1: footprint (none) -> TestPoint:TestPoint_Pad_D2.0mm
- U7: footprint (none) -> *CapStone*:SOT-5X3-6_DRL_TEX
- U8: footprint (none) -> *CapStone*:IC26_MP2632BGR-Z_MNP
Changed lines of the file:
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@@
 			)
 		)
-		(property "Footprint" ""
+		(property "Footprint" "Resistor_SMD:R_0603_1608Metric"
 			(at 125.73 173.482 90)
 			(effects
@@
 			)
 		)
-		(property "Footprint" ""
+		(property "Footprint" "TestPoint:TestPoint_Pad_D2.0mm"
 			(at 15.24 162.56 0)
 			(effects
@@
 			)
 		)
-		(property "Footprint" ""
+		(property "Footprint" "Resistor_SMD:R_0603_1608Metric"
 			(at 166.878 31.75 90)
 			(effects
@@
 			)
 		)
-		(property "Footprint" ""
+		(property "Footprint" "Resistor_SMD:R_0603_1608Metric"
 			(at 64.77 164.338 90)
 			(effects
@@
 			)
 		)
-		(property "Footprint" ""
+		(property "Footprint" "Resistor_SMD:R_0603_1608Metric"
 			(at 187.198 125.73 90)
 			(effects
@@
 			)
 		)
-		(property "Footprint" ""
+		(property "Footprint" "Resistor_SMD:R_0603_1608Metric"
 			(at 153.67 130.302 90)
 			(effects
@@
 			)
 		)
-		(property "Footprint" ""
+		(property "Footprint" "*CapStone*:IC26_MP2632BGR-Z_MNP"
 			(at 78.74 91.44 0)
 			(effects
@@
 			)
 		)
-		(property "Footprint" ""
+		(property "Footprint" "Resistor_SMD:R_0603_1608Metric"
 			(at 161.29 135.382 90)
 			(effects
@@
 			)
 		)
-		(property "Footprint" ""
+		(property "Footprint" "Resistor_SMD:R_0603_1608Metric"
 			(at 138.43 120.142 90)
 			(effects
@@
 			)
 		)
-		(property "Footprint" ""
+		(property "Footprint" "*CapStone*:SW_TL1105LF160Q"
 			(at 58.42 165.1 0)
 			(effects
@@
 			)
 		)
-		(property "Footprint" ""
+		(property "Footprint" "Resistor_SMD:R_0603_1608Metric"
 			(at 24.13 136.398 90)
 			(effects
@@
 			)
 		)
-		(property "Footprint" ""
+		(property "Footprint" "*CapStone*:SOT-5X3-6_DRL_TEX"
 			(at 83.82 25.4 0)
 			(effects
@@
 			)
 		)
-		(property "Footprint" ""
+		(property "Footprint" "*CapStone*:SW_TL2230EEF140"
 			(at 66.04 33.02 0)
 			(effects
@@
 			)
 		)
-		(property "Footprint" ""
+		(property "Footprint" "NetTie:NetTie-2_SMD_Pad2.0mm"
 			(at 127 193.04 0)
 			(effects
@@
 			)
 		)
-		(property "Footprint" ""
+		(property "Footprint" "Resistor_SMD:R_0603_1608Metric"
 			(at 74.422 49.53 90)
 			(effects
@@
 			)
 		)
-		(property "Footprint" ""
+		(property "Footprint" "Resistor_SMD:R_0603_1608Metric"
 			(at 125.73 168.402 90)
 			(effects
@@
 			)
 		)
-		(property "Footprint" ""
+		(property "Footprint" "Resistor_SMD:R_0603_1608Metric"
 			(at 187.198 113.03 90)
 			(effects
@@
 			)
 		)
-		(property "Footprint" ""
+		(property "Footprint" "Resistor_SMD:R_0603_1608Metric"
 			(at 168.91 140.462 90)
 			(effects
@@
 			)
 		)
-		(property "Footprint" ""
+		(property "Footprint" "Resistor_SMD:R_0603_1608Metric"
 			(at 146.05 125.222 90)
 			(effects
@@
 			)
 		)
-		(property "Footprint" ""
+		(property "Footprint" "Resistor_SMD:R_0603_1608Metric"
 			(at 166.878 49.53 90)
 			(effects
@@
 			)
 		)
-		(property "Footprint" ""
+		(property "Footprint" "Resistor_SMD:R_0603_1608Metric"
 			(at 125.73 163.322 90)
 			(effects
@@
 			)
 		)
-		(property "Footprint" ""
+		(property "Footprint" "Resistor_SMD:R_0603_1608Metric"
 			(at 74.422 36.83 90)
 			(effects
@@
 			)
 		)
-		(property "Footprint" ""
+		(property "Footprint" "Resistor_SMD:R_0603_1608Metric"
 			(at 32.258 118.11 90)
 			(effects

Commit message: March 3rd
Parts:
- C32, C33, C34: footprint (none) -> Capacitor_SMD:C_1206_3216Metric
- C35: footprint (none) -> Capacitor_SMD:C_0603_1608Metric; Digikey Link https://www.digikey.ca/en/products/detail/yageo/CC0805KRX7R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 -> https://www.digikey.ca/en/products/detail/yageo/CC0603KRX7R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; Manufacturer Part CC0805KRX7R9BB104 -> CC0603KRX7R9BB104; Package 0805 (2012 Metric) -> 0603 (1608 Metric); Supplier P/N 311-1140-1-ND -> 311-1344-1-ND
- C36: footprint (none) -> Capacitor_SMD:C_0603_1608Metric; Digikey Link https://www.digikey.ca/en/products/detail/kemet/C0805C330J5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 -> https://www.digikey.ca/en/products/detail/kemet/c0603c330j5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; Manufacturer Part C0805C330J5GACTU -> 399-C0603C330J5GACTUCT-ND; Package 0805 -> 0603; Price 0.1 -> 0.12; Supplier P/N 399-C0805C330J5GACTUCT-ND -> 399-C0603C330J5GACTUCT-ND
- C37, C38, C39, C40: footprint (none) -> Capacitor_SMD:C_1210_3225Metric; Digikey Link https://www.digikey.ca/en/products/detail/samsung-electro-mechanics/cl31a226kahnnne/3888705 -> https://www.digikey.ca/en/products/detail/samsung-electro-mechanics/CL32B226MOJNNNE/3889053; Manufacturer Part CL31A226KAHNNNE -> CL32B226MOJNNNE; Package 1206 (3216 Metric) -> 1210 (3225 Metric); Price 0.08 -> 0.41; Supplier P/N 1276-3047-1-ND -> 1276-3395-1-ND; Type SMD -> SMD, MLCC
- C41: footprint (none) -> Capacitor_SMD:C_0603_1608Metric; Digikey Link https://www.digikey.ca/en/products/detail/kemet/C0805C104K5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 -> https://www.digikey.ca/en/products/detail/yageo/CC0603KRX7R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; Manufacturer KEMET -> YAGEO; Manufacturer Part C0805C104K5RACTU -> CC0603KRX7R9BB104; Package 0805 -> 0603 (1608 Metric); Supplier P/N 399-C0805C104K5RACTUCT-ND -> 311-1344-1-ND
- C42, C49, C5, C55: value 0.1u -> 100n; footprint (none) -> Capacitor_SMD:C_0603_1608Metric; Digikey Link https://www.digikey.ca/en/products/detail/samsung-electro-m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 -> https://www.digikey.ca/en/products/detail/yageo/CC0603KRX7R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; Manufacturer Samsung Electro-Mechanics -> YAGEO; Manufacturer Part CL31B104KBCNNNC -> CC0603KRX7R9BB104; Package 1206 (3216 Metric) -> 0603 (1608 Metric); Price 0.11 -> 0.08; Supplier P/N 1276-1017-1-ND -> 311-1344-1-ND
- C43: footprint (none) -> Capacitor_SMD:C_1206_3216Metric; Digikey Link https://www.digikey.ca/en/products/detail/samsung-electro-mechanics/CL21B105KAFNNNE/3886724 -> https://www.digikey.ca/en/products/detail/samsung-electro-mechanics/CL31B105KAHNNNE/3886755; Manufacturer Part CL21B105KAFNNNE -> CL31B105KAHNNNE; Package 0805 -> 1206 (3216 Metric); Price 0.08 -> 0.13; Supplier P/N 1276-1066-1-ND -> 1276-1097-1-ND
- C44: footprint (none) -> Capacitor_SMD:C_1210_3225Metric; Digikey Link https://www.digikey.ca/en/products/detail/samsung-electro-m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 -> https://www.digikey.ca/en/products/detail/taiyo-yuden/TMK32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; Manufacturer Samsung Electro-Mechanics -> Taiyo Yuden; Manufacturer Part CL31A226KAHNNNE -> TMK325B7226KM-PR; Package 1206 (3216 Metric) -> 1210 (3225 Metric); Price 0.08 -> 0.58; Supplier P/N 1276-3047-1-ND -> 587-5480-1-ND; Type SMD -> SMD, MLCC
- C45, C47: footprint (none) -> Capacitor_SMD:C_0603_1608Metric; Digikey Link https://www.digikey.ca/en/products/detail/kemet/c1206c475k8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 -> https://www.digikey.ca/en/products/detail/murata-electronic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; Manufacturer KEMET -> Murata Electronics; Manufacturer Part C1206C475K8RACTU -> GRM188Z71A475KE15D; Package 1206 (3216 Metric) -> 0603 (1608 Metric); Price 0.51 -> 0.22; Supplier P/N 399-C1206C475K8RACTUCT-ND -> 490-GRM188Z71A475KE15DCT-ND; Type SMD -> SMD, MLCC
- C46: footprint (none) -> Capacitor_SMD:C_1210_3225Metric; Digikey Link https://www.digikey.ca/en/products/detail/samsung-electro-mechanics/CL31B226KPHNNNE/3888427?s=N4IgTCBcDaIMIBkDMBGAQmMA2A0gBQAkA5EgURAF0BfIA -> https://www.digikey.ca/en/products/detail/samsung-electro-mechanics/CL32B226MOJNNNE/3889053; Manufacturer Part CL31B226KPHNNNE -> CL32B226MOJNNNE; Package 1206 (3216 Metric) -> 1210 (3225 Metric); Price 0.39 -> 0.41; Supplier P/N 1276-2769-1-ND -> 1276-3395-1-ND; Type SMD -> SMD, MLCC
- C48: footprint (none) -> Capacitor_SMD:C_0603_1608Metric; Digikey Link https://www.digikey.ca/en/products/detail/samsung-electro-m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 -> https://www.digikey.ca/en/products/detail/taiyo-yuden/UMK10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; Manufacturer Samsung Electro-Mechanics -> Taiyo Yuden; Manufacturer Part CL21B105KAFNNNE -> UMK107AB7105KA-T; Package 0805 -> 0603; Supplier P/N 1276-1066-1-ND -> 587-3247-1-ND
- D11, D12, D13, D14: value LED -> LTST-C170GKT
- D15: value LED -> LTST-C170YKT
- NT1: now in the parts list
- R10, R26, R32: footprint Resistor_SMD:R_0603_1608Metric -> Resistor_SMD:R_0805_2012Metric; Digikey Link https://www.digikey.ca/en/products/detail/yageo/RC1206FR-07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 -> https://www.digikey.ca/en/products/detail/yageo/RC0805FR-07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; Manufacturer Part RC1206FR-0710KL -> RC0805FR-0710KL; Package 1206 -> 0805; Price 0.1 -> 0.14; Supplier P/N 311-10.0KFRCT-ND -> 311-10.0KCRCT-ND
- R2, R27, R36: footprint Resistor_SMD:R_0603_1608Metric -> Resistor_SMD:R_0805_2012Metric
- R22: footprint Resistor_SMD:R_0603_1608Metric -> Resistor_SMD:R_0805_2012Metric; Digikey Link https://www.digikey.ca/en/products/detail/yageo/RC1206FR-07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 -> https://www.digikey.ca/en/products/detail/yageo/RC0805FR-07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; Manufacturer Part RC1206FR-07220KL -> RC0805FR-07220KL; Package 1206 -> 0805; Supplier P/N 311-220KFRCT-ND -> 311-220KCRCT-ND
- R23: value 100K -> 100k; footprint Resistor_SMD:R_0603_1608Metric -> Resistor_SMD:R_0805_2012Metric; Digikey Link https://www.digikey.ca/en/products/detail/yageo/RC1206FR-07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 -> https://www.digikey.ca/en/products/detail/yageo/RC0805FR-07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; Manufacturer Part RC1206FR-07100KL -> RC0805FR-07100KL; Package 1206 -> 0805; Supplier P/N 311-100KFRCT-ND -> 311-100KCRCT-ND
- R24: footprint Resistor_SMD:R_0603_1608Metric -> Resistor_SMD:R_0805_2012Metric; Digikey Link https://www.digikey.ca/en/products/detail/yageo/RC1206FR-07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 -> https://www.digikey.ca/en/products/detail/yageo/RC0805FR-07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; Manufacturer Part RC1206FR-0730K1L -> RC0805FR-0730K1L; Package 1206 -> 0805; Supplier P/N 311-30.1KFRCT-ND -> 311-30.1KCRCT-ND
- R25: footprint Resistor_SMD:R_0603_1608Metric -> Resistor_SMD:R_0805_2012Metric; Digikey Link https://www.digikey.ca/en/products/detail/yageo/RC1206FR-07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 -> https://www.digikey.ca/en/products/detail/yageo/RC0805FR-13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; Manufacturer Part RC1206FR-0730KL -> RC0805FR-1330KL; Package 1206 -> 0805; Supplier P/N 311-30.0KFRCT-ND -> 13-RC0805FR-1330KLCT-ND
- R28, R30, R31, R33, R34: footprint Resistor_SMD:R_0603_1608Metric -> Resistor_SMD:R_0805_2012Metric; Digikey Link https://www.digikey.ca/en/products/detail/yageo/RC1206FR-07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 -> https://www.digikey.ca/en/products/detail/yageo/RC0805FR-07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; Manufacturer Part RC1206FR-071K5L -> RC0805FR-071K5L; Package 1206 -> 0805; Supplier P/N 311-1.50KFRCT-ND -> 311-1.50KCRCT-ND
- R29: footprint Resistor_SMD:R_0603_1608Metric -> Resistor_SMD:R_0805_2012Metric; Digikey Link https://www.digikey.ca/en/products/detail/yageo/AC1206FR-07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 -> https://www.digikey.ca/en/products/detail/yageo/AC0805FR-07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; Manufacturer Part AC1206FR-0715KL -> AC0805FR-0715KL; Package 1206 -> 0805; Supplier P/N YAG3815CT-ND -> YAG3695CT-ND
- R35: footprint Resistor_SMD:R_0603_1608Metric -> Resistor_SMD:R_0805_2012Metric; Digikey Link https://www.digikey.ca/en/products/detail/yageo/RC1206FR-07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 -> https://www.digikey.ca/en/products/detail/yageo/RC0805FR-07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; Manufacturer Part RC1206FR-07120KL -> RC0805FR-07120KL; Package 1206 -> 0805; Supplier P/N 311-120KFRCT-ND -> 311-120KCRCT-ND
- R8: footprint Resistor_THT:R_Axial_DIN0207_L6.3mm_D2.5mm_P10.16mm_Horizontal -> Resistor_SMD:R_0805_2012Metric; Digikey Link https://www.digikey.ca/en/products/detail/yageo/RC1206FR-07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 -> https://www.digikey.ca/en/products/detail/yageo/RC0805FR-07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; Manufacturer Part RC1206FR-0776K8L -> RC0805FR-0776K8L; Package 1206 (3216 Metric) -> 0805; Supplier P/N 311-76.8KFRCT-ND -> 311-76.8KCRCT-ND
- R9: footprint Resistor_THT:R_Axial_DIN0207_L6.3mm_D2.5mm_P10.16mm_Horizontal -> Resistor_SMD:R_0805_2012Metric; Digikey Link https://www.digikey.ca/en/products/detail/yageo/RC1206FR-07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 -> https://www.digikey.ca/en/products/detail/yageo/RC0805FR-07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; Manufacturer Part RC1206FR-0724K3L -> RC0805FR-0724K3L; Package 1206 (3216 Metric) -> 0805; Supplier P/N 311-24.3KFRCT-ND -> 311-24.3KCRCT-ND

Commit message: Generated BOM
Parts:
- TP1: now in the parts list
Changed lines of the file:
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@@
 		(unit 1)
 		(exclude_from_sim no)
-		(in_bom no)
+		(in_bom yes)
 		(on_board yes)
 		(dnp no)

Commit message: Added side B for SW1
Parts:
- C32, C33, C34, C35, C36, C37, C38, C39, C40, C41, C42, C43, C44, C45, C46, C47, C48, C49, C5, C55: symbol PCM_Elektuur:C -> capstone_parts:C
- D10: symbol Diode:MBRA340 -> capstone_parts:MBRA340
- D11, D12, D13, D14, D15: symbol Device:LED -> capstone_parts:LED
- J15: symbol PCM_4ms_Connector:Conn_01x03 -> capstone_parts:Conn_01x03
- J20: symbol PCM_4ms_Connector:Conn_01x02 -> capstone_parts:Conn_01x02
- L1, L2: symbol PCM_SparkFun-Coil:2.2uH_0806_1.2A -> capstone_parts:2.2uH_0806_1.2A
- NT1: symbol Device:NetTie_2 -> capstone_parts:NetTie_2
- R10, R2, R22, R23, R24, R25, R26, R27, R28, R29, R30, R31, R32, R33, R34, R35, R36: symbol Device:R -> capstone_parts:R
- R8, R9: symbol PCM_SL_Resistors:0ohm -> capstone_parts:0ohm
- SW1: symbol Switch:SW_DPDT_x2 -> capstone_parts:SW_DPDT_x2
- SW8: symbol Switch:SW_Push -> capstone_parts:SW_Push
- TP1: symbol Connector:TestPoint -> capstone_parts:TestPoint
Connections:
- no-connect marks 2 -> 5

Commit message: switch fix
Connections:
- net +VBATT_7V4: now also SW1.3 (C), SW1.6 (C); no longer SW1.2 (B)
- net at SW1.1 (A): no longer R23.2
- net at SW1.5 (B): now also R23.2, SW1.2 (B)
- no-connect marks 5 -> 3
Other:
- moved on the sheet: SW1B
Changed lines of the file:
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@@
 	)
 	(junction
+		(at 58.42 33.02)
+		(diameter 0)
+		(color 0 0 0 0)
+	)
+	(junction
 		(at 180.34 25.4)
 		(diameter 0)
@@
 	)
 	(junction
+		(at 73.66 30.48)
+		(diameter 0)
+		(color 0 0 0 0)
+	)
+	(junction
 		(at 193.04 25.4)
 		(diameter 0)
@@
 	)
 	(no_connect
-		(at 71.12 35.56)
-	)
-	(no_connect
 		(at 60.96 48.26)
 	)
 	(no_connect
-		(at 71.12 45.72)
-	)
-	(no_connect
-		(at 71.12 50.8)
+		(at 60.96 27.94)
 	)
 	(no_connect
@@
 	(wire
 		(pts
+			(xy 60.96 43.18) (xy 58.42 43.18)
+		)
+		(stroke
+			(width 0)
+			(type default)
+		)
+	)
+	(wire
+		(pts
 			(xy 53.34 101.6) (xy 53.34 99.06)
 		)
@@
 	(wire
 		(pts
+			(xy 73.66 45.72) (xy 73.66 30.48)
+		)
+		(stroke
+			(width 0)
+			(type default)
+		)
+	)
+	(wire
+		(pts
 			(xy 114.3 121.92) (xy 119.38 121.92)
 		)
@@
 	(wire
 		(pts
-			(xy 76.2 30.48) (xy 71.12 30.48)
+			(xy 76.2 30.48) (xy 73.66 30.48)
 		)
 		(stroke
@@
 	(wire
 		(pts
+			(xy 71.12 45.72) (xy 73.66 45.72)
+		)
+		(stroke
+			(width 0)
+			(type default)
+		)
+	)
+	(wire
+		(pts
 			(xy 43.18 25.4) (xy 53.34 25.4)
 		)
@@
 	(wire
 		(pts
+			(xy 58.42 43.18) (xy 58.42 33.02)
+		)
+		(stroke
+			(width 0)
+			(type default)
+		)
+	)
+	(wire
+		(pts
 			(xy 76.2 33.02) (xy 76.2 30.48)
 		)
@@
 	(wire
 		(pts
+			(xy 73.66 30.48) (xy 71.12 30.48)
+		)
+		(stroke
+			(width 0)
+			(type default)
+		)
+	)
+	(wire
+		(pts
 			(xy 203.2 137.16) (xy 203.2 109.22)
 		)
@@
 	(symbol
 		(lib_id "capstone_parts:SW_DPDT_x2")
-		(at 66.04 33.02 0)
-		(unit 1)
+		(at 66.04 45.72 180)
+		(unit 2)
 		(exclude_from_sim no)
 		(in_bom yes)
@@
 		(dnp no)
 		(property "Reference" "SW1"
-			(at 66.04 38.608 0)
+			(at 66.04 54.61 0)
 			(effects
 				(font
@@
 		)
 		(property "Value" "TL2230EEF140"
-			(at 66.802 40.894 0)
+			(at 66.04 52.07 0)
 			(effects
 				(font
@@
 		)
 		(property "Footprint" "*CapStone*:SW_TL2230EEF140"
-			(at 66.04 33.02 0)
+			(at 66.04 45.72 0)
 			(effects
 				(font
@@
 		)
 		(property "Datasheet" "~"
-			(at 66.04 33.02 0)
+			(at 66.04 45.72 0)
 			(effects
 				(font
@@
 		)
 		(property "Description" "Switch, dual pole double throw, separate symbols"
-			(at 66.04 33.02 0)
+			(at 66.04 45.72 0)
 			(effects
 				(font
@@
 		)
 		(property "Digikey Link" "https://www.digikey.ca/en/products/detail/e-switch/TL2230EEF140/4029358"
-			(at 66.04 33.02 0)
+			(at 66.04 45.72 0)
 			(effects
 				(font
@@
 		)
 		(property "Manufacturer" "E-Switch"
-			(at 66.04 33.02 0)
+			(at 66.04 45.72 0)
 			(effects
 				(font
@@
 		)
 		(property "Manufacturer Part" "TL2230EEF140"
-			(at 66.04 33.02 0)
+			(at 66.04 45.72 0)
 			(effects
 				(font
@@
 		)
 		(property "Package" "Bulk"
-			(at 66.04 33.02 0)
+			(at 66.04 45.72 0)
 			(effects
 				(font
@@
 		)
 		(property "Price" "0.85"
-			(at 66.04 33.02 0)
+			(at 66.04 45.72 0)
 			(effects
 				(font
@@
 		)
 		(property "Supplier" "DigiKey"
-			(at 66.04 33.02 0)
+			(at 66.04 45.72 0)
 			(effects
 				(font
@@
 		)
 		(property "Supplier P/N" "EG6031-ND"
-			(at 66.04 33.02 0)
+			(at 66.04 45.72 0)
 			(effects
 				(font
@@
 		)
 		(property "Type" "Through Hole"
-			(at 66.04 33.02 0)
+			(at 66.04 45.72 0)
 			(effects
 				(font
@@
 		)
 		(property "Unit" "pcs"
-			(at 66.04 33.02 0)
+			(at 66.04 45.72 0)
 			(effects
 				(font
@@
 				(path "/365a82ed-827d-43e1-aa2f-b98221c4179c/f9f22bb2-829e-4ff5-89be-c4b5e2122135/9b56d3ca-82a9-4c6a-8125-2948d5100470"
 					(reference "SW1")
-					(unit 1)
+					(unit 2)
 				)
 			)
@@
 	(symbol
 		(lib_id "capstone_parts:SW_DPDT_x2")
-		(at 66.04 48.26 0)
-		(mirror x)
-		(unit 2)
+		(at 66.04 30.48 0)
+		(mirror y)
+		(unit 1)
 		(exclude_from_sim no)
 		(in_bom yes)
@@
 		(dnp no)
 		(property "Reference" "SW1"
-			(at 66.04 57.15 0)
+			(at 66.04 36.068 0)
 			(effects
 				(font
@@
 		)
 		(property "Value" "TL2230EEF140"
-			(at 66.04 54.61 0)
+			(at 66.294 38.608 0)
 			(effects
 				(font
@@
 		)
 		(property "Footprint" "*CapStone*:SW_TL2230EEF140"
-			(at 66.04 48.26 0)
+			(at 66.04 30.48 0)
 			(effects
 				(font
@@
 		)
 		(property "Datasheet" "~"
-			(at 66.04 48.26 0)
+			(at 66.04 30.48 0)
 			(effects
 				(font
@@
 		)
 		(property "Description" "Switch, dual pole double throw, separate symbols"
-			(at 66.04 48.26 0)
+			(at 66.04 30.48 0)
 			(effects
 				(font
@@
 		)
 		(property "Digikey Link" "https://www.digikey.ca/en/products/detail/e-switch/TL2230EEF140/4029358"
-			(at 66.04 48.26 0)
+			(at 66.04 30.48 0)
 			(effects
 				(font
@@
 		)
 		(property "Manufacturer" "E-Switch"
-			(at 66.04 48.26 0)
+			(at 66.04 30.48 0)
 			(effects
 				(font
@@
 		)
 		(property "Manufacturer Part" "TL2230EEF140"
-			(at 66.04 48.26 0)
+			(at 66.04 30.48 0)
 			(effects
 				(font
@@
 		)
 		(property "Package" "Bulk"
-			(at 66.04 48.26 0)
+			(at 66.04 30.48 0)
 			(effects
 				(font
@@
 		)
 		(property "Price" "0.85"
-			(at 66.04 48.26 0)
+			(at 66.04 30.48 0)
 			(effects
 				(font
@@
 		)
 		(property "Supplier" "DigiKey"
-			(at 66.04 48.26 0)
+			(at 66.04 30.48 0)
 			(effects
 				(font
@@
 		)
 		(property "Supplier P/N" "EG6031-ND"
-			(at 66.04 48.26 0)
+			(at 66.04 30.48 0)
 			(effects
 				(font
@@
 		)
 		(property "Type" "Through Hole"
-			(at 66.04 48.26 0)
+			(at 66.04 30.48 0)
 			(effects
 				(font
@@
 		)
 		(property "Unit" "pcs"
-			(at 66.04 48.26 0)
+			(at 66.04 30.48 0)
 			(effects
 				(font
@@
 				(path "/365a82ed-827d-43e1-aa2f-b98221c4179c/f9f22bb2-829e-4ff5-89be-c4b5e2122135/9b56d3ca-82a9-4c6a-8125-2948d5100470"
 					(reference "SW1")
-					(unit 2)
+					(unit 1)
 				)
 			)

Commit message: Changed connector 15 pin
Parts:
- added unit 1 of SW1
Connections:
- net +VBATT_7V4: now also SW1.3 (C); no longer SW1.3 (C)
- net at R23.2, SW1.5 (B): now also SW1.2 (B); no longer SW1.2 (B)

Commit message: started routing up to HDMI ESD impedance matching
Parts:
- J20: footprint Connector_PinHeader_2.54mm:PinHeader_1x02_P2.54mm_Vertical -> TerminalBlock_4Ucon:TerminalBlock_4Ucon_1x02_P3.50mm_Horizontal
Changed lines of the file:
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@@
 			)
 		)
-		(property "Footprint" "Connector_PinHeader_2.54mm:PinHeader_1x02_P2.54mm_Vertical"
+		(property "Footprint" "TerminalBlock_4Ucon:TerminalBlock_4Ucon_1x02_P3.50mm_Horizontal"
 			(at 227.965 71.755 0)
 			(effects
