File: 490_0/USBCurrentLimiter.kicad_sch (KiCad schematic)
At the start: 18 parts, among them U2 TPS2553DBVR, U3 TPS2553DBVR

Commit message: Reviewed BOM
- changed some capacitors to a more fitting voltage rating
Parts:
- C11, C3, C63, C64: value 0.1u -> 100n; Digikey Link https://www.digikey.ca/en/products/detail/yageo/CC0805JRX7R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 -> https://www.digikey.ca/en/products/detail/yageo/CC0805KRX7R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; Manufacturer Part CC0805JRX7R7BB104 -> CC0805KRX7R9BB104; Package 0805 -> 0805 (2012 Metric); Price 0.11 -> 0.08; Supplier P/N 311-4266-1-ND -> 311-1140-1-ND
- C16, C8: Digikey Link https://www.digikey.ca/en/products/detail/vishay-sprague/29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 -> https://www.digikey.ca/en/products/detail/vishay-sprague/59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; Manufacturer Part 293D127X96R3D2TE3 -> 594D127X9020R2T; Package 2917 (7343 Metric) -> 2824 (7260 Metric); Price 0.99 -> 6.97; Supplier P/N 718-1745-1-ND -> 718-594D127X9020R2TCT-ND
Changed lines of the file:
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@@
 			)
 		)
-		(property "Value" "0.1u"
+		(property "Value" "100n"
 			(at 71.882 79.248 0)
 			(effects
@@
 			)
 		)
-		(property "Description" "CAP CER 0.1UF 16V X7R 0805"
+		(property "Description" "CAP CER 0.1UF 50V X7R 0805"
 			(at 78.74 76.2 0)
 			(effects
@@
 			)
 		)
-		(property "Digikey Link" "https://www.digikey.ca/en/products/detail/yageo/CC0805JRX7R7BB104/5884101"
+		(property "Digikey Link" "https://www.digikey.ca/en/products/detail/yageo/CC0805KRX7R9BB104/302874?s=N4IgTCBcDaIMJwAwA5EFYDSAlAGgdiwE4AhYgRkQBYQBdAXyA"
 			(at 78.74 76.2 0)
 			(effects
@@
 			)
 		)
-		(property "Manufacturer Part" "CC0805JRX7R7BB104"
+		(property "Manufacturer Part" "CC0805KRX7R9BB104"
 			(at 78.74 76.2 0)
 			(effects
@@
 			)
 		)
-		(property "Package" "0805"
+		(property "Package" "0805 (2012 Metric)"
 			(at 78.74 76.2 0)
 			(effects
@@
 			)
 		)
-		(property "Price" "0.11"
+		(property "Price" "0.08"
 			(at 78.74 76.2 0)
 			(effects
@@
 			)
 		)
-		(property "Supplier P/N" "311-4266-1-ND"
+		(property "Supplier P/N" "311-1140-1-ND"
 			(at 78.74 76.2 0)
 			(effects
@@
 			)
 		)
-		(property "Value" "0.1u"
+		(property "Value" "100n"
 			(at 99.822 132.588 0)
 			(effects
@@
 			)
 		)
-		(property "Description" "CAP CER 0.1UF 16V X7R 0805"
+		(property "Description" "CAP CER 0.1UF 50V X7R 0805"
 			(at 106.68 129.54 0)
 			(effects
@@
 			)
 		)
-		(property "Digikey Link" "https://www.digikey.ca/en/products/detail/yageo/CC0805JRX7R7BB104/5884101"
+		(property "Digikey Link" "https://www.digikey.ca/en/products/detail/yageo/CC0805KRX7R9BB104/302874?s=N4IgTCBcDaIMJwAwA5EFYDSAlAGgdiwE4AhYgRkQBYQBdAXyA"
 			(at 106.68 129.54 0)
 			(effects
@@
 			)
 		)
-		(property "Manufacturer Part" "CC0805JRX7R7BB104"
+		(property "Manufacturer Part" "CC0805KRX7R9BB104"
 			(at 106.68 129.54 0)
 			(effects
@@
 			)
 		)
-		(property "Package" "0805"
+		(property "Package" "0805 (2012 Metric)"
 			(at 106.68 129.54 0)
 			(effects
@@
 			)
 		)
-		(property "Price" "0.11"
+		(property "Price" "0.08"
 			(at 106.68 129.54 0)
 			(effects
@@
 			)
 		)
-		(property "Supplier P/N" "311-4266-1-ND"
+		(property "Supplier P/N" "311-1140-1-ND"
 			(at 106.68 129.54 0)
 			(effects
@@
 			)
 		)
-		(property "Datasheet" "kicad-embed://293d.pdf"
+		(property "Datasheet" "kicad-embed://594d.pdf"
 			(at 175.26 120.65 0)
 			(effects
@@
 			)
 		)
-		(property "Description" "CAP TANT 120UF 10% 6.3V 2917"
+		(property "Description" "CAP TANT 120UF 10% 20V 2824"
 			(at 175.26 120.65 0)
 			(effects
@@
 			)
 		)
-		(property "Manufacturer Part" "293D127X96R3D2TE3"
+		(property "Manufacturer Part" "594D127X9020R2T"
 			(at 175.26 120.65 0)
 			(effects
@@
 			)
 		)
-		(property "Supplier P/N" "718-1745-1-ND"
+		(property "Supplier P/N" "718-594D127X9020R2TCT-ND"
 			(at 175.26 120.65 0)
 			(effects
@@
 			)
 		)
-		(property "Digikey Link" "https://www.digikey.ca/en/products/detail/vishay-sprague/293D127X96R3D2TE3/2259902"
+		(property "Digikey Link" "https://www.digikey.ca/en/products/detail/vishay-sprague/594D127X9020R2T/1577743"
 			(at 175.26 120.65 0)
 			(effects
@@
 			)
 		)
-		(property "Package" "2917 (7343 Metric)"
+		(property "Package" "2824 (7260 Metric)"
 			(at 175.26 120.65 0)
 			(effects
@@
 			)
 		)
-		(property "Price" "0.99"
+		(property "Price" "6.97"
 			(at 175.26 120.65 0)
 			(effects
@@
 			)
 		)
-		(property "Value" "0.1u"
+		(property "Value" "100n"
 			(at 99.822 89.408 0)
 			(effects
@@
 			)
 		)
-		(property "Description" "CAP CER 0.1UF 16V X7R 0805"
+		(property "Description" "CAP CER 0.1UF 50V X7R 0805"
 			(at 106.68 86.36 0)
 			(effects
@@
 			)
 		)
-		(property "Digikey Link" "https://www.digikey.ca/en/products/detail/yageo/CC0805JRX7R7BB104/5884101"
+		(property "Digikey Link" "https://www.digikey.ca/en/products/detail/yageo/CC0805KRX7R9BB104/302874?s=N4IgTCBcDaIMJwAwA5EFYDSAlAGgdiwE4AhYgRkQBYQBdAXyA"
 			(at 106.68 86.36 0)
 			(effects
@@
 			)
 		)
-		(property "Manufacturer Part" "CC0805JRX7R7BB104"
+		(property "Manufacturer Part" "CC0805KRX7R9BB104"
 			(at 106.68 86.36 0)
 			(effects
@@
 			)
 		)
-		(property "Package" "0805"
+		(property "Package" "0805 (2012 Metric)"
 			(at 106.68 86.36 0)
 			(effects
@@
 			)
 		)
-		(property "Price" "0.11"
+		(property "Price" "0.08"
 			(at 106.68 86.36 0)
 			(effects
@@
 			)
 		)
-		(property "Supplier P/N" "311-4266-1-ND"
+		(property "Supplier P/N" "311-1140-1-ND"
 			(at 106.68 86.36 0)
 			(effects
@@
 			)
 		)
-		(property "Datasheet" "kicad-embed://293d.pdf"
+		(property "Datasheet" "kicad-embed://594d.pdf"
 			(at 175.26 77.47 0)
 			(effects
@@
 			)
 		)
-		(property "Description" "CAP TANT 120UF 10% 6.3V 2917"
+		(property "Description" "CAP TANT 120UF 10% 20V 2824"
 			(at 175.26 77.47 0)
 			(effects
@@
 			)
 		)
-		(property "Manufacturer Part" "293D127X96R3D2TE3"
+		(property "Manufacturer Part" "594D127X9020R2T"
 			(at 175.26 77.47 0)
 			(effects
@@
 			)
 		)
-		(property "Supplier P/N" "718-1745-1-ND"
+		(property "Supplier P/N" "718-594D127X9020R2TCT-ND"
 			(at 175.26 77.47 0)
 			(effects
@@
 			)
 		)
-		(property "Digikey Link" "https://www.digikey.ca/en/products/detail/vishay-sprague/293D127X96R3D2TE3/2259902"
+		(property "Digikey Link" "https://www.digikey.ca/en/products/detail/vishay-sprague/594D127X9020R2T/1577743"
 			(at 175.26 77.47 0)
 			(effects
@@
 			)
 		)
-		(property "Package" "2917 (7343 Metric)"
+		(property "Package" "2824 (7260 Metric)"
 			(at 175.26 77.47 0)
 			(effects
@@
 			)
 		)
-		(property "Price" "0.99"
+		(property "Price" "6.97"
 			(at 175.26 77.47 0)
 			(effects
@@
 			)
 		)
-		(property "Value" "0.1u"
+		(property "Value" "100n"
 			(at 71.882 122.428 0)
 			(effects
@@
 			)
 		)
-		(property "Description" "CAP CER 0.1UF 16V X7R 0805"
+		(property "Description" "CAP CER 0.1UF 50V X7R 0805"
 			(at 78.74 119.38 0)
 			(effects
@@
 			)
 		)
-		(property "Digikey Link" "https://www.digikey.ca/en/products/detail/yageo/CC0805JRX7R7BB104/5884101"
+		(property "Digikey Link" "https://www.digikey.ca/en/products/detail/yageo/CC0805KRX7R9BB104/302874?s=N4IgTCBcDaIMJwAwA5EFYDSAlAGgdiwE4AhYgRkQBYQBdAXyA"
 			(at 78.74 119.38 0)
 			(effects
@@
 			)
 		)
-		(property "Manufacturer Part" "CC0805JRX7R7BB104"
+		(property "Manufacturer Part" "CC0805KRX7R9BB104"
 			(at 78.74 119.38 0)
 			(effects
@@
 			)
 		)
-		(property "Package" "0805"
+		(property "Package" "0805 (2012 Metric)"
 			(at 78.74 119.38 0)
 			(effects
@@
 			)
 		)
-		(property "Price" "0.11"
+		(property "Price" "0.08"
 			(at 78.74 119.38 0)
 			(effects
@@
 			)
 		)
-		(property "Supplier P/N" "311-4266-1-ND"
+		(property "Supplier P/N" "311-1140-1-ND"
 			(at 78.74 119.38 0)
 			(effects
