File: 490_0/USBCurrentLimiter.kicad_sch (KiCad schematic)
At the start: 18 parts, among them U2 TPS2553DBVR, U3 TPS2553DBVR

Commit message: Changed 8conn and BOM update
Parts:
- C11, C3, C63, C64: footprint (none) -> Capacitor_SMD:C_0805_2012Metric
- C12, C4: footprint (none) -> Capacitor_SMD:C_1206_3216Metric
- C16, C8: footprint (none) -> Capacitor_Tantalum_SMD:CP_EIA-7260-38_AVX-R_HandSolder
Changed lines of the file:
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@@
 			)
 		)
-		(property "Footprint" ""
+		(property "Footprint" "Capacitor_SMD:C_0805_2012Metric"
 			(at 78.74 76.2 0)
 			(effects
@@
 			)
 		)
-		(property "Footprint" ""
+		(property "Footprint" "Capacitor_SMD:C_0805_2012Metric"
 			(at 106.68 129.54 0)
 			(effects
@@
 			)
 		)
-		(property "Footprint" ""
+		(property "Footprint" "Capacitor_SMD:C_1206_3216Metric"
 			(at 193.04 76.2 0)
 			(effects
@@
 			)
 		)
-		(property "Footprint" ""
+		(property "Footprint" "Capacitor_Tantalum_SMD:CP_EIA-7260-38_AVX-R_HandSolder"
 			(at 176.2252 124.46 0)
 			(effects
@@
 			)
 		)
-		(property "Footprint" ""
+		(property "Footprint" "Capacitor_SMD:C_0805_2012Metric"
 			(at 106.68 86.36 0)
 			(effects
@@
 			)
 		)
-		(property "Footprint" ""
+		(property "Footprint" "Capacitor_SMD:C_1206_3216Metric"
 			(at 193.04 119.38 0)
 			(effects
@@
 			)
 		)
-		(property "Footprint" ""
+		(property "Footprint" "Capacitor_Tantalum_SMD:CP_EIA-7260-38_AVX-R_HandSolder"
 			(at 176.2252 81.28 0)
 			(effects
@@
 			)
 		)
-		(property "Footprint" ""
+		(property "Footprint" "Capacitor_SMD:C_0805_2012Metric"
 			(at 78.74 119.38 0)
 			(effects

Commit message: LED names + 5V routing through ESD + renamed ESD chips to "U"
Parts:
- D1, D2: value LED -> LTST-C170TBKT
Changed lines of the file:
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@@
 			)
 		)
-		(property "Value" "LED"
-			(at 156.21 108.458 0)
+		(property "Value" "LTST-C170TBKT"
+			(at 150.114 101.346 0)
 			(effects
 				(font
@@
 			)
 		)
-		(property "Value" "LED"
-			(at 156.21 65.278 0)
-			(effects
-				(font
+		(property "Value" "LTST-C170TBKT"
+			(at 156.21 57.404 0)
+			(effects
+				(font

Commit message: Changed footprint for R4 and R6 to SMD
Parts:
- R4, R6: footprint Resistor_THT:R_Axial_DIN0207_L6.3mm_D2.5mm_P10.16mm_Horizontal -> Resistor_SMD:R_0805_2012Metric
Changed lines of the file:
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@@
 			)
 		)
-		(property "Footprint" "Resistor_THT:R_Axial_DIN0207_L6.3mm_D2.5mm_P10.16mm_Horizontal"
+		(property "Footprint" "Resistor_SMD:R_0805_2012Metric"
 			(at 162.179 121.158 0)
 			(effects
@@
 			)
 		)
-		(property "Footprint" "Resistor_THT:R_Axial_DIN0207_L6.3mm_D2.5mm_P10.16mm_Horizontal"
+		(property "Footprint" "Resistor_SMD:R_0805_2012Metric"
 			(at 162.179 77.978 0)
 			(effects

Commit message: Changed capacitor sizes
🟢 Group 1: 100% Safe to Shrink to 0603These capacitors handle logic-level decoupling or high-frequency filtering on your 3.3V and 5V lines. Because the capacitance values are low (1µF or less), an 0603 package can easily handle the DC bias without losing performance.All 0.1µF (100nF) Capacitors: You have 25 of these scattered across the board (e.g., C35, C41, C42, C49, C53-C61). Change every single one of these to 0603.The 1µF Logic Capacitors (C48, C62): C48 sits on the VCC pin of your battery charger. C62 is on the 3.3V rail for the USB hub. Change these to 0603.The 4.7µF Capacitors (C45, C47, C50): C45 and C47 sit on the 5V VL pin. C50 filters the 5V HDMI line. Change these to 0603.The 33pF Capacitors (C17, C18, C36): C17 and C18 are your crystal load capacitors and are already perfectly sized. C36 is a feedforward capacitor for your buck converter. Make sure all three are 0603.
🟡 Group 2: The "Compromise" - Shrink to 0805These 10µF capacitors sit on your 5V and 3.3V rails to smooth out the power for your motors, speakers, and USB hub (e.g., C1, C2, C4, C6, C12, C13, C15, C20, C22, C24).The Recommendation: While you have them listed as 1206, shrinking a 10µF ceramic capacitor all the way down to 0603 for a noisy 5V motor line will cause it to lose too much effective capacitance. 0805 is the perfect middle-ground here. It saves space but keeps your motor rails stable.
🔴 Group 3: DO NOT SHRINK (Keep 1206 / 1210 / 2824)These capacitors are exposed to the +VBATT_7V4 rail (up to 8.4V) or act as massive bulk storage. If you shrink these, your system will likely fail under heavy load.C32, C33, C34 (10µF): These connect directly to the high-voltage VIN pin of your main buck converter. Keep as 1206.C44 (22µF): This is the main switching capacitor for the battery charger inductor. Keep as 1210.C37, C38, C39, C40, C46 (22µF): These are the massive bulk output capacitors holding up your main 5V rail. Keep as 1210.C43 (1µF): Because this sits on the VH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
Parts:
- C11, C3, C63, C64: Digikey Link https://www.digikey.ca/en/products/detail/yageo/CC0805KRX7R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 -> https://www.digikey.ca/en/products/detail/yageo/CC0603KRX7R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; Manufacturer Part CC0805KRX7R9BB104 -> CC0603KRX7R9BB104; Package 0805 (2012 Metric) -> 0603 (1608 Metric); Supplier P/N 311-1140-1-ND -> 311-1344-1-ND
- C12, C4: Digikey Link https://www.digikey.ca/en/products/detail/kemet/c1206c106k4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 -> https://www.digikey.ca/en/products/detail/samsung-electro-m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; Manufacturer KEMET -> Samsung Electro-Mechanics; Manufacturer Part C1206C106K4RACTU -> CL21B106KOQNNNE; Package 1206 (3216 Metric) -> 0805; Price 0.31 -> 0.22; Supplier P/N 399-C1206C106K4RACTUCT-ND -> 1276-2872-1-ND
Changed lines of the file:
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@@
 			)
 		)
-		(property "Description" "CAP CER 0.1UF 50V X7R 0805"
+		(property "Description" "CAP CER 0.1UF 50V X7R 0603"
 			(at 78.74 76.2 0)
 			(effects
@@
 			)
 		)
-		(property "Digikey Link" "https://www.digikey.ca/en/products/detail/yageo/CC0805KRX7R9BB104/302874?s=N4IgTCBcDaIMJwAwA5EFYDSAlAGgdiwE4AhYgRkQBYQBdAXyA"
+		(property "Digikey Link" "https://www.digikey.ca/en/products/detail/yageo/CC0603KRX7R9BB104/2103082"
 			(at 78.74 76.2 0)
 			(effects
@@
 			)
 		)
-		(property "Manufacturer Part" "CC0805KRX7R9BB104"
+		(property "Manufacturer Part" "CC0603KRX7R9BB104"
 			(at 78.74 76.2 0)
 			(effects
@@
 			)
 		)
-		(property "Package" "0805 (2012 Metric)"
+		(property "Package" "0603 (1608 Metric)"
 			(at 78.74 76.2 0)
 			(effects
@@
 			)
 		)
-		(property "Supplier P/N" "311-1140-1-ND"
+		(property "Supplier P/N" "311-1344-1-ND"
 			(at 78.74 76.2 0)
 			(effects
@@
 			)
 		)
-		(property "Description" "CAP CER 0.1UF 50V X7R 0805"
+		(property "Description" "CAP CER 0.1UF 50V X7R 0603"
 			(at 106.68 129.54 0)
 			(effects
@@
 			)
 		)
-		(property "Digikey Link" "https://www.digikey.ca/en/products/detail/yageo/CC0805KRX7R9BB104/302874?s=N4IgTCBcDaIMJwAwA5EFYDSAlAGgdiwE4AhYgRkQBYQBdAXyA"
+		(property "Digikey Link" "https://www.digikey.ca/en/products/detail/yageo/CC0603KRX7R9BB104/2103082"
 			(at 106.68 129.54 0)
 			(effects
@@
 			)
 		)
-		(property "Manufacturer Part" "CC0805KRX7R9BB104"
+		(property "Manufacturer Part" "CC0603KRX7R9BB104"
 			(at 106.68 129.54 0)
 			(effects
@@
 			)
 		)
-		(property "Package" "0805 (2012 Metric)"
+		(property "Package" "0603 (1608 Metric)"
 			(at 106.68 129.54 0)
 			(effects
@@
 			)
 		)
-		(property "Supplier P/N" "311-1140-1-ND"
+		(property "Supplier P/N" "311-1344-1-ND"
 			(at 106.68 129.54 0)
 			(effects
@@
 			)
 		)
-		(property "Datasheet" "kicad-embed://KEM_C1002_X7R_SMD.pdf"
+		(property "Datasheet" "kicad-embed://CL_Series_MLCC_ds.pdf"
 			(at 193.04 76.2 0)
 			(effects
@@
 			)
 		)
-		(property "Description" "CAP CER 10UF 16V X7R 1206"
+		(property "Description" "CAP CER 10UF 16V X7R 0805"
 			(at 193.04 76.2 0)
 			(effects
@@
 			)
 		)
-		(property "Digikey Link" "https://www.digikey.ca/en/products/detail/kemet/c1206c106k4ractu/789657"
+		(property "Digikey Link" "https://www.digikey.ca/en/products/detail/samsung-electro-mechanics/CL21B106KOQNNNE/3888530"
 			(at 193.04 76.2 0)
 			(effects
@@
 			)
 		)
-		(property "Manufacturer" "KEMET"
+		(property "Manufacturer" "Samsung Electro-Mechanics"
 			(at 193.04 76.2 0)
 			(effects
@@
 			)
 		)
-		(property "Manufacturer Part" "C1206C106K4RACTU"
+		(property "Manufacturer Part" "CL21B106KOQNNNE"
 			(at 193.04 76.2 0)
 			(effects
@@
 			)
 		)
-		(property "Supplier P/N" "399-C1206C106K4RACTUCT-ND"
+		(property "Supplier P/N" "1276-2872-1-ND"
 			(at 193.04 76.2 0)
 			(effects
@@
 			)
 		)
-		(property "Package" "1206 (3216 Metric)"
+		(property "Package" "0805"
 			(at 193.04 76.2 0)
 			(effects
@@
 			)
 		)
-		(property "Price" "0.31"
+		(property "Price" "0.22"
 			(at 193.04 76.2 0)
 			(effects
@@
 			)
 		)
-		(property "Description" "CAP CER 0.1UF 50V X7R 0805"
+		(property "Description" "CAP CER 0.1UF 50V X7R 0603"
 			(at 106.68 86.36 0)
 			(effects
@@
 			)
 		)
-		(property "Digikey Link" "https://www.digikey.ca/en/products/detail/yageo/CC0805KRX7R9BB104/302874?s=N4IgTCBcDaIMJwAwA5EFYDSAlAGgdiwE4AhYgRkQBYQBdAXyA"
+		(property "Digikey Link" "https://www.digikey.ca/en/products/detail/yageo/CC0603KRX7R9BB104/2103082"
 			(at 106.68 86.36 0)
 			(effects
@@
 			)
 		)
-		(property "Manufacturer Part" "CC0805KRX7R9BB104"
+		(property "Manufacturer Part" "CC0603KRX7R9BB104"
 			(at 106.68 86.36 0)
 			(effects
@@
 			)
 		)
-		(property "Package" "0805 (2012 Metric)"
+		(property "Package" "0603 (1608 Metric)"
 			(at 106.68 86.36 0)
 			(effects
@@
 			)
 		)
-		(property "Supplier P/N" "311-1140-1-ND"
+		(property "Supplier P/N" "311-1344-1-ND"
 			(at 106.68 86.36 0)
 			(effects
@@
 			)
 		)
-		(property "Datasheet" "kicad-embed://KEM_C1002_X7R_SMD.pdf"
+		(property "Datasheet" "kicad-embed://CL_Series_MLCC_ds.pdf"
 			(at 193.04 119.38 0)
 			(effects
@@
 			)
 		)
-		(property "Description" "CAP CER 10UF 16V X7R 1206"
+		(property "Description" "CAP CER 10UF 16V X7R 0805"
 			(at 193.04 119.38 0)
 			(effects
@@
 			)
 		)
-		(property "Digikey Link" "https://www.digikey.ca/en/products/detail/kemet/c1206c106k4ractu/789657"
+		(property "Digikey Link" "https://www.digikey.ca/en/products/detail/samsung-electro-mechanics/CL21B106KOQNNNE/3888530"
 			(at 193.04 119.38 0)
 			(effects
@@
 			)
 		)
-		(property "Manufacturer" "KEMET"
+		(property "Manufacturer" "Samsung Electro-Mechanics"
 			(at 193.04 119.38 0)
 			(effects
@@
 			)
 		)
-		(property "Manufacturer Part" "C1206C106K4RACTU"
+		(property "Manufacturer Part" "CL21B106KOQNNNE"
 			(at 193.04 119.38 0)
 			(effects
@@
 			)
 		)
-		(property "Supplier P/N" "399-C1206C106K4RACTUCT-ND"
+		(property "Supplier P/N" "1276-2872-1-ND"
 			(at 193.04 119.38 0)
 			(effects
@@
 			)
 		)
-		(property "Package" "1206 (3216 Metric)"
+		(property "Package" "0805"
 			(at 193.04 119.38 0)
 			(effects
@@
 			)
 		)
-		(property "Price" "0.31"
+		(property "Price" "0.22"
 			(at 193.04 119.38 0)
 			(effects
@@
 			)
 		)
-		(property "Description" "CAP CER 0.1UF 50V X7R 0805"
+		(property "Description" "CAP CER 0.1UF 50V X7R 0603"
 			(at 78.74 119.38 0)
 			(effects
@@
 			)
 		)
-		(property "Digikey Link" "https://www.digikey.ca/en/products/detail/yageo/CC0805KRX7R9BB104/302874?s=N4IgTCBcDaIMJwAwA5EFYDSAlAGgdiwE4AhYgRkQBYQBdAXyA"
+		(property "Digikey Link" "https://www.digikey.ca/en/products/detail/yageo/CC0603KRX7R9BB104/2103082"
 			(at 78.74 119.38 0)
 			(effects
@@
 			)
 		)
-		(property "Manufacturer Part" "CC0805KRX7R9BB104"
+		(property "Manufacturer Part" "CC0603KRX7R9BB104"
 			(at 78.74 119.38 0)
 			(effects
@@
 			)
 		)
-		(property "Package" "0805 (2012 Metric)"
+		(property "Package" "0603 (1608 Metric)"
 			(at 78.74 119.38 0)
 			(effects
@@
 			)
 		)
-		(property "Supplier P/N" "311-1140-1-ND"
+		(property "Supplier P/N" "311-1344-1-ND"
 			(at 78.74 119.38 0)
 			(effects

Commit message: Assigned capacitor footprints
Parts:
- C11, C3, C63, C64: footprint Capacitor_SMD:C_0805_2012Metric -> Capacitor_SMD:C_0603_1608Metric
- C12, C4: footprint Capacitor_SMD:C_1206_3216Metric -> Capacitor_SMD:C_0805_2012Metric
Changed lines of the file:
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@@
 			)
 		)
-		(property "Footprint" "Capacitor_SMD:C_0805_2012Metric"
+		(property "Footprint" "Capacitor_SMD:C_0603_1608Metric"
 			(at 78.74 76.2 0)
 			(effects
@@
 			)
 		)
-		(property "Footprint" "Capacitor_SMD:C_0805_2012Metric"
+		(property "Footprint" "Capacitor_SMD:C_0603_1608Metric"
 			(at 106.68 129.54 0)
 			(effects
@@
 			)
 		)
-		(property "Footprint" "Capacitor_SMD:C_1206_3216Metric"
+		(property "Footprint" "Capacitor_SMD:C_0805_2012Metric"
 			(at 193.04 76.2 0)
 			(effects
@@
 			)
 		)
-		(property "Footprint" "Capacitor_SMD:C_0805_2012Metric"
+		(property "Footprint" "Capacitor_SMD:C_0603_1608Metric"
 			(at 106.68 86.36 0)
 			(effects
@@
 			)
 		)
-		(property "Footprint" "Capacitor_SMD:C_1206_3216Metric"
+		(property "Footprint" "Capacitor_SMD:C_0805_2012Metric"
 			(at 193.04 119.38 0)
 			(effects
@@
 			)
 		)
-		(property "Footprint" "Capacitor_SMD:C_0805_2012Metric"
+		(property "Footprint" "Capacitor_SMD:C_0603_1608Metric"
 			(at 78.74 119.38 0)
 			(effects

Commit message: Changed all the resistors to 0805 size
Parts:
- R3, R5: footprint Resistor_SMD:R_0603_1608Metric -> Resistor_SMD:R_0805_2012Metric; Digikey Link https://www.digikey.ca/en/products/detail/yageo/RC1206FR-07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 -> https://www.digikey.ca/en/products/detail/yageo/RC0805FR-07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; Manufacturer Part RC1206FR-071KL -> RC0805FR-071KL; Package 1206 -> 0805; Price 0.11 -> 0.1; Supplier P/N 311-1.00KFRCT-ND -> 311-1.00KCRCT-ND
- R39, R40: value 100K -> 100k; footprint Resistor_SMD:R_0603_1608Metric -> Resistor_SMD:R_0805_2012Metric; Digikey Link https://www.digikey.ca/en/products/detail/yageo/RC1206FR-07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 -> https://www.digikey.ca/en/products/detail/yageo/RC0805FR-07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; Manufacturer Part RC1206FR-07100KL -> RC0805FR-07100KL; Package 1206 -> 0805; Supplier P/N 311-100KFRCT-ND -> 311-100KCRCT-ND
Changed lines of the file:
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@@
 			)
 		)
-		(property "Value" "100K"
+		(property "Value" "100k"
 			(at 100.076 78.74 90)
 			(effects
@@
 			)
 		)
-		(property "Footprint" "Resistor_SMD:R_0603_1608Metric"
+		(property "Footprint" "Resistor_SMD:R_0805_2012Metric"
 			(at 100.33 76.962 90)
 			(effects
@@
 			)
 		)
-		(property "Datasheet" "kicad-embed://PYU-RC_GROUP_51_ROHS_L (YAGEO resistors).pdf"
+		(property "Datasheet" "kicad-embed://RC0805FR-07100KL (100k ohm resistor).pdf"
 			(at 100.33 78.74 0)
 			(effects
@@
 			)
 		)
-		(property "Description" "RES 100K OHM 1% 1/4W 1206"
+		(property "Description" "RES 100K OHM 1% 1/8W 0805"
 			(at 100.33 78.74 0)
 			(effects
@@
 			)
 		)
-		(property "Digikey Link" "https://www.digikey.ca/en/products/detail/yageo/RC1206FR-07100KL/728492"
+		(property "Digikey Link" "https://www.digikey.ca/en/products/detail/yageo/RC0805FR-07100KL/727544"
 			(at 100.33 78.74 90)
 			(effects
@@
 			)
 		)
-		(property "Manufacturer Part" "RC1206FR-07100KL"
+		(property "Manufacturer Part" "RC0805FR-07100KL"
 			(at 100.33 78.74 90)
 			(effects
@@
 			)
 		)
-		(property "Supplier P/N" "311-100KFRCT-ND"
+		(property "Supplier P/N" "311-100KCRCT-ND"
 			(at 100.33 78.74 90)
 			(effects
@@
 			)
 		)
-		(property "Package" "1206"
+		(property "Package" "0805"
 			(at 100.33 78.74 90)
 			(effects
@@
 			)
 		)
-		(property "Footprint" "Resistor_SMD:R_0603_1608Metric"
+		(property "Footprint" "Resistor_SMD:R_0805_2012Metric"
 			(at 163.83 62.738 90)
 			(effects
@@
 			)
 		)
-		(property "Description" "RES 1K OHM 1% 1/4W 1206"
+		(property "Description" "RES 1K OHM 1% 1/8W 0805"
 			(at 163.83 60.96 0)
 			(effects
@@
 			)
 		)
-		(property "Digikey Link" "https://www.digikey.ca/en/products/detail/yageo/RC1206FR-071KL/728387"
+		(property "Digikey Link" "https://www.digikey.ca/en/products/detail/yageo/RC0805FR-071KL/727444"
 			(at 163.83 60.96 90)
 			(effects
@@
 			)
 		)
-		(property "Manufacturer Part" "RC1206FR-071KL"
+		(property "Manufacturer Part" "RC0805FR-071KL"
 			(at 163.83 60.96 90)
 			(effects
@@
 			)
 		)
-		(property "Supplier P/N" "311-1.00KFRCT-ND"
+		(property "Supplier P/N" "311-1.00KCRCT-ND"
 			(at 163.83 60.96 90)
 			(effects
@@
 			)
 		)
-		(property "Package" "1206"
+		(property "Package" "0805"
 			(at 163.83 60.96 90)
 			(effects
@@
 			)
 		)
-		(property "Price" "0.11"
+		(property "Price" "0.1"
 			(at 163.83 60.96 90)
 			(effects
@@
 			)
 		)
-		(property "Value" "100K"
+		(property "Value" "100k"
 			(at 100.076 121.92 90)
 			(effects
@@
 			)
 		)
-		(property "Footprint" "Resistor_SMD:R_0603_1608Metric"
+		(property "Footprint" "Resistor_SMD:R_0805_2012Metric"
 			(at 100.33 120.142 90)
 			(effects
@@
 			)
 		)
-		(property "Datasheet" "kicad-embed://PYU-RC_GROUP_51_ROHS_L (YAGEO resistors).pdf"
+		(property "Datasheet" "kicad-embed://RC0805FR-07100KL (100k ohm resistor).pdf"
 			(at 100.33 121.92 0)
 			(effects
@@
 			)
 		)
-		(property "Description" "RES 100K OHM 1% 1/4W 1206"
+		(property "Description" "RES 100K OHM 1% 1/8W 0805"
 			(at 100.33 121.92 0)
 			(effects
@@
 			)
 		)
-		(property "Digikey Link" "https://www.digikey.ca/en/products/detail/yageo/RC1206FR-07100KL/728492"
+		(property "Digikey Link" "https://www.digikey.ca/en/products/detail/yageo/RC0805FR-07100KL/727544"
 			(at 100.33 121.92 90)
 			(effects
@@
 			)
 		)
-		(property "Manufacturer Part" "RC1206FR-07100KL"
+		(property "Manufacturer Part" "RC0805FR-07100KL"
 			(at 100.33 121.92 90)
 			(effects
@@
 			)
 		)
-		(property "Supplier P/N" "311-100KFRCT-ND"
+		(property "Supplier P/N" "311-100KCRCT-ND"
 			(at 100.33 121.92 90)
 			(effects
@@
 			)
 		)
-		(property "Package" "1206"
+		(property "Package" "0805"
 			(at 100.33 121.92 90)
 			(effects
@@
 			)
 		)
-		(property "Footprint" "Resistor_SMD:R_0603_1608Metric"
+		(property "Footprint" "Resistor_SMD:R_0805_2012Metric"
 			(at 163.83 105.918 90)
 			(effects
@@
 			)
 		)
-		(property "Description" "RES 1K OHM 1% 1/4W 1206"
+		(property "Description" "RES 1K OHM 1% 1/8W 0805"
 			(at 163.83 104.14 0)
 			(effects
@@
 			)
 		)
-		(property "Digikey Link" "https://www.digikey.ca/en/products/detail/yageo/RC1206FR-071KL/728387"
+		(property "Digikey Link" "https://www.digikey.ca/en/products/detail/yageo/RC0805FR-071KL/727444"
 			(at 163.83 104.14 90)
 			(effects
@@
 			)
 		)
-		(property "Manufacturer Part" "RC1206FR-071KL"
+		(property "Manufacturer Part" "RC0805FR-071KL"
 			(at 163.83 104.14 90)
 			(effects
@@
 			)
 		)
-		(property "Supplier P/N" "311-1.00KFRCT-ND"
+		(property "Supplier P/N" "311-1.00KCRCT-ND"
 			(at 163.83 104.14 90)
 			(effects
@@
 			)
 		)
-		(property "Package" "1206"
+		(property "Package" "0805"
 			(at 163.83 104.14 90)
 			(effects
@@
 			)
 		)
-		(property "Price" "0.11"
+		(property "Price" "0.1"
 			(at 163.83 104.14 90)
 			(effects
