File: 490_0/pwm_motors.kicad_sch (KiCad schematic)
At the start: 38 parts, among them J10 PAD, J4 PAD, J5 PAD, J6 PAD, J9 PAD, Q1 AO3400A, Q2 AO3400A, Q3 AO3400A, Q4 AO3400A, Q5 AO3400A, U6 PCA9685

Commit message: Changed capacitor sizes
🟢 Group 1: 100% Safe to Shrink to 0603These capacitors handle logic-level decoupling or high-frequency filtering on your 3.3V and 5V lines. Because the capacitance values are low (1µF or less), an 0603 package can easily handle the DC bias without losing performance.All 0.1µF (100nF) Capacitors: You have 25 of these scattered across the board (e.g., C35, C41, C42, C49, C53-C61). Change every single one of these to 0603.The 1µF Logic Capacitors (C48, C62): C48 sits on the VCC pin of your battery charger. C62 is on the 3.3V rail for the USB hub. Change these to 0603.The 4.7µF Capacitors (C45, C47, C50): C45 and C47 sit on the 5V VL pin. C50 filters the 5V HDMI line. Change these to 0603.The 33pF Capacitors (C17, C18, C36): C17 and C18 are your crystal load capacitors and are already perfectly sized. C36 is a feedforward capacitor for your buck converter. Make sure all three are 0603.
🟡 Group 2: The "Compromise" - Shrink to 0805These 10µF capacitors sit on your 5V and 3.3V rails to smooth out the power for your motors, speakers, and USB hub (e.g., C1, C2, C4, C6, C12, C13, C15, C20, C22, C24).The Recommendation: While you have them listed as 1206, shrinking a 10µF ceramic capacitor all the way down to 0603 for a noisy 5V motor line will cause it to lose too much effective capacitance. 0805 is the perfect middle-ground here. It saves space but keeps your motor rails stable.
🔴 Group 3: DO NOT SHRINK (Keep 1206 / 1210 / 2824)These capacitors are exposed to the +VBATT_7V4 rail (up to 8.4V) or act as massive bulk storage. If you shrink these, your system will likely fail under heavy load.C32, C33, C34 (10µF): These connect directly to the high-voltage VIN pin of your main buck converter. Keep as 1206.C44 (22µF): This is the main switching capacitor for the battery charger inductor. Keep as 1210.C37, C38, C39, C40, C46 (22µF): These are the massive bulk output capacitors holding up your main 5V rail. Keep as 1210.C43 (1µF): Because this sits on the VH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
Parts:
- C1, C13, C15, C20, C22, C24: Digikey Link https://www.digikey.ca/en/products/detail/kemet/c1206c106k4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 -> https://www.digikey.ca/en/products/detail/samsung-electro-m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; Manufacturer KEMET -> Samsung Electro-Mechanics; Manufacturer Part C1206C106K4RACTU -> CL21B106KOQNNNE; Package 1206 (3216 Metric) -> 0805; Price 0.31 -> 0.22; Supplier P/N 399-C1206C106K4RACTUCT-ND -> 1276-2872-1-ND
- C10, C14, C19, C21, C23, C9: Digikey Link https://www.digikey.ca/en/products/detail/yageo/CC0805KRX7R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 -> https://www.digikey.ca/en/products/detail/yageo/CC0603KRX7R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; Manufacturer Part CC0805KRX7R9BB104 -> CC0603KRX7R9BB104; Package 0805 (2012 Metric) -> 0603 (1608 Metric); Supplier P/N 311-1140-1-ND -> 311-1344-1-ND
