File: 490_0/pwm_motors.kicad_sch (KiCad schematic)
At the start: 38 parts, among them J10 PAD, J4 PAD, J5 PAD, J6 PAD, J9 PAD, Q1 AO3400A, Q2 AO3400A, Q3 AO3400A, Q4 AO3400A, Q5 AO3400A, U6 PCA9685

Commit message: Assigned capacitor footprints
Parts:
- C1, C13, C15, C20, C22, C24: footprint Capacitor_SMD:C_1206_3216Metric -> Capacitor_SMD:C_0805_2012Metric
- C10, C14, C19, C21, C23, C9: footprint Capacitor_SMD:C_0805_2012Metric -> Capacitor_SMD:C_0603_1608Metric
Changed lines of the file:
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@@
 			)
 		)
-		(property "Footprint" "Capacitor_SMD:C_1206_3216Metric"
+		(property "Footprint" "Capacitor_SMD:C_0805_2012Metric"
 			(at 55.88 139.7 0)
 			(effects
@@
 			)
 		)
-		(property "Footprint" "Capacitor_SMD:C_0805_2012Metric"
+		(property "Footprint" "Capacitor_SMD:C_0603_1608Metric"
 			(at 33.02 88.9 0)
 			(effects
@@
 			)
 		)
-		(property "Footprint" "Capacitor_SMD:C_0805_2012Metric"
+		(property "Footprint" "Capacitor_SMD:C_0603_1608Metric"
 			(at 172.72 30.48 0)
 			(effects
@@
 			)
 		)
-		(property "Footprint" "Capacitor_SMD:C_1206_3216Metric"
+		(property "Footprint" "Capacitor_SMD:C_0805_2012Metric"
 			(at 40.64 88.9 0)
 			(effects
@@
 			)
 		)
-		(property "Footprint" "Capacitor_SMD:C_1206_3216Metric"
+		(property "Footprint" "Capacitor_SMD:C_0805_2012Metric"
 			(at 40.64 33.02 0)
 			(effects
@@
 			)
 		)
-		(property "Footprint" "Capacitor_SMD:C_0805_2012Metric"
+		(property "Footprint" "Capacitor_SMD:C_0603_1608Metric"
 			(at 33.02 33.02 0)
 			(effects
@@
 			)
 		)
-		(property "Footprint" "Capacitor_SMD:C_0805_2012Metric"
+		(property "Footprint" "Capacitor_SMD:C_0603_1608Metric"
 			(at 50.8 139.7 0)
 			(effects
@@
 			)
 		)
-		(property "Footprint" "Capacitor_SMD:C_1206_3216Metric"
+		(property "Footprint" "Capacitor_SMD:C_0805_2012Metric"
 			(at 111.76 86.36 0)
 			(effects
@@
 			)
 		)
-		(property "Footprint" "Capacitor_SMD:C_0805_2012Metric"
+		(property "Footprint" "Capacitor_SMD:C_0603_1608Metric"
 			(at 104.14 33.02 0)
 			(effects
@@
 			)
 		)
-		(property "Footprint" "Capacitor_SMD:C_1206_3216Metric"
+		(property "Footprint" "Capacitor_SMD:C_0805_2012Metric"
 			(at 111.76 33.02 0)
 			(effects
@@
 			)
 		)
-		(property "Footprint" "Capacitor_SMD:C_0805_2012Metric"
+		(property "Footprint" "Capacitor_SMD:C_0603_1608Metric"
 			(at 104.14 86.36 0)
 			(effects
@@
 			)
 		)
-		(property "Footprint" "Capacitor_SMD:C_1206_3216Metric"
+		(property "Footprint" "Capacitor_SMD:C_0805_2012Metric"
 			(at 180.34 30.48 0)
 			(effects

Commit message: Changed all the resistors to 0805 size
Parts:
- R12, R13, R14, R15, R16, R17, R18, R19, R20, R21: footprint Resistor_SMD:R_0603_1608Metric -> Resistor_SMD:R_0805_2012Metric
Changed lines of the file:
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@@
 			)
 		)
-		(property "Footprint" "Resistor_SMD:R_0603_1608Metric"
+		(property "Footprint" "Resistor_SMD:R_0805_2012Metric"
 			(at 120.65 104.902 90)
 			(effects
@@
 			)
 		)
-		(property "Footprint" "Resistor_SMD:R_0603_1608Metric"
+		(property "Footprint" "Resistor_SMD:R_0805_2012Metric"
 			(at 181.102 54.61 90)
 			(effects
@@
 			)
 		)
-		(property "Footprint" "Resistor_SMD:R_0603_1608Metric"
+		(property "Footprint" "Resistor_SMD:R_0805_2012Metric"
 			(at 112.522 57.15 90)
 			(effects
@@
 			)
 		)
-		(property "Footprint" "Resistor_SMD:R_0603_1608Metric"
+		(property "Footprint" "Resistor_SMD:R_0805_2012Metric"
 			(at 112.522 110.49 90)
 			(effects
@@
 			)
 		)
-		(property "Footprint" "Resistor_SMD:R_0603_1608Metric"
+		(property "Footprint" "Resistor_SMD:R_0805_2012Metric"
 			(at 49.53 51.562 90)
 			(effects
@@
 			)
 		)
-		(property "Footprint" "Resistor_SMD:R_0603_1608Metric"
+		(property "Footprint" "Resistor_SMD:R_0805_2012Metric"
 			(at 189.23 49.022 90)
 			(effects
@@
 			)
 		)
-		(property "Footprint" "Resistor_SMD:R_0603_1608Metric"
+		(property "Footprint" "Resistor_SMD:R_0805_2012Metric"
 			(at 41.402 113.03 90)
 			(effects
@@
 			)
 		)
-		(property "Footprint" "Resistor_SMD:R_0603_1608Metric"
+		(property "Footprint" "Resistor_SMD:R_0805_2012Metric"
 			(at 41.402 57.15 90)
 			(effects
@@
 			)
 		)
-		(property "Footprint" "Resistor_SMD:R_0603_1608Metric"
+		(property "Footprint" "Resistor_SMD:R_0805_2012Metric"
 			(at 49.53 107.442 90)
 			(effects
@@
 			)
 		)
-		(property "Footprint" "Resistor_SMD:R_0603_1608Metric"
+		(property "Footprint" "Resistor_SMD:R_0805_2012Metric"
 			(at 120.65 51.562 90)
 			(effects

Commit message: changed power and ground symbols for glasses
Connections:
- net +3.3V renamed +3.3V_GLASSES
- net +5V renamed +5V_GLASSES
- net GND renamed GND_GLASSES

Commit message: Generated BOM
Parts:
- J10, J4, J5, J6, J9: now in the parts list
Changed lines of the file:
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@@
 		(unit 1)
 		(exclude_from_sim no)
-		(in_bom no)
+		(in_bom yes)
 		(on_board yes)
 		(dnp no)
@@
 		(unit 1)
 		(exclude_from_sim no)
-		(in_bom no)
+		(in_bom yes)
 		(on_board yes)
 		(dnp no)
@@
 		(unit 1)
 		(exclude_from_sim no)
-		(in_bom no)
+		(in_bom yes)
 		(on_board yes)
 		(dnp no)
@@
 		(unit 1)
 		(exclude_from_sim no)
-		(in_bom no)
+		(in_bom yes)
 		(on_board yes)
 		(dnp no)
@@
 		(unit 1)
 		(exclude_from_sim no)
-		(in_bom no)
+		(in_bom yes)
 		(on_board yes)
 		(dnp no)

Commit message: ERC check fix
Connections:
- net GNDD renamed GND2

Commit message: Added side B for SW1
Parts:
- C1, C10, C13, C14, C15, C19, C20, C21, C22, C23, C24, C9: symbol PCM_Elektuur:C -> capstone_parts:C
- D5: symbol Device:D -> capstone_parts:D_2
- D6: symbol Device:D -> capstone_parts:D_1
- D7: symbol Device:D -> capstone_parts:D_3
- D8: symbol Device:D -> capstone_parts:D_4
- D9: symbol Device:D -> capstone_parts:D
- J10, J4, J5, J6, J9: symbol PCM_4ms_Connector:Conn_01x02 -> capstone_parts:Conn_01x02
- Q1, Q2, Q3, Q4, Q5: symbol Simulation_SPICE:NMOS -> capstone_parts:NMOS
- R12, R13, R14, R15, R16, R17, R18, R19, R20, R21: symbol Device:R -> capstone_parts:R
Connections:
- net GND2 is gone; now on net GND_GLASSES: C1.2 (-), C10.1 (+), C13.2 (-), C14.1 (+), C15.2 (-), C19.1 (+), C20.2 (-), C21.1 (+), C22.2 (-), C9.1 (+), Q1.3 (S), Q2.3 (S), Q3.3 (S), Q4.3 (S), Q5.3 (S), R15.2, R16.2, R17.2, R20.2, R21.2

Commit message: Friday, March 20th: PCB Final for BOM
Parts:
- D5, D6, D7, D8, D9: footprint *CapStone*:SODFL3816X120N -> capstone:SODFL3816X120N
- Q1, Q2, Q3, Q4, Q5: footprint *CapStone*:SOT95P280X125-3N -> capstone:SOT95P280X125-3N
- U6: footprint *CapStone*:TSSOP28_SOT361-1_NXP -> capstone:TSSOP28_SOT361-1_NXP
Connections:
- net +5V_GLASSES: now also D5.1 (K), D6.1 (C), D7.1 (K), D8.1 (K), D9.1 (K); no longer D5.C (K), D6.C, D7.C (K), D8.C (K), D9.C (K)
- net at J5.1 (Pin_1), Q1.1 (D): now also D5.2 (A); no longer D5.A
- net at J9.1 (Pin_1), Q5.1 (D): now also D9.2 (A); no longer D9.A
- net at J10.1 (Pin_1), Q4.1 (D): now also D8.2 (A); no longer D8.A
- net at J6.1 (Pin_1), Q2.1 (D): now also D6.2 (A); no longer D6.A
- net at J4.1 (Pin_1), Q3.1 (D): now also D7.2 (A); no longer D7.A
