File: 490_0/untitled.kicad_sch (KiCad schematic)
At the start: 31 parts, among them J2 PAD, J3 PAD, U16 SP3003-02XTG, U17 SP3003-02XTG, U4 USB2512B-I/M2, Y1 24M20P2/XT324-10/10

Commit message: Changed capacitor sizes
🟢 Group 1: 100% Safe to Shrink to 0603These capacitors handle logic-level decoupling or high-frequency filtering on your 3.3V and 5V lines. Because the capacitance values are low (1µF or less), an 0603 package can easily handle the DC bias without losing performance.All 0.1µF (100nF) Capacitors: You have 25 of these scattered across the board (e.g., C35, C41, C42, C49, C53-C61). Change every single one of these to 0603.The 1µF Logic Capacitors (C48, C62): C48 sits on the VCC pin of your battery charger. C62 is on the 3.3V rail for the USB hub. Change these to 0603.The 4.7µF Capacitors (C45, C47, C50): C45 and C47 sit on the 5V VL pin. C50 filters the 5V HDMI line. Change these to 0603.The 33pF Capacitors (C17, C18, C36): C17 and C18 are your crystal load capacitors and are already perfectly sized. C36 is a feedforward capacitor for your buck converter. Make sure all three are 0603.
🟡 Group 2: The "Compromise" - Shrink to 0805These 10µF capacitors sit on your 5V and 3.3V rails to smooth out the power for your motors, speakers, and USB hub (e.g., C1, C2, C4, C6, C12, C13, C15, C20, C22, C24).The Recommendation: While you have them listed as 1206, shrinking a 10µF ceramic capacitor all the way down to 0603 for a noisy 5V motor line will cause it to lose too much effective capacitance. 0805 is the perfect middle-ground here. It saves space but keeps your motor rails stable.
🔴 Group 3: DO NOT SHRINK (Keep 1206 / 1210 / 2824)These capacitors are exposed to the +VBATT_7V4 rail (up to 8.4V) or act as massive bulk storage. If you shrink these, your system will likely fail under heavy load.C32, C33, C34 (10µF): These connect directly to the high-voltage VIN pin of your main buck converter. Keep as 1206.C44 (22µF): This is the main switching capacitor for the battery charger inductor. Keep as 1210.C37, C38, C39, C40, C46 (22µF): These are the massive bulk output capacitors holding up your main 5V rail. Keep as 1210.C43 (1µF): Because this sits on the VH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
Parts:
- C53, C54, C56, C57, C58, C59, C60, C61: Digikey Link https://www.digikey.ca/en/products/detail/yageo/CC0805KRX7R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 -> https://www.digikey.ca/en/products/detail/yageo/CC0603KRX7R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; Manufacturer Part CC0805KRX7R9BB104 -> CC0603KRX7R9BB104; Package 0805 (2012 Metric) -> 0603 (1608 Metric); Supplier P/N 311-1140-1-ND -> 311-1344-1-ND
- C62: Digikey Link https://www.digikey.ca/en/products/detail/samsung-electro-m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 -> https://www.digikey.ca/en/products/detail/taiyo-yuden/UMK10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; Manufacturer Samsung Electro-Mechanics -> Taiyo Yuden; Manufacturer Part CL21B105KAFNNNE -> UMK107AB7105KA-T; Package 0805 -> 0603; Supplier P/N 1276-1066-1-ND -> 587-3247-1-ND
Changed lines of the file:
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@@
 			)
 		)
-		(property "Description" "CAP CER 0.1UF 50V X7R 0805"
+		(property "Description" "CAP CER 0.1UF 50V X7R 0603"
 			(at 177.8 88.9 0)
 			(effects
@@
 			)
 		)
-		(property "Digikey Link" "https://www.digikey.ca/en/products/detail/yageo/CC0805KRX7R9BB104/302874?s=N4IgTCBcDaIMJwAwA5EFYDSAlAGgdiwE4AhYgRkQBYQBdAXyA"
+		(property "Digikey Link" "https://www.digikey.ca/en/products/detail/yageo/CC0603KRX7R9BB104/2103082"
 			(at 177.8 88.9 0)
 			(effects
@@
 			)
 		)
-		(property "Manufacturer Part" "CC0805KRX7R9BB104"
+		(property "Manufacturer Part" "CC0603KRX7R9BB104"
 			(at 177.8 88.9 0)
 			(effects
@@
 			)
 		)
-		(property "Package" "0805 (2012 Metric)"
+		(property "Package" "0603 (1608 Metric)"
 			(at 177.8 88.9 0)
 			(effects
@@
 			)
 		)
-		(property "Supplier P/N" "311-1140-1-ND"
+		(property "Supplier P/N" "311-1344-1-ND"
 			(at 177.8 88.9 0)
 			(effects
@@
 			)
 		)
-		(property "Description" "CAP CER 0.1UF 50V X7R 0805"
+		(property "Description" "CAP CER 0.1UF 50V X7R 0603"
 			(at 88.9 88.9 0)
 			(effects
@@
 			)
 		)
-		(property "Digikey Link" "https://www.digikey.ca/en/products/detail/yageo/CC0805KRX7R9BB104/302874?s=N4IgTCBcDaIMJwAwA5EFYDSAlAGgdiwE4AhYgRkQBYQBdAXyA"
+		(property "Digikey Link" "https://www.digikey.ca/en/products/detail/yageo/CC0603KRX7R9BB104/2103082"
 			(at 88.9 88.9 0)
 			(effects
@@
 			)
 		)
-		(property "Manufacturer Part" "CC0805KRX7R9BB104"
+		(property "Manufacturer Part" "CC0603KRX7R9BB104"
 			(at 88.9 88.9 0)
 			(effects
@@
 			)
 		)
-		(property "Package" "0805 (2012 Metric)"
+		(property "Package" "0603 (1608 Metric)"
 			(at 88.9 88.9 0)
 			(effects
@@
 			)
 		)
-		(property "Supplier P/N" "311-1140-1-ND"
+		(property "Supplier P/N" "311-1344-1-ND"
 			(at 88.9 88.9 0)
 			(effects
@@
 			)
 		)
-		(property "Datasheet" "kicad-embed://CL21B105KAFNNNE_Spec.pdf"
+		(property "Datasheet" "kicad-embed://UMK107AB7105KA-T_SS.pdf"
 			(at 53.34 88.9 0)
 			(effects
@@
 			)
 		)
-		(property "Description" "1 µF ±10% 25V Ceramic Capacitor X7R 0805 (2012 Metric)"
+		(property "Description" "CAP CER 1UF 50V X7R 0603"
 			(at 53.34 88.9 0)
 			(effects
@@
 			)
 		)
-		(property "Digikey Link" "https://www.digikey.ca/en/products/detail/samsung-electro-mechanics/CL21B105KAFNNNE/3886724"
+		(property "Digikey Link" "https://www.digikey.ca/en/products/detail/taiyo-yuden/UMK107AB7105KA-T/3660085"
 			(at 53.34 88.9 0)
 			(effects
@@
 			)
 		)
-		(property "Manufacturer" "Samsung Electro-Mechanics"
+		(property "Manufacturer" "Taiyo Yuden"
 			(at 53.34 88.9 0)
 			(effects
@@
 			)
 		)
-		(property "Manufacturer Part" "CL21B105KAFNNNE"
+		(property "Manufacturer Part" "UMK107AB7105KA-T"
 			(at 53.34 88.9 0)
 			(effects
@@
 			)
 		)
-		(property "Package" "0805"
+		(property "Package" "0603"
 			(at 53.34 88.9 0)
 			(effects
@@
 			)
 		)
-		(property "Supplier P/N" "1276-1066-1-ND"
+		(property "Supplier P/N" "587-3247-1-ND"
 			(at 53.34 88.9 0)
 			(effects
@@
 			)
 		)
-		(property "Description" "CAP CER 0.1UF 50V X7R 0805"
+		(property "Description" "CAP CER 0.1UF 50V X7R 0603"
 			(at 81.28 142.24 0)
 			(effects
@@
 			)
 		)
-		(property "Digikey Link" "https://www.digikey.ca/en/products/detail/yageo/CC0805KRX7R9BB104/302874?s=N4IgTCBcDaIMJwAwA5EFYDSAlAGgdiwE4AhYgRkQBYQBdAXyA"
+		(property "Digikey Link" "https://www.digikey.ca/en/products/detail/yageo/CC0603KRX7R9BB104/2103082"
 			(at 81.28 142.24 0)
 			(effects
@@
 			)
 		)
-		(property "Manufacturer Part" "CC0805KRX7R9BB104"
+		(property "Manufacturer Part" "CC0603KRX7R9BB104"
 			(at 81.28 142.24 0)
 			(effects
@@
 			)
 		)
-		(property "Supplier P/N" "311-1140-1-ND"
+		(property "Supplier P/N" "311-1344-1-ND"
 			(at 81.28 142.24 0)
 			(effects
@@
 			)
 		)
-		(property "Package" "0805 (2012 Metric)"
+		(property "Package" "0603 (1608 Metric)"
 			(at 81.28 142.24 90)
 			(effects
@@
 			)
 		)
-		(property "Description" "CAP CER 0.1UF 50V X7R 0805"
+		(property "Description" "CAP CER 0.1UF 50V X7R 0603"
 			(at 66.04 78.74 0)
 			(effects
@@
 			)
 		)
-		(property "Digikey Link" "https://www.digikey.ca/en/products/detail/yageo/CC0805KRX7R9BB104/302874?s=N4IgTCBcDaIMJwAwA5EFYDSAlAGgdiwE4AhYgRkQBYQBdAXyA"
+		(property "Digikey Link" "https://www.digikey.ca/en/products/detail/yageo/CC0603KRX7R9BB104/2103082"
 			(at 66.04 78.74 0)
 			(effects
@@
 			)
 		)
-		(property "Manufacturer Part" "CC0805KRX7R9BB104"
+		(property "Manufacturer Part" "CC0603KRX7R9BB104"
 			(at 66.04 78.74 0)
 			(effects
@@
 			)
 		)
-		(property "Package" "0805 (2012 Metric)"
+		(property "Package" "0603 (1608 Metric)"
 			(at 66.04 78.74 0)
 			(effects
@@
 			)
 		)
-		(property "Supplier P/N" "311-1140-1-ND"
+		(property "Supplier P/N" "311-1344-1-ND"
 			(at 66.04 78.74 0)
 			(effects
@@
 			)
 		)
-		(property "Description" "CAP CER 0.1UF 50V X7R 0805"
+		(property "Description" "CAP CER 0.1UF 50V X7R 0603"
 			(at 81.28 137.16 0)
 			(effects
@@
 			)
 		)
-		(property "Digikey Link" "https://www.digikey.ca/en/products/detail/yageo/CC0805KRX7R9BB104/302874?s=N4IgTCBcDaIMJwAwA5EFYDSAlAGgdiwE4AhYgRkQBYQBdAXyA"
+		(property "Digikey Link" "https://www.digikey.ca/en/products/detail/yageo/CC0603KRX7R9BB104/2103082"
 			(at 81.28 137.16 0)
 			(effects
@@
 			)
 		)
-		(property "Manufacturer Part" "CC0805KRX7R9BB104"
+		(property "Manufacturer Part" "CC0603KRX7R9BB104"
 			(at 81.28 137.16 0)
 			(effects
@@
 			)
 		)
-		(property "Supplier P/N" "311-1140-1-ND"
+		(property "Supplier P/N" "311-1344-1-ND"
 			(at 81.28 137.16 0)
 			(effects
@@
 			)
 		)
-		(property "Package" "0805 (2012 Metric)"
+		(property "Package" "0603 (1608 Metric)"
 			(at 81.28 137.16 90)
 			(effects
@@
 			)
 		)
-		(property "Description" "CAP CER 0.1UF 50V X7R 0805"
+		(property "Description" "CAP CER 0.1UF 50V X7R 0603"
 			(at 73.66 88.9 0)
 			(effects
@@
 			)
 		)
-		(property "Digikey Link" "https://www.digikey.ca/en/products/detail/yageo/CC0805KRX7R9BB104/302874?s=N4IgTCBcDaIMJwAwA5EFYDSAlAGgdiwE4AhYgRkQBYQBdAXyA"
+		(property "Digikey Link" "https://www.digikey.ca/en/products/detail/yageo/CC0603KRX7R9BB104/2103082"
 			(at 73.66 88.9 0)
 			(effects
@@
 			)
 		)
-		(property "Manufacturer Part" "CC0805KRX7R9BB104"
+		(property "Manufacturer Part" "CC0603KRX7R9BB104"
 			(at 73.66 88.9 0)
 			(effects
@@
 			)
 		)
-		(property "Package" "0805 (2012 Metric)"
+		(property "Package" "0603 (1608 Metric)"
 			(at 73.66 88.9 0)
 			(effects
@@
 			)
 		)
-		(property "Supplier P/N" "311-1140-1-ND"
+		(property "Supplier P/N" "311-1344-1-ND"
 			(at 73.66 88.9 0)
 			(effects
@@
 			)
 		)
-		(property "Description" "CAP CER 0.1UF 50V X7R 0805"
+		(property "Description" "CAP CER 0.1UF 50V X7R 0603"
 			(at 185.42 78.74 0)
 			(effects
@@
 			)
 		)
-		(property "Digikey Link" "https://www.digikey.ca/en/products/detail/yageo/CC0805KRX7R9BB104/302874?s=N4IgTCBcDaIMJwAwA5EFYDSAlAGgdiwE4AhYgRkQBYQBdAXyA"
+		(property "Digikey Link" "https://www.digikey.ca/en/products/detail/yageo/CC0603KRX7R9BB104/2103082"
 			(at 185.42 78.74 0)
 			(effects
@@
 			)
 		)
-		(property "Manufacturer Part" "CC0805KRX7R9BB104"
+		(property "Manufacturer Part" "CC0603KRX7R9BB104"
 			(at 185.42 78.74 0)
 			(effects
@@
 			)
 		)
-		(property "Package" "0805 (2012 Metric)"
+		(property "Package" "0603 (1608 Metric)"
 			(at 185.42 78.74 0)
 			(effects
@@
 			)
 		)
-		(property "Supplier P/N" "311-1140-1-ND"
+		(property "Supplier P/N" "311-1344-1-ND"
 			(at 185.42 78.74 0)
 			(effects
@@
 			)
 		)
-		(property "Description" "CAP CER 0.1UF 50V X7R 0805"
+		(property "Description" "CAP CER 0.1UF 50V X7R 0603"
 			(at 81.28 78.74 0)
 			(effects
@@
 			)
 		)
-		(property "Digikey Link" "https://www.digikey.ca/en/products/detail/yageo/CC0805KRX7R9BB104/302874?s=N4IgTCBcDaIMJwAwA5EFYDSAlAGgdiwE4AhYgRkQBYQBdAXyA"
+		(property "Digikey Link" "https://www.digikey.ca/en/products/detail/yageo/CC0603KRX7R9BB104/2103082"
 			(at 81.28 78.74 0)
 			(effects
@@
 			)
 		)
-		(property "Manufacturer Part" "CC0805KRX7R9BB104"
+		(property "Manufacturer Part" "CC0603KRX7R9BB104"
 			(at 81.28 78.74 0)
 			(effects
@@
 			)
 		)
-		(property "Package" "0805 (2012 Metric)"
+		(property "Package" "0603 (1608 Metric)"
 			(at 81.28 78.74 0)
 			(effects
@@
 			)
 		)
-		(property "Supplier P/N" "311-1140-1-ND"
+		(property "Supplier P/N" "311-1344-1-ND"
 			(at 81.28 78.74 0)
 			(effects

Commit message: Assigned capacitor footprints
Parts:
- C53, C54, C56, C57, C58, C59, C60, C61, C62: footprint Capacitor_SMD:C_0805_2012Metric -> Capacitor_SMD:C_0603_1608Metric
Changed lines of the file:
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@@
 			)
 		)
-		(property "Footprint" "Capacitor_SMD:C_0805_2012Metric"
+		(property "Footprint" "Capacitor_SMD:C_0603_1608Metric"
 			(at 177.8 88.9 0)
 			(effects
@@
 			)
 		)
-		(property "Footprint" "Capacitor_SMD:C_0805_2012Metric"
+		(property "Footprint" "Capacitor_SMD:C_0603_1608Metric"
 			(at 88.9 88.9 0)
 			(effects
@@
 			)
 		)
-		(property "Footprint" "Capacitor_SMD:C_0805_2012Metric"
+		(property "Footprint" "Capacitor_SMD:C_0603_1608Metric"
 			(at 53.34 88.9 0)
 			(effects
@@
 			)
 		)
-		(property "Footprint" "Capacitor_SMD:C_0805_2012Metric"
+		(property "Footprint" "Capacitor_SMD:C_0603_1608Metric"
 			(at 81.28 142.24 0)
 			(effects
@@
 			)
 		)
-		(property "Footprint" "Capacitor_SMD:C_0805_2012Metric"
+		(property "Footprint" "Capacitor_SMD:C_0603_1608Metric"
 			(at 66.04 78.74 0)
 			(effects
@@
 			)
 		)
-		(property "Footprint" "Capacitor_SMD:C_0805_2012Metric"
+		(property "Footprint" "Capacitor_SMD:C_0603_1608Metric"
 			(at 81.28 137.16 0)
 			(effects
@@
 			)
 		)
-		(property "Footprint" "Capacitor_SMD:C_0805_2012Metric"
+		(property "Footprint" "Capacitor_SMD:C_0603_1608Metric"
 			(at 73.66 88.9 0)
 			(effects
@@
 			)
 		)
-		(property "Footprint" "Capacitor_SMD:C_0805_2012Metric"
+		(property "Footprint" "Capacitor_SMD:C_0603_1608Metric"
 			(at 185.42 78.74 0)
 			(effects
@@
 			)
 		)
-		(property "Footprint" "Capacitor_SMD:C_0805_2012Metric"
+		(property "Footprint" "Capacitor_SMD:C_0603_1608Metric"
 			(at 81.28 78.74 0)
 			(effects
