File: 490_0/untitled.kicad_sch (KiCad schematic)
At the start: 32 parts, among them J2 PAD, J3 PAD, U16 SP3003-02XTG, U17 SP3003-02XTG, U4 USB2512B-I/M2, Y1 24M20P2/XT324-10/10

Commit message: Tuesday March 10th: 13:25
Connections:
- net D1+: now also U16.5; no longer U16.4
- net D1-: now also U16.4; no longer U16.5
- net D2+: now also J3.2 (Pin_2), U17.5; no longer J3.3 (Pin_3), U17.4
- net D2-: now also J3.3 (Pin_3), U17.4; no longer J3.2 (Pin_2), U17.5
- net GND_GLASSES: now also J3.1 (Pin_1); no longer J3.4 (Pin_4)
- net VBUS2: now also J3.4 (Pin_4); no longer J3.1 (Pin_1)
Changed lines of the file:
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@@
 	)
 	(label "D2-"
-		(at 63.5 15.24 0)
+		(at 73.66 15.24 0)
 		(effects
 			(font
@@
 	)
 	(label "D1+"
-		(at 30.48 15.24 0)
+		(at 20.32 15.24 0)
 		(effects
 			(font
@@
 	)
 	(label "D1-"
-		(at 20.32 15.24 0)
+		(at 30.48 15.24 0)
 		(effects
 			(font
@@
 	)
 	(label "D2+"
-		(at 73.66 15.24 0)
+		(at 63.5 15.24 0)
 		(effects
 			(font
@@
 	(symbol
 		(lib_id "capstone_parts:Conn_01x04_P2.54mm")
-		(at 231.14 144.78 0)
+		(at 231.14 147.32 0)
+		(mirror x)
 		(unit 1)
 		(exclude_from_sim no)
@@
 		(on_board yes)
 		(dnp no)
-		(fields_autoplaced yes)
 		(property "Reference" "J3"
-			(at 233.68 144.7799 0)
+			(at 233.68 147.3201 0)
 			(effects
 				(font
@@
 		)
 		(property "Value" "PAD"
-			(at 233.68 147.3199 0)
+			(at 233.68 144.7801 0)
 			(effects
 				(font
@@
 		)
 		(property "Footprint" "Connector_PinHeader_1.27mm:PinHeader_1x04_P1.27mm_Vertical"
-			(at 231.14 154.94 0)
+			(at 231.14 137.16 0)
 			(effects
 				(font
@@
 		)
 		(property "Datasheet" "kicad-embed://ePA-F.pdf"
-			(at 231.14 157.48 0)
+			(at 231.14 134.62 0)
 			(effects
 				(font
@@
 		)
 		(property "Description" "CONN HEADER SMD 4POS 2MM"
-			(at 231.14 160.02 0)
+			(at 231.14 132.08 0)
 			(effects
 				(font
@@
 		)
 		(property "AVAILABILITY" ""
-			(at 231.14 144.78 0)
+			(at 231.14 147.32 0)
 			(effects
 				(font
@@
 		)
 		(property "PACKAGE" ""
-			(at 231.14 144.78 0)
+			(at 231.14 147.32 0)
 			(effects
 				(font
@@
 		)
 		(property "PRICE" ""
-			(at 231.14 144.78 0)
+			(at 231.14 147.32 0)
 			(effects
 				(font
@@
 		)
 		(property "Digikey Link" "https://www.digikey.com/en/products/detail/jst-sales-america-inc/BM04B-PASS-1-TFT/2773434"
-			(at 231.14 144.78 0)
+			(at 231.14 147.32 0)
 			(effects
 				(font
@@
 		)
 		(property "Manufacturer" "JST Sales America Inc."
-			(at 231.14 144.78 0)
+			(at 231.14 147.32 0)
 			(effects
 				(font
@@
 		)
 		(property "Manufacturer Part" "BM04B-PASS-1-TFT"
-			(at 231.14 144.78 0)
+			(at 231.14 147.32 0)
 			(effects
 				(font
@@
 		)
 		(property "Price" "0.71"
-			(at 231.14 144.78 0)
+			(at 231.14 147.32 0)
 			(effects
 				(font
@@
 		)
 		(property "Supplier" "DigiKey"
-			(at 231.14 144.78 0)
+			(at 231.14 147.32 0)
 			(effects
 				(font
@@
 		)
 		(property "Supplier P/N" "455-BM04B-PASS-1-TFTCT-ND"
-			(at 231.14 144.78 0)
+			(at 231.14 147.32 0)
 			(effects
 				(font
@@
 		)
 		(property "Type" "SMD"
-			(at 231.14 144.78 0)
+			(at 231.14 147.32 0)
 			(effects
 				(font
@@
 		)
 		(property "Unit" "pcs"
-			(at 231.14 144.78 0)
+			(at 231.14 147.32 0)
 			(effects
 				(font
@@
 		)
 		(property "Voltage Raing" ""
-			(at 231.14 144.78 0)
+			(at 231.14 147.32 0)
 			(effects
 				(font
@@
 		)
 		(property "Voltage Rating" ""
-			(at 231.14 144.78 0)
+			(at 231.14 147.32 0)
 			(effects
 				(font
@@
 		(on_board yes)
 		(dnp no)
-		(fields_autoplaced yes)
 		(property "Reference" "J2"
 			(at 233.68 114.2999 0)

Commit message: Friday, March 20th: PCB Final for BOM
Parts:
- U16, U17: footprint *CapStone*:SOT553_LTF_SP3003_02XTG -> capstone:SOT553_LTF_SP3003_02XTG
- U4: footprint *CapStone*:SQFN36_M2_MCH_USB2512B_I_M2 -> capstone:SQFN36_M2_MCH_USB2512B_I_M2
