File: 490_0/TOF_HDMI_CONNECTOR_PCB1.kicad_sch (KiCad schematic)
At the start: 4 parts, among them J12 2000-1-1-20-00-BK

Commit message: Footprint Update
1st half of footprints updated
Parts:
- CR7: footprint MSOP10_MO-187_LTF -> *CapStone*:MSOP10_MO-187_LTF
- D21, D24: footprint PCM_Diode_SMD_AKL:D_SOD-123F -> Diode_SMD:D_SOD-123F
- J12: footprint (none) -> *CapStone*:CNCTECH_2000-1-1-20-00-BK
Changed lines of the file:
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@@
 			)
 		)
-		(property "Footprint" ""
+		(property "Footprint" "*CapStone*:CNCTECH_2000-1-1-20-00-BK"
 			(at 80.645 81.28 0)
 			(effects
@@
 			)
 		)
-		(property "Footprint" "PCM_Diode_SMD_AKL:D_SOD-123F"
+		(property "Footprint" "Diode_SMD:D_SOD-123F"
 			(at 132.08 101.6 0)
 			(effects
@@
 			)
 		)
-		(property "Footprint" "MSOP10_MO-187_LTF"
+		(property "Footprint" "*CapStone*:MSOP10_MO-187_LTF"
 			(at 187.96 99.06 0)
 			(effects
@@
 			)
 		)
-		(property "Footprint" "PCM_Diode_SMD_AKL:D_SOD-123F"
+		(property "Footprint" "Diode_SMD:D_SOD-123F"
 			(at 200.66 100.33 0)
 			(effects

Commit message: March 3rd
Parts:
- removed CR7: SP3003-08ATG, *CapStone*:MSOP10_MO-187_LTF, symbol capstone_parts:SP3003-08ATG
- added U18: TPD8S009DSMR, *CapStone*:TPD8S009DSMR, symbol capstone_parts:TPD8S009DSMR
Connections:
- net +3.3V: now also U18.13 (VCC), U18.15 (VCC)
- net CLK+: now also U18.7 (D2+)
- net CLK-: now also U18.9 (D2-)
- net D0+: now also U18.1 (D0+)
- net D0-: now also U18.3 (D0-)
- net D1+: now also U18.4 (D1+)
- net D1-: now also U18.6 (D1-)
- net GND: now also J12.SH1, J12.SH2, J12.SH3, J12.SH4, U18.11 (GND), U18.2 (GND), U18.5 (GND), U18.8 (GND); no longer J12.SH
- net SCL: now also U18.10 (D3+)
- net SDA: now also U18.12 (D3-)
- no-connect marks 4 -> 5
