File: 490_0/board_connector_a.kicad_sch (KiCad schematic)
At the start: 14 parts, among them J16 DF40HC(3.0)-100DS-0.4V(58), J17 DF40HC(3.0)-100DS-0.4V(58), J21 TS-102-G-A, Q6 BSS84, SW2 TL1105LF160Q, SW3 TL1105LF160Q, SW4 TL1105LF160Q, SW5 TL1105LF160Q, SW6 TL1105LF160Q, SW7 TL1105LF160Q

Commit message: Footprint Update #2
All footprints except for the capacitors have been attributed
Parts:
- Q6: footprint (none) -> *CapStone*:SOT95P240X120-3N
- R37, R44: footprint (none) -> Resistor_SMD:R_0603_1608Metric
- SW2, SW3, SW4, SW5, SW6, SW7: footprint (none) -> *CapStone*:SW_TL1105LF160Q
Changed lines of the file:
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@@
 			)
 		)
-		(property "Footprint" ""
+		(property "Footprint" "*CapStone*:SOT95P240X120-3N"
 			(at 66.04 165.1 0)
 			(effects
@@
 			)
 		)
-		(property "Footprint" ""
+		(property "Footprint" "*CapStone*:SW_TL1105LF160Q"
 			(at 35.56 93.98 0)
 			(effects
@@
 			)
 		)
-		(property "Footprint" ""
+		(property "Footprint" "*CapStone*:SW_TL1105LF160Q"
 			(at 177.8 86.36 0)
 			(effects
@@
 			)
 		)
-		(property "Footprint" ""
+		(property "Footprint" "*CapStone*:SW_TL1105LF160Q"
 			(at 177.8 74.93 0)
 			(effects
@@
 			)
 		)
-		(property "Footprint" ""
+		(property "Footprint" "Resistor_SMD:R_0603_1608Metric"
 			(at 70.358 173.99 90)
 			(effects
@@
 			)
 		)
-		(property "Footprint" ""
+		(property "Footprint" "*CapStone*:SW_TL1105LF160Q"
 			(at 35.56 72.39 0)
 			(effects
@@
 			)
 		)
-		(property "Footprint" ""
+		(property "Footprint" "Resistor_SMD:R_0603_1608Metric"
 			(at 85.598 35.56 90)
 			(effects
@@
 			)
 		)
-		(property "Footprint" ""
+		(property "Footprint" "*CapStone*:SW_TL1105LF160Q"
 			(at 177.8 96.52 0)
 			(effects
@@
 			)
 		)
-		(property "Footprint" ""
+		(property "Footprint" "*CapStone*:SW_TL1105LF160Q"
 			(at 35.56 83.82 0)
 			(effects

Commit message: March 3rd
Parts:
- D16: value LED -> LTST-C170GKT
- D17: value LED -> LTST-C170KRKT
- R37, R44: footprint Resistor_SMD:R_0603_1608Metric -> Resistor_SMD:R_0805_2012Metric
Changed lines of the file:
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@@
 	(text "This LED flashes when the CM4 is reading from or writing to the eMMC or SD card."
 		(exclude_from_sim no)
-		(at 59.944 45.974 0)
+		(at 44.704 49.276 0)
 		(effects
 			(font
@@
 		(on_board yes)
 		(dnp no)
-		(fields_autoplaced yes)
 		(property "Reference" "D16"
-			(at 87.63 46.0374 90)
+			(at 73.152 44.958 90)
 			(effects
 				(font
@@
 			)
 		)
-		(property "Value" "LED"
-			(at 87.63 48.5774 90)
+		(property "Value" "LTST-C170GKT"
+			(at 68.072 47.498 90)
 			(effects
 				(font
@@
 			)
 		)
-		(property "Footprint" "Resistor_SMD:R_0603_1608Metric"
+		(property "Footprint" "Resistor_SMD:R_0805_2012Metric"
 			(at 70.358 173.99 90)
 			(effects
@@
 			)
 		)
-		(property "Footprint" "Resistor_SMD:R_0603_1608Metric"
+		(property "Footprint" "Resistor_SMD:R_0805_2012Metric"
 			(at 85.598 35.56 90)
 			(effects
@@
 			)
 		)
-		(property "Value" "LED"
+		(property "Value" "LTST-C170KRKT"
 			(at 72.39 187.0074 90)
 			(effects
