File: 490_0/powerport.kicad_sch (KiCad schematic)
At the start: 5 parts, among them J18 TS-103-G-A, J7 629105150521, U5 TS3USB221AQRSERQ1

Commit message: March 3rd
Parts:
- C6: footprint (none) -> Capacitor_SMD:C_0805_2012Metric; Digikey Link https://www.digikey.ca/en/products/detail/kemet/c1206c106k4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 -> https://www.digikey.ca/en/products/detail/samsung-electro-m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; Manufacturer KEMET -> Samsung Electro-Mechanics; Manufacturer Part C1206C106K4RACTU -> CL21B106KOQNNNE; Package 1206 (3216 Metric) -> 0805; Price 0.31 -> 0.22; Supplier P/N 399-C1206C106K4RACTUCT-ND -> 1276-2872-1-ND
- renumbered CR3 to U11
Changed lines of the file:
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@@
 	)
 	(hierarchical_label "USBhub_P"
-		(shape input)
+		(shape bidirectional)
 		(at 165.1 88.9 180)
 		(effects
@@
 	)
 	(hierarchical_label "USB_N"
-		(shape output)
+		(shape bidirectional)
 		(at 226.06 91.44 0)
 		(effects
@@
 	)
 	(hierarchical_label "USB_P"
-		(shape output)
+		(shape bidirectional)
 		(at 226.06 88.9 0)
 		(effects
@@
 	)
 	(hierarchical_label "USBhub_N"
-		(shape input)
+		(shape bidirectional)
 		(at 165.1 91.44 180)
 		(effects
@@
 			)
 		)
-		(property "Footprint" ""
-			(at 109.22 71.12 0)
-			(effects
-				(font
-					(size 1.27 1.27)
-				)
-				(hide yes)
-			)
-		)
-		(property "Datasheet" "kicad-embed://KEM_C1002_X7R_SMD.pdf"
-			(at 109.22 71.12 0)
-			(effects
-				(font
-					(size 1.27 1.27)
-				)
-				(hide yes)
-			)
-		)
-		(property "Description" "CAP CER 10UF 16V X7R 1206"
+		(property "Footprint" "Capacitor_SMD:C_0805_2012Metric"
+			(at 109.22 71.12 0)
+			(effects
+				(font
+					(size 1.27 1.27)
+				)
+				(hide yes)
+			)
+		)
+		(property "Datasheet" "kicad-embed://CL_Series_MLCC_ds.pdf"
+			(at 109.22 71.12 0)
+			(effects
+				(font
+					(size 1.27 1.27)
+				)
+				(hide yes)
+			)
+		)
+		(property "Description" "CAP CER 10UF 16V X7R 0805"
 			(at 109.22 71.12 0)
 			(effects
@@
 			)
 		)
-		(property "Digikey Link" "https://www.digikey.ca/en/products/detail/kemet/c1206c106k4ractu/789657"
+		(property "Digikey Link" "https://www.digikey.ca/en/products/detail/samsung-electro-mechanics/CL21B106KOQNNNE/3888530"
 			(at 109.22 71.12 0)
 			(effects
@@
 			)
 		)
-		(property "Manufacturer" "KEMET"
+		(property "Manufacturer" "Samsung Electro-Mechanics"
 			(at 109.22 71.12 0)
 			(effects
@@
 			)
 		)
-		(property "Manufacturer Part" "C1206C106K4RACTU"
+		(property "Manufacturer Part" "CL21B106KOQNNNE"
 			(at 109.22 71.12 0)
 			(effects
@@
 			)
 		)
-		(property "Supplier P/N" "399-C1206C106K4RACTUCT-ND"
+		(property "Supplier P/N" "1276-2872-1-ND"
 			(at 109.22 71.12 0)
 			(effects
@@
 			)
 		)
-		(property "Package" "1206 (3216 Metric)"
-			(at 109.22 71.12 0)
-			(effects
-				(font
-					(size 1.27 1.27)
-				)
-				(hide yes)
-			)
-		)
-		(property "Price" "0.31"
+		(property "Package" "0805"
+			(at 109.22 71.12 0)
+			(effects
+				(font
+					(size 1.27 1.27)
+				)
+				(hide yes)
+			)
+		)
+		(property "Price" "0.22"
 			(at 109.22 71.12 0)
 			(effects
@@
 		(dnp no)
 		(fields_autoplaced yes)
-		(property "Reference" "CR3"
+		(property "Reference" "U11"
 			(at 151.13 102.8699 90)
 			(effects
@@
 			(project "490_0"
 				(path "/365a82ed-827d-43e1-aa2f-b98221c4179c/f9f22bb2-829e-4ff5-89be-c4b5e2122135/d28f2748-3083-434f-ab92-5f07809e59a3"
-					(reference "CR3")
+					(reference "U11")
 					(unit 1)
 				)
