File: 490_0/powerport.kicad_sch (KiCad schematic)
At the start: 5 parts, among them J18 TS-103-G-A, J7 629105150521, U5 TS3USB221AQRSERQ1

Commit message: LED names + 5V routing through ESD + renamed ESD chips to "U"
Parts:
- renumbered CR3 to U11
Changed lines of the file:
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@@
 		(dnp no)
 		(fields_autoplaced yes)
-		(property "Reference" "CR3"
+		(property "Reference" "U11"
 			(at 151.13 102.8699 90)
 			(effects
@@
 			(project "490_0"
 				(path "/365a82ed-827d-43e1-aa2f-b98221c4179c/f9f22bb2-829e-4ff5-89be-c4b5e2122135/d28f2748-3083-434f-ab92-5f07809e59a3"
-					(reference "CR3")
+					(reference "U11")
 					(unit 1)
 				)

Commit message: PCB Jumpstart
Changed lines of the file:
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@@
 	)
 	(hierarchical_label "USBhub_P"
-		(shape input)
+		(shape bidirectional)
 		(at 165.1 88.9 180)
 		(effects
@@
 	)
 	(hierarchical_label "USB_N"
-		(shape output)
+		(shape bidirectional)
 		(at 226.06 91.44 0)
 		(effects
@@
 	)
 	(hierarchical_label "USB_P"
-		(shape output)
+		(shape bidirectional)
 		(at 226.06 88.9 0)
 		(effects
@@
 	)
 	(hierarchical_label "USBhub_N"
-		(shape input)
+		(shape bidirectional)
 		(at 165.1 91.44 180)
 		(effects

Commit message: Changed capacitor sizes
🟢 Group 1: 100% Safe to Shrink to 0603These capacitors handle logic-level decoupling or high-frequency filtering on your 3.3V and 5V lines. Because the capacitance values are low (1µF or less), an 0603 package can easily handle the DC bias without losing performance.All 0.1µF (100nF) Capacitors: You have 25 of these scattered across the board (e.g., C35, C41, C42, C49, C53-C61). Change every single one of these to 0603.The 1µF Logic Capacitors (C48, C62): C48 sits on the VCC pin of your battery charger. C62 is on the 3.3V rail for the USB hub. Change these to 0603.The 4.7µF Capacitors (C45, C47, C50): C45 and C47 sit on the 5V VL pin. C50 filters the 5V HDMI line. Change these to 0603.The 33pF Capacitors (C17, C18, C36): C17 and C18 are your crystal load capacitors and are already perfectly sized. C36 is a feedforward capacitor for your buck converter. Make sure all three are 0603.
🟡 Group 2: The "Compromise" - Shrink to 0805These 10µF capacitors sit on your 5V and 3.3V rails to smooth out the power for your motors, speakers, and USB hub (e.g., C1, C2, C4, C6, C12, C13, C15, C20, C22, C24).The Recommendation: While you have them listed as 1206, shrinking a 10µF ceramic capacitor all the way down to 0603 for a noisy 5V motor line will cause it to lose too much effective capacitance. 0805 is the perfect middle-ground here. It saves space but keeps your motor rails stable.
🔴 Group 3: DO NOT SHRINK (Keep 1206 / 1210 / 2824)These capacitors are exposed to the +VBATT_7V4 rail (up to 8.4V) or act as massive bulk storage. If you shrink these, your system will likely fail under heavy load.C32, C33, C34 (10µF): These connect directly to the high-voltage VIN pin of your main buck converter. Keep as 1206.C44 (22µF): This is the main switching capacitor for the battery charger inductor. Keep as 1210.C37, C38, C39, C40, C46 (22µF): These are the massive bulk output capacitors holding up your main 5V rail. Keep as 1210.C43 (1µF): Because this sits on the VH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
Parts:
- C6: Digikey Link https://www.digikey.ca/en/products/detail/kemet/c1206c106k4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 -> https://www.digikey.ca/en/products/detail/samsung-electro-m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; Manufacturer KEMET -> Samsung Electro-Mechanics; Manufacturer Part C1206C106K4RACTU -> CL21B106KOQNNNE; Package 1206 (3216 Metric) -> 0805; Price 0.31 -> 0.22; Supplier P/N 399-C1206C106K4RACTUCT-ND -> 1276-2872-1-ND
Changed lines of the file:
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@@
 			)
 		)
-		(property "Datasheet" "kicad-embed://KEM_C1002_X7R_SMD.pdf"
-			(at 109.22 71.12 0)
-			(effects
-				(font
-					(size 1.27 1.27)
-				)
-				(hide yes)
-			)
-		)
-		(property "Description" "CAP CER 10UF 16V X7R 1206"
+		(property "Datasheet" "kicad-embed://CL_Series_MLCC_ds.pdf"
+			(at 109.22 71.12 0)
+			(effects
+				(font
+					(size 1.27 1.27)
+				)
+				(hide yes)
+			)
+		)
+		(property "Description" "CAP CER 10UF 16V X7R 0805"
 			(at 109.22 71.12 0)
 			(effects
@@
 			)
 		)
-		(property "Digikey Link" "https://www.digikey.ca/en/products/detail/kemet/c1206c106k4ractu/789657"
+		(property "Digikey Link" "https://www.digikey.ca/en/products/detail/samsung-electro-mechanics/CL21B106KOQNNNE/3888530"
 			(at 109.22 71.12 0)
 			(effects
@@
 			)
 		)
-		(property "Manufacturer" "KEMET"
+		(property "Manufacturer" "Samsung Electro-Mechanics"
 			(at 109.22 71.12 0)
 			(effects
@@
 			)
 		)
-		(property "Manufacturer Part" "C1206C106K4RACTU"
+		(property "Manufacturer Part" "CL21B106KOQNNNE"
 			(at 109.22 71.12 0)
 			(effects
@@
 			)
 		)
-		(property "Supplier P/N" "399-C1206C106K4RACTUCT-ND"
+		(property "Supplier P/N" "1276-2872-1-ND"
 			(at 109.22 71.12 0)
 			(effects
@@
 			)
 		)
-		(property "Package" "1206 (3216 Metric)"
-			(at 109.22 71.12 0)
-			(effects
-				(font
-					(size 1.27 1.27)
-				)
-				(hide yes)
-			)
-		)
-		(property "Price" "0.31"
-			(at 109.22 71.12 0)
-			(effects
+		(property "Package" "0805"
+			(at 109.22 71.12 0)
+			(effects
+				(font
+					(size 1.27 1.27)
+				)
+				(hide yes)
+			)
+		)
+		(property "Price" "0.22"
+			(at 109.22 71.12 0)
+			(effects

Commit message: Assigned capacitor footprints
Parts:
- C6: footprint Capacitor_SMD:C_1206_3216Metric -> Capacitor_SMD:C_0805_2012Metric
Changed lines of the file:
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@@
 			)
 		)
-		(property "Footprint" "Capacitor_SMD:C_1206_3216Metric"
+		(property "Footprint" "Capacitor_SMD:C_0805_2012Metric"
 			(at 109.22 71.12 0)
 			(effects

Commit message: Added side B for SW1
Parts:
- C6: symbol PCM_Elektuur:C -> capstone_parts:C
- J18: symbol PCM_4ms_Connector:Conn_01x03 -> capstone_parts:Conn_01x03
- J7: symbol Connector:USB_B_Micro -> capstone_parts:USB_B_Micro
Changed lines of the file:
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@@
 	)
 	(symbol
-		(lib_id "PCM_4ms_Connector:Conn_01x03")
+		(lib_id "capstone_parts:Conn_01x03")
 		(at 246.38 86.36 0)
 		(unit 1)
@@
 	)
 	(symbol
-		(lib_id "Connector:USB_B_Micro")
+		(lib_id "capstone_parts:USB_B_Micro")
 		(at 91.44 83.82 0)
 		(unit 1)
@@
 	)
 	(symbol
-		(lib_id "PCM_Elektuur:C")
+		(lib_id "capstone_parts:C")
 		(at 109.22 71.12 0)
 		(mirror y)

Commit message: Place CM4 footprint, starting to reroute everything
Connections:
- net MICROD-: now reaches J7.2 (D-), U11.4, U5.2 (1D-)
- net MICROD+: now reaches J7.3 (D+), U11.5, U5.1 (1D+)
Changed lines of the file:
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@@
+		)
+	)
+	(label "MICROD-"
+		(at 120.65 86.36 0)
+		(effects
+			(font
+				(size 1.27 1.27)
+			)
+			(justify left bottom)
+		)
+	)
+	(label "MICROD+"
+		(at 120.65 83.82 0)
+		(effects
+			(font
+				(size 1.27 1.27)
+			)
+			(justify left bottom)
 		)
 	)

Commit message: Friday, March 20th: PCB Final for BOM
Parts:
- J18: footprint *CapStone*:CON3_1X3_TU_HTS_SAI - 3POS Connector -> capstone:CON3_1X3_TU_HTS_SAI - 3POS Connector
- U11: footprint *CapStone*:SOT553_LTF_SP3003_02XTG -> capstone:SOT553_LTF_SP3003_02XTG
- U5: footprint *CapStone*:RSE10 -> capstone:RSE10
Changed lines of the file:
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@@
 			)
 		)
-		(property "Footprint" "*CapStone*:CON3_1X3_TU_HTS_SAI - 3POS Connector"
+		(property "Footprint" "capstone:CON3_1X3_TU_HTS_SAI - 3POS Connector"
 			(at 246.38 79.375 0)
 			(effects
@@
 		)
 		(property "Unit" "pcs"
+			(at 246.38 86.36 0)
+			(effects
+				(font
+					(size 1.27 1.27)
+				)
+				(hide yes)
+			)
+		)
+		(property "OPTION" ""
 			(at 246.38 86.36 0)
 			(effects
@@
 			)
 		)
+		(property "OPTION" ""
+			(at 91.44 83.82 0)
+			(effects
+				(font
+					(size 1.27 1.27)
+				)
+				(hide yes)
+			)
+		)
 		(pin "2"
 		)
@@
 			)
 		)
-		(property "Footprint" "*CapStone*:RSE10"
+		(property "Footprint" "capstone:RSE10"
 			(at 165.1 83.82 0)
 			(effects
@@
 		)
 		(property "Voltage Rating" ""
+			(at 165.1 83.82 0)
+			(effects
+				(font
+					(size 1.27 1.27)
+				)
+				(hide yes)
+			)
+		)
+		(property "OPTION" ""
 			(at 165.1 83.82 0)
 			(effects
@@
 			)
 		)
+		(property "OPTION" ""
+			(at 109.22 71.12 0)
+			(effects
+				(font
+					(size 1.27 1.27)
+				)
+				(hide yes)
+			)
+		)
 		(pin "2"
 		)
@@
 			)
 		)
-		(property "Footprint" "*CapStone*:SOT553_LTF_SP3003_02XTG"
+		(property "Footprint" "capstone:SOT553_LTF_SP3003_02XTG"
 			(at 137.16 119.38 0)
 			(effects
@@
 			(at 137.16 119.38 90)
 			(effects
+				(font
+					(size 1.27 1.27)
+				)
+				(hide yes)
+			)
+		)
+		(property "OPTION" ""
+			(at 137.16 119.38 90)
+			(effects
