File: 490_0/PCB3.kicad_sch (KiCad schematic)
At the start: 7 parts, among them J13 S2B-ZR, J14 Conn_01x10, J22 2000-1-1-20-00-BK, J8 0522711579, U12 TPD8S009DSMR

Commit message: Added side B for SW1
Parts:
- D22, D23: symbol PCM_Diode_TVS_AKL:SMF5.0A -> capstone_parts:SMF5.0A
- J13: symbol PCM_4ms_Connector:Conn_01x02 -> capstone_parts:Conn_01x02
- J14: symbol Connector_Generic:Conn_01x10 -> capstone_parts:Conn_01x10
- J22: symbol Connector:HDMI_A -> capstone_parts:HDMI_A
- J8: symbol Connector_Generic:Conn_01x15 -> capstone_parts:Conn_01x15
Connections:
- net GND2 is gone; now on net GND_GLASSES: J14.10 (Pin_10)
Changed lines of the file:
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@@
 	)
 	(junction
-		(at 195.58 55.88)
-		(diameter 0)
-		(color 0 0 0 0)
-	)
-	(junction
 		(at 129.54 106.68)
 		(diameter 0)
@@
 	)
 	(junction
+		(at 190.5 53.34)
+		(diameter 0)
+		(color 0 0 0 0)
+	)
+	(junction
 		(at 77.47 96.52)
 		(diameter 0)
@@
 	(wire
 		(pts
-			(xy 195.58 66.04) (xy 195.58 55.88)
-		)
-		(stroke
-			(width 0)
-			(type default)
-		)
-	)
-	(wire
-		(pts
 			(xy 185.42 30.48) (xy 185.42 33.02)
 		)
@@
 	(wire
 		(pts
-			(xy 129.54 106.68) (xy 129.54 132.08)
+			(xy 190.5 53.34) (xy 198.12 53.34)
 		)
 		(stroke
@@
 	(wire
 		(pts
-			(xy 177.8 116.84) (xy 200.66 116.84)
+			(xy 129.54 106.68) (xy 129.54 132.08)
 		)
 		(stroke
@@
 	(wire
 		(pts
-			(xy 83.82 185.42) (xy 86.36 185.42)
+			(xy 177.8 116.84) (xy 200.66 116.84)
 		)
 		(stroke
@@
 	(wire
 		(pts
-			(xy 142.24 25.4) (xy 149.86 25.4)
+			(xy 83.82 185.42) (xy 86.36 185.42)
 		)
 		(stroke
@@
 	(wire
 		(pts
-			(xy 172.72 109.22) (xy 172.72 124.46)
+			(xy 142.24 25.4) (xy 149.86 25.4)
 		)
 		(stroke
@@
 	(wire
 		(pts
-			(xy 195.58 55.88) (xy 195.58 53.34)
+			(xy 172.72 109.22) (xy 172.72 124.46)
 		)
 		(stroke
@@
 	(wire
 		(pts
-			(xy 190.5 63.5) (xy 190.5 50.8)
+			(xy 190.5 63.5) (xy 190.5 53.34)
 		)
 		(stroke
@@
 	(wire
 		(pts
-			(xy 195.58 55.88) (xy 210.82 55.88)
-		)
-		(stroke
-			(width 0)
-			(type default)
-		)
-	)
-	(wire
-		(pts
 			(xy 149.86 25.4) (xy 149.86 40.64)
 		)
@@
 	(wire
 		(pts
-			(xy 195.58 53.34) (xy 198.12 53.34)
-		)
-		(stroke
-			(width 0)
-			(type default)
-		)
-	)
-	(wire
-		(pts
 			(xy 219.71 149.86) (xy 219.71 152.4)
 		)
@@
 	(wire
 		(pts
+			(xy 190.5 53.34) (xy 190.5 50.8)
+		)
+		(stroke
+			(width 0)
+			(type default)
+		)
+	)
+	(wire
+		(pts
 			(xy 67.31 101.6) (xy 180.34 101.6)
 		)
@@
 	(wire
 		(pts
-			(xy 190.5 63.5) (xy 210.82 63.5)
+			(xy 190.5 63.5) (xy 198.12 63.5)
 		)
 		(stroke
@@
 	)
 	(symbol
-		(lib_id "Connector_Generic:Conn_01x15")
+		(lib_id "capstone_parts:Conn_01x15")
 		(at 33.02 101.6 0)
 		(mirror y)
@@
 	)
 	(symbol
-		(lib_id "PCM_4ms_Power-symbol:GNDA")
-		(at 195.58 66.04 0)
-		(unit 1)
-		(exclude_from_sim no)
-		(in_bom yes)
-		(on_board yes)
-		(dnp no)
-		(property "Reference" "#PWR0147"
-			(at 195.58 72.39 0)
-			(effects
-				(font
-					(size 1.27 1.27)
-				)
-				(hide yes)
-			)
-		)
-		(property "Value" "GND2"
-			(at 195.58 69.596 0)
-			(effects
-				(font
-					(size 1.27 1.27)
-				)
-			)
-		)
-		(property "Footprint" ""
-			(at 195.58 66.04 0)
-			(effects
-				(font
-					(size 1.27 1.27)
-				)
-				(hide yes)
-			)
-		)
-		(property "Datasheet" ""
-			(at 195.58 66.04 0)
-			(effects
-				(font
-					(size 1.27 1.27)
-				)
-				(hide yes)
-			)
-		)
-		(property "Description" "(analog) ground power-flag symbol"
-			(at 195.58 66.04 0)
-			(effects
-				(font
-					(size 1.27 1.27)
-				)
-				(hide yes)
-			)
-		)
-		(pin "1"
-		)
-		(instances
-			(project ""
-				(path "/365a82ed-827d-43e1-aa2f-b98221c4179c/a8971e06-9d2b-4df6-83ab-783791bb1c3f"
-					(reference "#PWR0147")
-					(unit 1)
-				)
-			)
-		)
-	)
-	(symbol
-		(lib_id "PCM_4ms_Connector:Conn_01x02")
+		(lib_id "capstone_parts:Conn_01x02")
 		(at 33.02 53.34 180)
 		(unit 1)
@@
 	)
 	(symbol
-		(lib_id "power:PWR_FLAG")
-		(at 210.82 55.88 0)
-		(unit 1)
-		(exclude_from_sim no)
-		(in_bom yes)
-		(on_board yes)
-		(dnp no)
-		(fields_autoplaced yes)
-		(property "Reference" "#FLG09"
-			(at 210.82 53.975 0)
-			(effects
-				(font
-					(size 1.27 1.27)
-				)
-				(hide yes)
-			)
-		)
-		(property "Value" "PWR_FLAG"
-			(at 210.82 50.8 0)
-			(effects
-				(font
-					(size 1.27 1.27)
-				)
-			)
-		)
-		(property "Footprint" ""
-			(at 210.82 55.88 0)
-			(effects
-				(font
-					(size 1.27 1.27)
-				)
-				(hide yes)
-			)
-		)
-		(property "Datasheet" "~"
-			(at 210.82 55.88 0)
-			(effects
-				(font
-					(size 1.27 1.27)
-				)
-				(hide yes)
-			)
-		)
-		(property "Description" "Special symbol for telling ERC where power comes from"
-			(at 210.82 55.88 0)
-			(effects
-				(font
-					(size 1.27 1.27)
-				)
-				(hide yes)
-			)
-		)
-		(pin "1"
-		)
-		(instances
-			(project "490_0"
-				(path "/365a82ed-827d-43e1-aa2f-b98221c4179c/a8971e06-9d2b-4df6-83ab-783791bb1c3f"
-					(reference "#FLG09")
-					(unit 1)
-				)
-			)
-		)
-	)
-	(symbol
 		(lib_id "power:+3.3V")
 		(at 40.64 48.26 0)
@@
 	)
 	(symbol
-		(lib_id "Connector_Generic:Conn_01x10")
+		(lib_id "capstone_parts:Conn_01x10")
 		(at 203.2 40.64 0)
 		(unit 1)
@@
 	)
 	(symbol
-		(lib_id "Connector:HDMI_A")
+		(lib_id "capstone_parts:HDMI_A")
 		(at 210.82 106.68 0)
 		(unit 1)
@@
 	(symbol
 		(lib_id "power:PWR_FLAG")
-		(at 210.82 63.5 0)
+		(at 198.12 63.5 0)
 		(unit 1)
 		(exclude_from_sim no)
@@
 		(fields_autoplaced yes)
 		(property "Reference" "#FLG010"
-			(at 210.82 61.595 0)
+			(at 198.12 61.595 0)
 			(effects
 				(font
@@
 		)
 		(property "Value" "PWR_FLAG"
-			(at 210.82 58.42 0)
+			(at 198.12 58.42 0)
 			(effects
 				(font
@@
 		)
 		(property "Footprint" ""
-			(at 210.82 63.5 0)
+			(at 198.12 63.5 0)
 			(effects
 				(font
@@
 		)
 		(property "Datasheet" "~"
-			(at 210.82 63.5 0)
+			(at 198.12 63.5 0)
 			(effects
 				(font
@@
 		)
 		(property "Description" "Special symbol for telling ERC where power comes from"
-			(at 210.82 63.5 0)
+			(at 198.12 63.5 0)
 			(effects
 				(font
@@
 	)
 	(symbol
-		(lib_id "PCM_Diode_TVS_AKL:SMF5.0A")
+		(lib_id "capstone_parts:SMF5.0A")
 		(at 43.18 125.73 90)
 		(unit 1)
@@
 	)
 	(symbol
-		(lib_id "PCM_Diode_TVS_AKL:SMF5.0A")
+		(lib_id "capstone_parts:SMF5.0A")
 		(at 111.76 125.73 90)
 		(unit 1)

Commit message: Rerouted + external coponents update
Parts:
- removed J14: Conn_01x10, Connector_JST:JST_XH_S10B-XH-A-1_1x10_P2.50mm_Horizontal, symbol capstone_parts:Conn_01x10
- added J23: S3B-XH-A, Connector_JST:JST_XH_S3B-XH-A_1x03_P2.50mm_Horizontal, symbol capstone_parts:Conn_01x03
- added U15: SP3003-02XTG, *CapStone*:SOT553_LTF_SP3003_02XTG, symbol capstone_parts:SP3003-02XTG
Connections:
- net +3.3V_GLASSES: now also J23.2 (Pin_2), U15.3
- net +5V_GLASSES: now also J23.3 (Pin_3)
- net GND_GLASSES: now also J23.1 (Pin_1), U15.2
- net PCB2-PWM and Motors/I2C_SCL: now also J22.15 (SCL), J8.13 (Pin_13), U15.5
- net PCB2-PWM and Motors/I2C_SDA: now also J22.16 (SDA), J8.14 (Pin_14), U15.4
- net PCB2-USB 2.0 Bridge/USB_N: now also J22.3 (D2-), U12.12 (D3-)
- net PCB2-USB 2.0 Bridge/USB_P: now also J22.1 (D2+), U12.10 (D3+)
- no-connect marks 6 -> 5
Other:
- sheet PCB2-USB 2.0 Bridge ports: added none; removed HUB_RESET_N
- note removed: "HUB_RESET_N"
- note removed: "I2C_SCL"
- note removed: "I2C_SDA"
- moved on the sheet: D22, J13, U12

Commit message: 15 pin connector mirrored
Connections:
- net GND_GLASSES: now also J8.12 (Pin_12), J8.15 (Pin_15), J8.6 (Pin_6), J8.9 (Pin_9); no longer J8.1 (Pin_1), J8.10 (Pin_10), J8.4 (Pin_4), J8.7 (Pin_7)
- net PCB2-PWM and Motors/I2C_SCL: now also J8.3 (Pin_3); no longer J8.13 (Pin_13)
- net PCB2-PWM and Motors/I2C_SDA: now also J8.2 (Pin_2); no longer J8.14 (Pin_14)
- net at D23.1 (K), J22.13 (CEC): now also J8.5 (Pin_5); no longer J8.11 (Pin_11)
- net at D22.1 (K), J22.18 (+5V): now also J8.1 (Pin_1); no longer J8.15 (Pin_15)
- net at J22.9 (D0-), U12.3 (D0-): now also J8.14 (Pin_14); no longer J8.2 (Pin_2)
- net at J22.7 (D0+), U12.1 (D0+): now also J8.13 (Pin_13); no longer J8.3 (Pin_3)
- net at J22.6 (D1-), U12.6 (D1-): now also J8.11 (Pin_11); no longer J8.5 (Pin_5)
- net at J22.4 (D1+), U12.4 (D1+): now also J8.10 (Pin_10); no longer J8.6 (Pin_6)
- net at J22.10 (CK+), U12.7 (D2+): now also J8.7 (Pin_7); no longer J8.9 (Pin_9)
Other:
- moved on the sheet: J8
Changed lines of the file:
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@@
 	(symbol
 		(lib_id "capstone_parts:Conn_01x15")
-		(at 33.02 101.6 0)
-		(mirror y)
+		(at 33.02 101.6 180)
 		(unit 1)
 		(exclude_from_sim no)
@@
 		(on_board yes)
 		(dnp no)
-		(fields_autoplaced yes)
 		(property "Reference" "J8"
-			(at 33.02 77.47 0)
+			(at 24.638 103.886 0)
 			(effects
 				(font
@@
 		)
 		(property "Value" "0522711579"
-			(at 33.02 80.01 0)
+			(at 24.638 106.426 0)
 			(effects
 				(font
